File: KB-01_kicad/KB-01/KB-01.kicad_sch (KiCad schematic)
At the start: 0 parts

Commit message: all
Signed-off-by: syauqi-alias <syauqi_nur@yahoo.com>
Other:
- added sheet pcie-nvme (pcie-nvme.kicad_sch)
Changed lines of the file:
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@@
 	(paper "A4")
 	(sheet
-		(at 196.215 25.4)
+		(at 174.625 34.29)
 		(size 28.575 23.495)
 		(exclude_from_sim no)
@@
 		)
 		(property "Sheetname" "gnss"
-			(at 196.215 24.6884 0)
+			(at 174.625 33.5784 0)
 			(effects
 				(font
@@
 		)
 		(property "Sheetfile" "gnss.kicad_sch"
-			(at 196.215 49.4796 0)
+			(at 174.625 58.3696 0)
 			(effects
 				(font
@@
 	)
 	(sheet
-		(at 116.84 25.4)
+		(at 95.25 34.29)
 		(size 27.94 23.495)
 		(exclude_from_sim no)
@@
 		)
 		(property "Sheetname" "battery_charger"
-			(at 116.84 24.6884 0)
+			(at 95.25 33.5784 0)
 			(effects
 				(font
@@
 		)
 		(property "Sheetfile" "battery_charger.kicad_sch"
-			(at 116.84 49.4796 0)
+			(at 95.25 58.3696 0)
 			(effects
 				(font
@@
 	)
 	(sheet
-		(at 116.84 60.96)
+		(at 95.25 69.85)
 		(size 27.94 36.83)
 		(exclude_from_sim no)
@@
 		)
 		(property "Sheetname" "CM5_high_speed"
-			(at 116.84 60.2484 0)
+			(at 95.25 69.1384 0)
 			(effects
 				(font
@@
 		)
 		(property "Sheetfile" "CM5_high_speed.kicad_sch"
-			(at 116.84 98.3746 0)
+			(at 95.25 107.2646 0)
 			(effects
 				(font
@@
 	)
 	(sheet
-		(at 157.48 60.96)
+		(at 135.89 69.85)
 		(size 27.94 37.465)
 		(exclude_from_sim no)
@@
 		)
 		(property "Sheetname" "CM5_GPIO"
-			(at 157.48 60.2484 0)
+			(at 135.89 69.1384 0)
 			(effects
 				(font
@@
 		)
 		(property "Sheetfile" "CM5_GPIO.kicad_sch"
-			(at 157.48 99.0096 0)
+			(at 135.89 107.8996 0)
 			(effects
 				(font
@@
 	)
 	(sheet
-		(at 157.48 25.4)
+		(at 174.625 69.85)
+		(size 28.575 37.465)
+		(exclude_from_sim no)
+		(in_bom yes)
+		(on_board yes)
+		(dnp no)
+		(fields_autoplaced yes)
+		(stroke
+			(width 0.1524)
+			(type solid)
+		)
+		(fill
+			(color 0 0 0 0.0000)
+		)
+		(property "Sheetname" "pcie-nvme"
+			(at 174.625 69.1384 0)
+			(effects
+				(font
+					(size 1.27 1.27)
+				)
+				(justify left bottom)
+			)
+		)
+		(property "Sheetfile" "pcie-nvme.kicad_sch"
+			(at 174.625 107.8996 0)
+			(effects
+				(font
+					(size 1.27 1.27)
+				)
+				(justify left top)
+			)
+		)
+		(instances
+			(project "KB-01"
+				(path "/e6144e29-1dc4-45a8-93e7-988a20131b94"
+					(page "7")
+				)
+			)
+		)
+	)
+	(sheet
+		(at 135.89 34.29)
 		(size 27.94 23.495)
 		(exclude_from_sim no)
@@
 		)
 		(property "Sheetname" "5v_boost_conv"
-			(at 157.48 24.6884 0)
+			(at 135.89 33.5784 0)
 			(effects
 				(font
@@
 		)
 		(property "Sheetfile" "5v_boost_conv.kicad_sch"
-			(at 157.48 49.4796 0)
-			(effects
-				(font
+			(at 135.89 58.3696 0)
+			(effects
+				(font

Commit message: up
Other:
- added sheet sensors (sensors.kicad_sch)
Changed lines of the file:
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@@
+	)
+	(sheet
+		(at 95.25 120.015)
+		(size 27.94 21.59)
+		(exclude_from_sim no)
+		(in_bom yes)
+		(on_board yes)
+		(dnp no)
+		(fields_autoplaced yes)
+		(stroke
+			(width 0.1524)
+			(type solid)
+		)
+		(fill
+			(color 0 0 0 0.0000)
+		)
+		(property "Sheetname" "sensors"
+			(at 95.25 119.3034 0)
+			(effects
+				(font
+					(size 1.27 1.27)
+				)
+				(justify left bottom)
+			)
+		)
+		(property "Sheetfile" "sensors.kicad_sch"
+			(at 95.25 142.1896 0)
+			(effects
+				(font
+					(size 1.27 1.27)
+				)
+				(justify left top)
+			)
+		)
+		(instances
+			(project "KB-01"
+				(path "/e6144e29-1dc4-45a8-93e7-988a20131b94"
+					(page "8")
+				)
+			)
+		)
 	)
 	(sheet

Commit message: up
Parts:
- added R22, R23: 4.7k, symbol Device:R
Connections:
- new net +3V3: R22.1, R23.1
- new net CM5_GPIO/I2C0_SCL: R22.2
- new net CM5_GPIO/I2C0_SDA: R23.2
Other:
- sheet 5v_boost_conv ports: added +5v, BST_EN, BST_MODE, BST_VIN; removed none
- sheet CM5_GPIO ports: added +3.3v, +5v, CAM_GPIO0, CAM_GPIO1, CC1, CC2, GPIO16, GPIO20, GPIO21, GPIO22, GPIO25, GPIO27, GPIO7, I2C0_SCL, I2C0_SDA, I2C1_SCL, I2C1_SDA, SCL0, SDA0, SPI0_CSn(0), SPI0_SCLK, SPI0_SIO(0), SPI0_SIO(1), UART4_RX, UART4_TX; removed none
- sheet CM5_high_speed ports: added +3.3v, CAM_GPIO0, CAM_GPIO1, PCIE_CLK_N, PCIE_CLK_P, PCIE_PWR_EN, PCIE_RX_N, PCIE_RX_P, PCIE_TX_N, PCIE_TX_P, PCIE_nCLKREQ, PCIE_nRST, PCIE_nWAKE, SCL0, SDA0, USB2_N, USB2_P; removed none
- sheet battery_charger ports: added BAT+, BQ_CE, BQ_INT, BQ_SCL, BQ_SDA, FG_INT, FG_SCL, FG_SDA, MUX_D+, MUX_D-, Vsys; removed none
- sheet gnss ports: added +5v, GNSS_PSU_EN, GNSS_RSTn, GNSS_RX, GNSS_SCL, GNSS_SDA, GNSS_TX, GNSS_Vbatt, GNSS_WAKEUP; removed none
- sheet pcie-nvme ports: added +5v, PCIE_CLK_N, PCIE_CLK_P, PCIE_PWR_EN, PCIE_RX_N, PCIE_RX_P, PCIE_TX_N, PCIE_TX_P, PCIE_nCLKREQ, PCIE_nRST, PCIE_nWAKE; removed none
- sheet sensors ports: added +3.3v, BMI270_CS, BMI270_INT1, BMI270_INT2, BMI270_SCK, BMI270_SDI, BMI270_SDO, BMP390_INT, BMP390_SCK, BMP390_SDA, LIS2MDL_INT, LIS2MDL_SCL, LIS2MDL_SDA, SHT40_SCK, SHT40_SDA; removed none
- note added: "MISO"
- note added: "MOSI"

Commit message: everything
Connections:
- net CM5_GPIO/I2C0_SCL renamed CM5_GPIO/I2C2_SCL
- net CM5_GPIO/I2C0_SDA renamed CM5_GPIO/I2C2_SDA
Other:
- sheet CM5_GPIO ports: added BMI270_INT1, BMI270_INT2, BMP390_INT, BQ_CE, BQ_INT, FG_INT, GNSS_PSU_EN, GNSS_RSTn, GNSS_WAKEUP, GPIO_VREF, I2C2_SCL, I2C2_SDA, I2C3_SCL, I2C3_SDA, ID_SC, ID_SD, LIS2MDL_INT, SPIO_SCLK, SPIO_SIO(1), UART0_RX, UART0_TX; removed CAM_GPIO0, CAM_GPIO1, CC1, CC2, GPIO16, GPIO20, GPIO21, GPIO22, GPIO25, GPIO27, GPIO7, I2C0_SCL, I2C0_SDA, SPI0_SCLK, SPI0_SIO(1), UART4_RX, UART4_TX
- sheet CM5_high_speed ports: added USBOTG_ID; removed none
- note added: "Has internal 1.8k pull-up"

Commit message: all
Connections:
- no-connect marks 0 -> 8
Other:
- sheet 5v_boost_conv renamed 5V_boost_conv
- sheet battery_charger renamed Battery_charger
- sheet gnss renamed GNSS
- sheet pcie-nvme renamed PCIe_NVMe
- sheet sensors renamed Sensors
- added sheet UI (ui.kicad_sch)
- sheet 5V_boost_conv ports: added none; removed BST_EN, BST_MODE
- sheet CM5_GPIO ports: added CAM_GPIO0, CAM_GPIO1, CC1, CC2, Coin_bat, GPIO12, GPIO13, GPIO18, GPIO19, GPIO6, GPIO7; removed I2C3_SCL, I2C3_SDA
- sheet Sensors ports: added Wheel_sensor; removed none
- note added: "---->"
- note added: "Act as a peripheral"
- note added: "Barometer"
- note added: "Battery Charger"
- note added: "Battery Charger Output"
- note added: "Fuel Gauge"
- note added: "Handshake handle by battery charger (BQ)"
- note added: "Has internal 4.7k pull-up"
- note added: "IMU"
- note added: "Magnetometer"
- note added: "No camera support for this version"
- note added: "Temp & Humidity"
- note added: "pull-up res"
- company: (none) -> Otai Labs
- title: (none) -> Komputer Basikal, KB-01
- moved on the sheet: R22, R23

Commit message: all
Other:
- note added: "Done"

Commit message: all
Other:
- sheet UI ports: added +3.3v; removed none
Changed lines of the file:
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@@
+	(wire
+		(pts
+			(xy 219.71 127) (xy 219.71 129.54)
+		)
+		(stroke
+			(width 0)
+			(type default)
+		)
+	)
 	(wire
 		(pts
@@
 	)
 	(symbol
+		(lib_id "power:+3V3")
+		(at 219.71 127 0)
+		(unit 1)
+		(body_style 1)
+		(exclude_from_sim no)
+		(in_bom yes)
+		(on_board yes)
+		(in_pos_files yes)
+		(dnp no)
+		(fields_autoplaced yes)
+		(property "Reference" "#PWR076"
+			(at 219.71 130.81 0)
+			(hide yes)
+			(show_name no)
+			(do_not_autoplace no)
+			(effects
+				(font
+					(size 1.27 1.27)
+				)
+			)
+		)
+		(property "Value" "+3V3"
+			(at 219.71 121.92 0)
+			(show_name no)
+			(do_not_autoplace no)
+			(effects
+				(font
+					(size 1.27 1.27)
+				)
+			)
+		)
+		(property "Footprint" ""
+			(at 219.71 127 0)
+			(hide yes)
+			(show_name no)
+			(do_not_autoplace no)
+			(effects
+				(font
+					(size 1.27 1.27)
+				)
+			)
+		)
+		(property "Datasheet" ""
+			(at 219.71 127 0)
+			(hide yes)
+			(show_name no)
+			(do_not_autoplace no)
+			(effects
+				(font
+					(size 1.27 1.27)
+				)
+			)
+		)
+		(property "Description" "Power symbol creates a global label with name \"+3V3\""
+			(at 219.71 127 0)
+			(hide yes)
+			(show_name no)
+			(do_not_autoplace no)
+			(effects
+				(font
+					(size 1.27 1.27)
+				)
+			)
+		)
+		(pin "1"
+		)
+		(instances
+			(project "KB-01"
+				(path "/e6144e29-1dc4-45a8-93e7-988a20131b94"
+					(reference "#PWR076")
+					(unit 1)
+				)
+			)
+		)
+	)
+	(symbol
 		(lib_id "power:+5V")
 		(at 220.98 86.36 0)
@@
 			)
 		)
+		(pin "+3.3v" input
+			(at 219.71 129.54 90)
+			(effects
+				(font
+					(size 1.27 1.27)
+				)
+				(justify right)
+			)
+		)

Commit message: all
Changed lines of the file:
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@@
+		)
+	)
+	(text "Done"
+		(exclude_from_sim no)
+		(at 218.44 49.276 0)
+		(effects
+			(font
+				(size 1.27 1.27)
+				(thickness 0.254)
+				(bold yes)
+				(color 59 255 63 1)
+			)
+		)
+	)
+	(text "Done"
+		(exclude_from_sim no)
+		(at 178.562 49.276 0)
+		(effects
+			(font
+				(size 1.27 1.27)
+				(thickness 0.254)
+				(bold yes)
+				(color 59 255 63 1)
+			)
 		)
 	)
@@
 			)
 		)
+	)
+	(text "Done"
+		(exclude_from_sim no)
+		(at 128.524 48.26 0)
+		(effects
+			(font
+				(size 1.27 1.27)
+				(thickness 0.254)
+				(bold yes)
+				(color 59 255 63 1)
+			)
+		)
