File: KB-01_kicad/KB-01/KB-01.kicad_sch (KiCad schematic)
At the start: 2 parts

Commit message: all
Changed lines of the file:
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@@
+		)
+	)
+	(text "Done"
+		(exclude_from_sim no)
+		(at 43.434 125.476 0)
+		(effects
+			(font
+				(size 1.27 1.27)
+				(thickness 0.254)
+				(bold yes)
+				(color 59 255 63 1)
+			)
 		)
 	)
@@
 			)
 		)
+		(property "SNAPEDA_PN" ""
+			(at 88.9 92.71 0)
+			(hide yes)
+			(show_name no)
+			(do_not_autoplace no)
+			(effects
+				(font
+					(size 1.27 1.27)
+				)
+			)
+		)
 		(pin "1"
 		)
@@
 			)
 		)
+		(property "SNAPEDA_PN" ""
+			(at 78.74 92.71 0)
+			(hide yes)
+			(show_name no)
+			(do_not_autoplace no)
+			(effects
+				(font
+					(size 1.27 1.27)
+				)
+			)
+		)
 		(pin "1"
 		)
@@
 			)
 		)
-		(pin "BMP390_SDA" output
+		(pin "BMP390_SDA" input
 			(at 66.04 110.49 0)
 			(effects

Commit message: all
Changed lines of the file:
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@@
+		)
+	)
+	(text "Done"
+		(exclude_from_sim no)
+		(at 219.964 101.854 0)
+		(effects
+			(font
+				(size 1.27 1.27)
+				(thickness 0.254)
+				(bold yes)
+				(color 59 255 63 1)
+			)
 		)
 	)

Commit message: all
Other:
- note added: "Done, SW is keyboard sw"
Changed lines of the file:
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@@
+		)
+	)
+	(text "Done, SW is keyboard sw"
+		(exclude_from_sim no)
+		(at 219.964 142.748 0)
+		(effects
+			(font
+				(size 1.27 1.27)
+				(thickness 0.254)
+				(bold yes)
+				(color 59 255 63 1)
+			)
 		)
 	)

Commit message: all
Parts:
- R1: renamed from R22; footprint (none) -> Resistor_SMD:R_0603_1608Metric_Pad0.98x0.95mm_HandSolder; mouser (none) -> 667-ERJ-3GEYJ472V
- R2: renamed from R23; footprint (none) -> Resistor_SMD:R_0603_1608Metric_Pad0.98x0.95mm_HandSolder; mouser (none) -> 667-ERJ-3GEYJ472V
Connections:
- no-connect marks 8 -> 9
Other:
- sheet Battery_charger ports: added none; removed BAT+
- sheet CM5_GPIO ports: added USBOTG; removed GPIO_VREF
Changed lines of the file:
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@@
 		)
 	)
+	(text "Done"
+		(exclude_from_sim no)
+		(at 152.146 121.158 0)
+		(effects
+			(font
+				(size 1.27 1.27)
+				(thickness 0.254)
+				(bold yes)
+				(color 59 255 63 1)
+			)
+		)
+	)
 	(text "Temp & \nHumidity"
 		(exclude_from_sim no)
@@
 	)
 	(no_connect
-		(at 162.56 27.94)
+		(at 177.8 83.82)
 	)
 	(no_connect
-		(at 177.8 83.82)
+		(at 102.87 119.38)
 	)
 	(no_connect
@@
 	)
 	(no_connect
+		(at 102.87 121.92)
+	)
+	(no_connect
 		(at 102.87 152.4)
 	)
@@
 	(wire
 		(pts
+			(xy 162.56 27.94) (xy 158.75 27.94)
+		)
+		(stroke
+			(width 0)
+			(type default)
+		)
+	)
+	(wire
+		(pts
 			(xy 73.66 100.33) (xy 88.9 100.33)
 		)
@@
 	(wire
 		(pts
+			(xy 158.75 27.94) (xy 158.75 83.82)
+		)
+		(stroke
+			(width 0)
+			(type default)
+		)
+	)
+	(wire
+		(pts
 			(xy 128.27 76.2) (xy 128.27 81.28)
 		)
@@
 		(in_pos_files yes)
 		(dnp no)
-		(property "Reference" "#PWR054"
+		(property "Reference" "#PWR01"
 			(at 181.61 25.4 0)
 			(hide yes)
@@
 			(project "KB-01"
 				(path "/e6144e29-1dc4-45a8-93e7-988a20131b94"
-					(reference "#PWR054")
+					(reference "#PWR01")
 					(unit 1)
 				)
@@
 		(in_pos_files yes)
 		(dnp no)
-		(property "Reference" "#PWR049"
+		(property "Reference" "#PWR04"
 			(at 148.59 85.09 0)
 			(hide yes)
@@
 			(project "KB-01"
 				(path "/e6144e29-1dc4-45a8-93e7-988a20131b94"
-					(reference "#PWR049")
+					(reference "#PWR04")
 					(unit 1)
 				)
@@
 		(dnp no)
 		(fields_autoplaced yes)
-		(property "Reference" "R23"
+		(property "Reference" "R2"
 			(at 91.44 91.4399 0)
 			(show_name no)
@@
 			)
 		)
-		(property "Footprint" ""
+		(property "Footprint" "Resistor_SMD:R_0603_1608Metric_Pad0.98x0.95mm_HandSolder"
 			(at 87.122 92.71 90)
 			(hide yes)
@@
 			)
 		)
+		(property "mouser" "667-ERJ-3GEYJ472V"
+			(at 88.9 92.71 0)
+			(hide yes)
+			(show_name no)
+			(do_not_autoplace no)
+			(effects
+				(font
+					(size 1.27 1.27)
+				)
+			)
+		)
 		(pin "1"
 		)
@@
 			(project "KB-01"
 				(path "/e6144e29-1dc4-45a8-93e7-988a20131b94"
-					(reference "R23")
+					(reference "R2")
 					(unit 1)
 				)
@@
 		(dnp no)
 		(fields_autoplaced yes)
-		(property "Reference" "#PWR028"
+		(property "Reference" "#PWR06"
 			(at 83.82 88.9 0)
 			(hide yes)
@@
 			(project "KB-01"
 				(path "/e6144e29-1dc4-45a8-93e7-988a20131b94"
-					(reference "#PWR028")
+					(reference "#PWR06")
 					(unit 1)
 				)
@@
 		(in_pos_files yes)
 		(dnp no)
-		(property "Reference" "#PWR052"
+		(property "Reference" "#PWR02"
 			(at 217.17 25.4 0)
 			(hide yes)
@@
 			(project "KB-01"
 				(path "/e6144e29-1dc4-45a8-93e7-988a20131b94"
-					(reference "#PWR052")
+					(reference "#PWR02")
 					(unit 1)
 				)
@@
 		(dnp no)
 		(fields_autoplaced yes)
-		(property "Reference" "#PWR05"
+		(property "Reference" "#PWR03"
 			(at 59.69 43.18 0)
 			(hide yes)
@@
 			(project "KB-01"
 				(path "/e6144e29-1dc4-45a8-93e7-988a20131b94"
-					(reference "#PWR05")
+					(reference "#PWR03")
 					(unit 1)
 				)
@@
 		(dnp no)
 		(fields_autoplaced yes)
-		(property "Reference" "#PWR032"
+		(property "Reference" "#PWR07"
 			(at 46.99 90.17 0)
 			(hide yes)
@@
 			(project "KB-01"
 				(path "/e6144e29-1dc4-45a8-93e7-988a20131b94"
-					(reference "#PWR032")
+					(reference "#PWR07")
 					(unit 1)
 				)
@@
 		(dnp no)
 		(fields_autoplaced yes)
-		(property "Reference" "R22"
+		(property "Reference" "R1"
 			(at 81.28 91.4399 0)
 			(show_name no)
@@
 			)
 		)
-		(property "Footprint" ""
+		(property "Footprint" "Resistor_SMD:R_0603_1608Metric_Pad0.98x0.95mm_HandSolder"
 			(at 76.962 92.71 90)
 			(hide yes)
@@
 			)
 		)
+		(property "mouser" "667-ERJ-3GEYJ472V"
+			(at 78.74 92.71 0)
+			(hide yes)
+			(show_name no)
+			(do_not_autoplace no)
+			(effects
+				(font
+					(size 1.27 1.27)
+				)
+			)
+		)
 		(pin "1"
 		)
@@
 			(project "KB-01"
 				(path "/e6144e29-1dc4-45a8-93e7-988a20131b94"
-					(reference "R22")
+					(reference "R1")
 					(unit 1)
 				)
@@
 		(in_pos_files yes)
 		(dnp no)
-		(property "Reference" "#PWR043"
+		(property "Reference" "#PWR05"
 			(at 151.13 85.09 0)
 			(hide yes)
@@
 			(project "KB-01"
 				(path "/e6144e29-1dc4-45a8-93e7-988a20131b94"
-					(reference "#PWR043")
+					(reference "#PWR05")
 					(unit 1)
 				)
@@
 		(dnp no)
 		(fields_autoplaced yes)
-		(property "Reference" "#PWR076"
+		(property "Reference" "#PWR09"
 			(at 219.71 130.81 0)
 			(hide yes)
@@
 			(project "KB-01"
 				(path "/e6144e29-1dc4-45a8-93e7-988a20131b94"
-					(reference "#PWR076")
+					(reference "#PWR09")
 					(unit 1)
 				)
@@
 		(in_pos_files yes)
 		(dnp no)
-		(property "Reference" "#PWR055"
+		(property "Reference" "#PWR08"
 			(at 220.98 90.17 0)
 			(hide yes)
@@
 			(project "KB-01"
 				(path "/e6144e29-1dc4-45a8-93e7-988a20131b94"
-					(reference "#PWR055")
+					(reference "#PWR08")
 					(unit 1)
 				)
@@
 			)
 		)
-		(pin "BAT+" input
-			(at 124.46 24.13 90)
-			(effects
-				(font
-					(size 1.27 1.27)
-				)
-				(justify right)
-			)
-		)
 		(instances
 			(project "KB-01"
@@
 			)
 		)
-		(pin "GPIO_VREF" output
-			(at 153.67 83.82 90)
-			(effects
-				(font
-					(size 1.27 1.27)
-				)
-				(justify right)
-			)
-		)
 		(pin "ID_SC" output
 			(at 102.87 119.38 180)
@@
 			(effects
 				(font
+					(size 1.27 1.27)
+				)
+				(justify right)
+			)
+		)
+		(pin "USBOTG" output
+			(at 158.75 83.82 90)
+			(effects
+				(font

Commit message: all
Connections:
- no-connect marks 9 -> 4
Other:
- sheet CM5_high_speed ports: added ID_SC, ID_SD; removed CAM_GPIO1
- note removed: "No camera support for this version"
Changed lines of the file:
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@@
-		)
-	)
-	(text "No camera support\nfor this version"
-		(exclude_from_sim no)
-		(at 177.038 80.264 0)
-		(effects
-			(font
-				(size 1.27 1.27)
-			)
-			(justify left)
 		)
 	)
@@
 	)
 	(no_connect
-		(at 180.34 76.2)
-	)
-	(no_connect
 		(at 205.74 113.03)
-	)
-	(no_connect
-		(at 177.8 76.2)
 	)
 	(no_connect
@@
 	)
 	(no_connect
-		(at 177.8 83.82)
-	)
-	(no_connect
-		(at 102.87 119.38)
-	)
-	(no_connect
 		(at 102.87 154.94)
-	)
-	(no_connect
-		(at 102.87 121.92)
 	)
 	(no_connect
@@
 	(wire
 		(pts
+			(xy 177.8 76.2) (xy 177.8 83.82)
+		)
+		(stroke
+			(width 0)
+			(type default)
+		)
+	)
+	(wire
+		(pts
 			(xy 196.85 147.32) (xy 205.74 147.32)
 		)
@@
 	(wire
 		(pts
+			(xy 182.88 76.2) (xy 182.88 83.82)
+		)
+		(stroke
+			(width 0)
+			(type default)
+		)
+	)
+	(wire
+		(pts
 			(xy 196.85 59.69) (xy 201.93 59.69)
 		)
@@
 	(wire
 		(pts
+			(xy 185.42 76.2) (xy 185.42 83.82)
+		)
+		(stroke
+			(width 0)
+			(type default)
+		)
+	)
+	(wire
+		(pts
 			(xy 196.85 48.26) (xy 201.93 48.26)
 		)
@@
 		(pts
 			(xy 196.85 63.5) (xy 201.93 63.5)
-		)
-		(stroke
-			(width 0)
-			(type default)
-		)
-	)
-	(wire
-		(pts
-			(xy 177.8 76.2) (xy 180.34 76.2)
 		)
 		(stroke
@@
 			)
 		)
-		(pin "CAM_GPIO1" input
-			(at 180.34 76.2 270)
-			(effects
-				(font
-					(size 1.27 1.27)
-				)
-				(justify left)
-			)
-		)
 		(pin "PCIE_CLK_N" output
 			(at 196.85 48.26 0)
@@
 		(pin "SCL0" input
 			(at 172.72 76.2 270)
+			(effects
+				(font
+					(size 1.27 1.27)
+				)
+				(justify left)
+			)
+		)
+		(pin "ID_SC" input
+			(at 182.88 76.2 270)
+			(effects
+				(font
+					(size 1.27 1.27)
+				)
+				(justify left)
+			)
+		)
+		(pin "ID_SD" input
+			(at 185.42 76.2 270)
 			(effects
 				(font
@@
 		)
 		(pin "ID_SC" output
-			(at 102.87 119.38 180)
-			(effects
-				(font
-					(size 1.27 1.27)
-				)
-				(justify left)
+			(at 182.88 83.82 90)
+			(effects
+				(font
+					(size 1.27 1.27)
+				)
+				(justify right)
 			)
 		)
 		(pin "ID_SD" output
-			(at 102.87 121.92 180)
-			(effects
-				(font
-					(size 1.27 1.27)
-				)
-				(justify left)
-			)
-		)
+			(at 185.42 83.82 90)
+			(effects
+				(font
+					(size 1.27 1.27)
+				)
+				(justify right)
+			)
+		)
