File: KB-01_kicad/KB-01/battery_charger.kicad_sch (KiCad schematic)
At the start: 1 part, among them U1 BQ25895RTW

Commit message: all
Signed-off-by: syauqi-alias <syauqi_nur@yahoo.com>
Parts:
- added C10: 47nF 16V, Capacitor_SMD:C_0603_1608Metric_Pad1.08x0.95mm_HandSolder, symbol Device:C
- added C11, C12, C14: 10uF 16V, Capacitor_SMD:C_0603_1608Metric_Pad1.08x0.95mm_HandSolder, symbol Device:C
- added C13: 4.7uF 16V, Capacitor_SMD:C_0603_1608Metric_Pad1.08x0.95mm_HandSolder, symbol Device:C
- added C15, C16: 22uF 16V, Capacitor_SMD:C_0603_1608Metric_Pad1.08x0.95mm_HandSolder, symbol Device:C
- added C17: 1uF 25V, Capacitor_SMD:C_0603_1608Metric_Pad1.08x0.95mm_HandSolder, symbol Device:C
- added C18, C19: 0.1uF 16V, Capacitor_SMD:C_0603_1608Metric_Pad1.08x0.95mm_HandSolder, symbol Device:C
- added D2: Green, Diode_SMD:D_0603_1608Metric_Pad1.05x0.95mm_HandSolder, symbol Device:D
- added IC1: MAX17048G+T10, SON50P200X200X80-9N-D, symbol MAX17048G+T10:MAX17048G+T10
- added J2: Conn_01x02_Socket, Connector_JST:JST_XH_B2B-XH-AM_1x02_P2.50mm_Vertical, symbol Connector:Conn_01x02_Socket
- added J3: USB_C_Receptacle_USB2.0_14P, Connector_USB:USB_C_Receptacle_JAE_DX07S016JA1R1500, symbol Connector:USB_C_Receptacle_USB2.0_14P
- added J4: NTC (optional), Connector_Wire:SolderWire-0.1sqmm_1x01_D0.4mm_OD1mm, symbol Connector:Conn_01x01_Socket
- added L2: 1.0uH, Inductor_SMD:L_Coilcraft_XAL5030-XXX, symbol Device:L
- added R10, R11, R12, R13, R14: 10K, Resistor_SMD:R_0603_1608Metric_Pad0.98x0.95mm_HandSolder, symbol Device:R
- added R5: 2.21K, Resistor_SMD:R_0603_1608Metric_Pad0.98x0.95mm_HandSolder, symbol Device:R
- added R6, R7: 5.1k, Resistor_SMD:R_0603_1608Metric_Pad0.98x0.95mm_HandSolder, symbol MCU_RaspberryPi_RP2350:R
- added R8: 133, Resistor_SMD:R_0603_1608Metric_Pad0.98x0.95mm_HandSolder, symbol Device:R
- added R9: R, Resistor_SMD:R_0603_1608Metric_Pad0.98x0.95mm_HandSolder, symbol Device:R
- added U6: TS3USB30ERSWR, Package_DFN_QFN:UQFN-10_1.4x1.8mm_P0.4mm, symbol Interface_USB:TS3USB30ERSWR
- U1: value BQ25895RTW -> BQ25895; mouser (none) -> 595-BQ25895RTWR
Connections:
- net VBUS: now reaches U1.1 (VBUS)
- net VBUS: now also C17.1, J3.A4 (VBUS), J3.A9 (VBUS), J3.B4 (VBUS), J3.B9 (VBUS)
- net at U1.10 (ILIM): now also R8.1
- net at U1.11 (TS): now also J4.1 (Pin_1), R13.2, R14.1
- net RESET: now reaches U1.12 (~{QON})
- net BAT+: now reaches U1.13 (BAT), U1.14 (BAT)
- net BAT+: now also C14.1, C18.1, C19.1, IC1.2 (CELL), IC1.3 (VDD), J2.1 (Pin_1)
- net Vsys: now reaches U1.15 (SYS), U1.16 (SYS)
- net Vsys: now also C11.1, C12.1, L2.2, R5.2
- net GND: now reaches U1.17 (PGND), U1.18 (PGND), U1.25 (PGND)
- net GND: now also C11.2, C12.2, C13.2, C14.2, C15.2, C16.2, C17.2, C18.2, C19.2, IC1.1 (CTG), IC1.4 (GND), IC1.6 (QSTRT), IC1.9 (EP), J2.2 (Pin_2), J3.A1 (GND), J3.A12 (GND), J3.B1 (GND), J3.B12 (GND), J3.S1 (SHIELD), R11.2, R12.2, R14.2, R6.2, R7.1, R8.2, U6.8 (~{OE})
- net at U1.19 (SW), U1.20 (SW): now also C10.1, L2.1
- net CHG_D+: now reaches U1.2 (D+)
- net CHG_D+: now also U6.1 (D1+)
- net at U1.21 (BTST): now also C10.2
- net at U1.22 (REGN): now also C13.1, R13.1
- net at U1.23 (PMID): now also C15.1, C16.1
- net SEL: now reaches U1.24 (DSEL)
- net SEL: now also R9.1, U6.10 (S)
- net CHG_D-: now reaches U1.3 (D-)
- net CHG_D-: now also U6.7 (D1-)
- net at U1.4 (STAT): now also D2.1 (K)
- net SCL: now reaches U1.5 (SCL)
- net SCL: now also IC1.7 (SCL)
- net SDA: now reaches U1.6 (SDA)
- net SDA: now also IC1.8 (SDA)
- net INT: now reaches U1.7 (~{INT})
- net INT: now also R10.2
- net OTG: now reaches U1.8 (OTG)
- net OTG: now also R11.1
- net CE: now reaches U1.9 (~{CE})
- net CE: now also R12.1
- new net: D2.2 (A), R5.1
- new net: J3.A5 (CC1), R6.1
- new net: J3.B5 (CC2), R7.2
- new net +3V3: R10.1, R9.2
- new net FG_ALERT: IC1.5 (~{ALRT})
- new net MUX_D+: U6.2 (D2+)
- new net MUX_D-: U6.6 (D2-)
- new net USB_D+: J3.A6 (D+), J3.B6 (D+), U6.5 (D-)
- new net USB_D-: J3.A7 (D-), J3.B7 (D-), U6.3 (D+)
Other:
- note added: "906090 3.7V 6000mAh"
- note added: "MAX17048 Fuel Gauge"
- note added: "USB current input limit"
- note added: "USB-C"
- note added: "charging status LED"
- note added: "close to the IC"
- note added: "connect with menu button"
- note added: "to boost converter"
- moved on the sheet: U1

Commit message: up
Parts:
- removed J4: NTC (optional), Connector_Wire:SolderWire-0.1sqmm_1x01_D0.4mm_OD1mm, symbol Connector:Conn_01x01_Socket
- added C45: 4.7uF, Capacitor_SMD:C_0603_1608Metric_Pad1.08x0.95mm_HandSolder, symbol Device:C
- added C46: 1uF 25V, Capacitor_SMD:C_0603_1608Metric_Pad1.08x0.95mm_HandSolder, symbol Device:C
- added C47: 0.1uF, Capacitor_SMD:C_0603_1608Metric_Pad1.08x0.95mm_HandSolder, symbol Device:C
- added D8: BAT54-05W, Package_TO_SOT_SMD:SOT-323_SC-70, symbol Device:D_Schottky_Dual_CommonCathode_AAK_Parallel
- added J8: Bat NTC 10k, symbol Connector:Conn_01x02_Socket
- added SW2: Power button, symbol Switch:SW_Push
- added TP1, TP2: TestPoint, TestPoint:TestPoint_Pad_1.0x1.0mm, symbol Connector:TestPoint
- added U14: TLV70430DBVR, DBV0005A_N, symbol TLV704:TLV70430DBVR
- C10: value 47nF 16V -> 47nF 25V
- C11, C12, C14: value 10uF 16V -> 10uF 25V
- C15: value 22uF 16V -> 10uF 25V
- C16: value 22uF 16V -> 0.1uF 25V
- C18, C19: value 0.1uF 16V -> 0.1uF 25V
- R9: value R -> 10k
Connections:
- net +3V3: now also R11.1; no longer R9.2
- net BAT+: now also D8.2 (A)
- net GND: now also U1.8 (OTG), U6.4 (GND), C45.2, C46.2, C47.2, J8.2 (Pin_2), SW2.1, U14.1 (GND); no longer R11.2
- net RESET: now also SW2.2
- net VBUS: now also D8.1 (A)
- net Vsys: now also TP1.1
- net at R13.2, R14.1, U1.11 (TS): now also J8.1 (Pin_1)
- net +3V_CHRG: now reaches U6.9 (VCC)
- net +3V_CHRG: now also R9.2, C45.1, C47.1, TP2.1, U14.3 (OUT)
- net CE renamed BQ_CE
- net FG_ALERT renamed FG_INT
- net FG_INT: now also R11.2
- net INT renamed BQ_INT
- removed net OTG: R11.1, U1.8 (OTG)
- net SCL renamed BQ_SCL
- net BQ_SCL: no longer IC1.7 (SCL)
- net SDA renamed BQ_SDA
- net BQ_SDA: no longer IC1.8 (SDA)
- new net: C46.1, D8.3 (K), U14.2 (IN)
- new net FG_SCL: IC1.7 (SCL)
- new net FG_SDA: IC1.8 (SDA)
Other:
- note added: "1160100 3.7V 10000mAh"
- note removed: "906090 3.7V 6000mAh"
- note removed: "connect with menu button"
- moved on the sheet: C10, C11, C12, C14, C16, C19, J2

Commit message: all
Connections:
- net +3V3 is gone; now on net +3V_CHRG: R10.1, R11.1
- net BAT+ renamed Fuel_G
Changed lines of the file:
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@@
 	)
 	(junction
-		(at 259.08 73.66)
-		(diameter 0)
-		(color 0 0 0 0)
-	)
-	(junction
 		(at 242.57 58.42)
 		(diameter 0)
@@
 	(wire
 		(pts
+			(xy 142.24 53.34) (xy 142.24 55.88)
+		)
+		(stroke
+			(width 0)
+			(type default)
+		)
+	)
+	(wire
+		(pts
 			(xy 113.03 149.86) (xy 120.65 149.86)
 		)
@@
 	(wire
 		(pts
-			(xy 142.24 54.61) (xy 142.24 55.88)
-		)
-		(stroke
-			(width 0)
-			(type default)
-		)
-	)
-	(wire
-		(pts
 			(xy 81.28 147.32) (xy 81.28 154.94)
 		)
@@
 	(wire
 		(pts
-			(xy 177.8 142.24) (xy 182.88 142.24)
-		)
-		(stroke
-			(width 0)
-			(type default)
-		)
-	)
-	(wire
-		(pts
 			(xy 212.09 107.95) (xy 212.09 121.92)
 		)
@@
 	(wire
 		(pts
+			(xy 175.26 142.24) (xy 182.88 142.24)
+		)
+		(stroke
+			(width 0)
+			(type default)
+		)
+	)
+	(wire
+		(pts
 			(xy 62.23 71.12) (xy 66.04 71.12)
 		)
@@
 	(wire
 		(pts
-			(xy 259.08 73.66) (xy 259.08 71.12)
+			(xy 259.08 71.12) (xy 259.08 77.47)
 		)
 		(stroke
@@
 	(wire
 		(pts
-			(xy 259.08 73.66) (xy 261.62 73.66)
-		)
-		(stroke
-			(width 0)
-			(type default)
-		)
-	)
-	(wire
-		(pts
 			(xy 199.39 105.41) (xy 212.09 105.41)
 		)
@@
 	(wire
 		(pts
-			(xy 259.08 77.47) (xy 259.08 73.66)
-		)
-		(stroke
-			(width 0)
-			(type default)
-		)
-	)
-	(wire
-		(pts
 			(xy 74.93 57.15) (xy 80.01 57.15)
 		)
@@
 		)
 	)
+	(label "Fuel_G"
+		(at 175.26 142.24 180)
+		(effects
+			(font
+				(size 1.27 1.27)
+			)
+			(justify right bottom)
+		)
+	)
 	(label "USB_D-"
 		(at 78.74 66.04 180)
@@
 		)
 	)
-	(hierarchical_label "BAT+"
-		(shape input)
-		(at 261.62 73.66 0)
-		(effects
-			(font
-				(size 1.27 1.27)
-			)
-			(justify left)
-		)
-	)
 	(hierarchical_label "BQ_SCL"
 		(shape input)
@@
 		)
 	)
-	(hierarchical_label "BAT+"
-		(shape input)
-		(at 177.8 142.24 180)
-		(effects
-			(font
-				(size 1.27 1.27)
-			)
-			(justify right)
-		)
-	)
 	(hierarchical_label "FG_SCL"
 		(shape input)
@@
 	)
 	(symbol
-		(lib_id "power:+3V3")
-		(at 133.35 142.24 0)
-		(unit 1)
-		(exclude_from_sim no)
-		(in_bom yes)
-		(on_board yes)
-		(dnp no)
-		(property "Reference" "#PWR068"
-			(at 133.35 146.05 0)
-			(effects
-				(font
-					(size 1.27 1.27)
-				)
-				(hide yes)
-			)
-		)
-		(property "Value" "+3V3"
-			(at 133.35 138.43 0)
-			(effects
-				(font
-					(size 1.27 1.27)
-				)
-			)
-		)
-		(property "Footprint" ""
-			(at 133.35 142.24 0)
-			(effects
-				(font
-					(size 1.27 1.27)
-				)
-				(hide yes)
-			)
-		)
-		(property "Datasheet" ""
-			(at 133.35 142.24 0)
-			(effects
-				(font
-					(size 1.27 1.27)
-				)
-				(hide yes)
-			)
-		)
-		(property "Description" "Power symbol creates a global label with name \"+3V3\""
-			(at 133.35 142.24 0)
-			(effects
-				(font
-					(size 1.27 1.27)
-				)
-				(hide yes)
-			)
-		)
-		(pin "1"
-		)
-		(instances
-			(project "KB-01"
-				(path "/e6144e29-1dc4-45a8-93e7-988a20131b94/8a655b9b-8849-4070-bc16-b30b70cfa2c5"
-					(reference "#PWR068")
-					(unit 1)
-				)
-			)
-		)
-	)
-	(symbol
 		(lib_id "power:GND")
 		(at 100.33 58.42 0)
@@
 	)
 	(symbol
+		(lib_id "power:+3V3")
+		(at 133.35 142.24 0)
+		(unit 1)
+		(exclude_from_sim no)
+		(in_bom yes)
+		(on_board yes)
+		(dnp no)
+		(property "Reference" "#PWR059"
+			(at 133.35 146.05 0)
+			(effects
+				(font
+					(size 1.27 1.27)
+				)
+				(hide yes)
+			)
+		)
+		(property "Value" "+3V_CHRG"
+			(at 133.35 138.176 0)
+			(effects
+				(font
+					(size 1.27 1.27)
+				)
+			)
+		)
+		(property "Footprint" ""
+			(at 133.35 142.24 0)
+			(effects
+				(font
+					(size 1.27 1.27)
+				)
+				(hide yes)
+			)
+		)
+		(property "Datasheet" ""
+			(at 133.35 142.24 0)
+			(effects
+				(font
+					(size 1.27 1.27)
+				)
+				(hide yes)
+			)
+		)
+		(property "Description" "Power symbol creates a global label with name \"+3V3\""
+			(at 133.35 142.24 0)
+			(effects
+				(font
+					(size 1.27 1.27)
+				)
+				(hide yes)
+			)
+		)
+		(pin "1"
+		)
+		(instances
+			(project "KB-01"
+				(path "/e6144e29-1dc4-45a8-93e7-988a20131b94/8a655b9b-8849-4070-bc16-b30b70cfa2c5"
+					(reference "#PWR059")
+					(unit 1)
+				)
+			)
+		)
+	)
+	(symbol
 		(lib_id "Device:C")
 		(at 196.85 143.51 0)
@@
 	)
 	(symbol
+		(lib_id "power:+3V3")
+		(at 142.24 53.34 0)
+		(unit 1)
+		(exclude_from_sim no)
+		(in_bom yes)
+		(on_board yes)
+		(dnp no)
+		(property "Reference" "#PWR068"
+			(at 142.24 57.15 0)
+			(effects
+				(font
+					(size 1.27 1.27)
+				)
+				(hide yes)
+			)
+		)
+		(property "Value" "+3V_CHRG"
+			(at 142.24 49.276 0)
+			(effects
+				(font
+					(size 1.27 1.27)
+				)
+			)
+		)
+		(property "Footprint" ""
+			(at 142.24 53.34 0)
+			(effects
+				(font
+					(size 1.27 1.27)
+				)
+				(hide yes)
+			)
+		)
+		(property "Datasheet" ""
+			(at 142.24 53.34 0)
+			(effects
+				(font
+					(size 1.27 1.27)
+				)
+				(hide yes)
+			)
+		)
+		(property "Description" "Power symbol creates a global label with name \"+3V3\""
+			(at 142.24 53.34 0)
+			(effects
+				(font
+					(size 1.27 1.27)
+				)
+				(hide yes)
+			)
+		)
+		(pin "1"
+		)
+		(instances
+			(project "KB-01"
+				(path "/e6144e29-1dc4-45a8-93e7-988a20131b94/8a655b9b-8849-4070-bc16-b30b70cfa2c5"
+					(reference "#PWR068")
+					(unit 1)
+				)
+			)
+		)
+	)
+	(symbol
 		(lib_id "power:PWR_FLAG")
 		(at 68.58 46.99 0)
@@
 					(unit 1)
 				)
-			)
-		)
-	)
-	(symbol
-		(lib_id "power:+3V3")
-		(at 142.24 54.61 0)
-		(unit 1)
-		(exclude_from_sim no)
-		(in_bom yes)
-		(on_board yes)
-		(dnp no)
-		(property "Reference" "#PWR023"
-			(at 142.24 58.42 0)
-			(effects
-				(font
-					(size 1.27 1.27)
-				)
-				(hide yes)
-			)
-		)
-		(property "Value" "+3V3"
-			(at 142.24 50.8 0)
-			(effects
-				(font
-					(size 1.27 1.27)
-				)
-			)
-		)
-		(property "Footprint" ""
-			(at 142.24 54.61 0)
-			(effects
-				(font
-					(size 1.27 1.27)
-				)
-				(hide yes)
-			)
-		)
-		(property "Datasheet" ""
-			(at 142.24 54.61 0)
-			(effects
-				(font
-					(size 1.27 1.27)
-				)
-				(hide yes)
-			)
-		)
-		(property "Description" "Power symbol creates a global label with name \"+3V3\""
-			(at 142.24 54.61 0)
-			(effects
-				(font
-					(size 1.27 1.27)
-				)
-				(hide yes)
-			)
-		)
-		(pin "1"
-		)
-		(instances
-			(project "KB-01"
-				(path "/e6144e29-1dc4-45a8-93e7-988a20131b94/8a655b9b-8849-4070-bc16-b30b70cfa2c5"
-					(reference "#PWR023")
-					(unit 1)
-				)

Commit message: all
Parts:
- C16, C18, C19: mouser (none) -> 603-CC603KRX7R8BB104
- C47: value 0.1uF -> 0.1uF 10V; mouser (none) -> 963-LMF107B7104KAHT
- IC1: mouser (none) -> 700-MAX17048G+T10
- R10, R11, R12, R13, R14: value 10K -> 10k; mouser (none) -> 71-CRCW060310K0FKEE
- R9: mouser (none) -> 71-CRCW060310K0FKEE
- U6: mouser (none) -> 595-TS3USB30ERSWR
Other:
- note added: "10K if no NTC connected, Change R13 and R14 to 5k and 30k respectively if theres NTC"
- note added: "Battery Connection"
- note added: "To boost converter"
- note removed: "to boost converter"

Commit message: all
Parts:
- SW2: footprint (none) -> Button_Switch_SMD:SW_Push_1P1T_NO_CK_KSC6xxJ
Changed lines of the file:
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@@
 			)
 		)
-		(property "Footprint" ""
+		(property "Footprint" "Button_Switch_SMD:SW_Push_1P1T_NO_CK_KSC6xxJ"
 			(at 120.65 95.25 0)
 			(hide yes)

Commit message: all
Parts:
- C10: mouser (none) -> 80-C0603C473K3R
- C11, C12, C14, C15: mouser (none) -> 81-GRM188R61E106KA3D
- C13: mouser (none) -> 81-GRM188Z71C475KE1D
- C17, C46: mouser (none) -> 187-CL10B105KA8NNNC
- C45: value 4.7uF -> 4.7uF 16V; mouser (none) -> 81-GRM188Z71C475KE1D
- D2: mouser (none) -> 859-LTST-C190KGKT
- D8: mouser (none) -> 726-BAT5405WH6327
- J2: footprint Connector_JST:JST_XH_B2B-XH-AM_1x02_P2.50mm_Vertical -> Connector_JST:JST_PH_B2B-PH-SM4-TB_1x02-1MP_P2.00mm_Vertical; mouser (none) -> 306-B2BPHSM4TBLFSN
- R5: mouser (none) -> 603-RC0603FR-072K21L
- R8: mouser (none) -> 708-RMCF0603FT133R
- SW2: mouser (none) -> 667-EVQP7B01P
- U14: mouser (none) -> 595-TLV70430DBVR
Changed lines of the file:
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@@
 			)
 		)
+		(property "mouser" "603-RC0603FR-072K21L"
+			(at 219.71 27.94 90)
+			(hide yes)
+			(show_name no)
+			(do_not_autoplace no)
+			(effects
+				(font
+					(size 1.27 1.27)
+				)
+			)
+		)
 		(pin "2"
 		)
@@
 			)
 		)
-		(property "Value" "4.7uF"
+		(property "Value" "4.7uF 16V"
 			(at 255.27 146.0499 0)
 			(show_name no)
@@
 			)
 		)
+		(property "mouser" "81-GRM188Z71C475KE1D"
+			(at 251.46 144.78 0)
+			(hide yes)
+			(show_name no)
+			(do_not_autoplace no)
+			(effects
+				(font
+					(size 1.27 1.27)
+				)
+			)
+		)
 		(pin "2"
 		)
@@
 			)
 		)
+		(property "mouser" "595-TLV70430DBVR"
+			(at 223.52 144.78 0)
+			(hide yes)
+			(show_name no)
+			(do_not_autoplace no)
+			(effects
+				(font
+					(size 1.27 1.27)
+				)
+			)
+		)
 		(pin "1"
 		)
@@
 			)
 		)
+		(property "mouser" "187-CL10B105KA8NNNC"
+			(at 196.85 143.51 0)
+			(hide yes)
+			(show_name no)
+			(do_not_autoplace no)
+			(effects
+				(font
+					(size 1.27 1.27)
+				)
+			)
+		)
 		(pin "2"
 		)
@@
 			)
 		)
+		(property "mouser" "81-GRM188Z71C475KE1D"
+			(at 203.2 80.01 0)
+			(hide yes)
+			(show_name no)
+			(do_not_autoplace no)
+			(effects
+				(font
+					(size 1.27 1.27)
+				)
+			)
+		)
 		(pin "2"
 		)
@@
 			)
 		)
+		(property "mouser" "667-EVQP7B01P"
+			(at 125.73 95.25 90)
+			(hide yes)
+			(show_name no)
+			(do_not_autoplace no)
+			(effects
+				(font
+					(size 1.27 1.27)
+				)
+			)
+		)
 		(pin "1"
 		)
@@
 			)
 		)
+		(property "mouser" "187-CL10B105KA8NNNC"
+			(at 153.67 49.53 0)
+			(hide yes)
+			(show_name no)
+			(do_not_autoplace no)
+			(effects
+				(font
+					(size 1.27 1.27)
+				)
+			)
+		)
 		(pin "2"
 		)
@@
 			)
 		)
+		(property "mouser" "81-GRM188R61E106KA3D"
+			(at 250.19 63.5 0)
+			(hide yes)
+			(show_name no)
+			(do_not_autoplace no)
+			(effects
+				(font
+					(size 1.27 1.27)
+				)
+			)
+		)
 		(pin "2"
 		)
@@
 			)
 		)
+		(property "mouser" "81-GRM188R61E106KA3D"
+			(at 234.95 63.5 0)
+			(hide yes)
+			(show_name no)
+			(do_not_autoplace no)
+			(effects
+				(font
+					(size 1.27 1.27)
+				)
+			)
+		)
 		(pin "2"
 		)
@@
 			)
 		)
+		(property "mouser" "708-RMCF0603FT133R"
+			(at 166.37 87.63 0)
+			(hide yes)
+			(show_name no)
+			(do_not_autoplace no)
+			(effects
+				(font
+					(size 1.27 1.27)
+				)
+			)
+		)
 		(pin "2"
 		)
@@
 			)
 		)
+		(property "mouser" "81-GRM188R61E106KA3D"
+			(at 209.55 48.26 0)
+			(hide yes)
+			(show_name no)
+			(do_not_autoplace no)
+			(effects
+				(font
+					(size 1.27 1.27)
+				)
+			)
+		)
 		(pin "2"
 		)
@@
 			)
 		)
+		(property "mouser" "81-GRM188R61E106KA3D"
+			(at 227.33 78.74 0)
+			(hide yes)
+			(show_name no)
+			(do_not_autoplace no)
+			(effects
+				(font
+					(size 1.27 1.27)
+				)
+			)
+		)
 		(pin "2"
 		)
@@
 			)
 		)
+		(property "mouser" "726-BAT5405WH6327 "
+			(at 187.96 139.7 0)
+			(hide yes)
+			(show_name no)
+			(do_not_autoplace no)
+			(effects
+				(font
+					(size 1.27 1.27)
+				)
+			)
+		)
 		(pin "2"
 		)
@@
 			)
 		)
+		(property "mouser" "859-LTST-C190KGKT"
+			(at 210.82 27.94 0)
+			(hide yes)
+			(show_name no)
+			(do_not_autoplace no)
+			(effects
+				(font
+					(size 1.27 1.27)
+				)
+			)
+		)
 		(pin "2"
 		)
@@
 			)
 		)
+		(property "mouser" "80-C0603C473K3R"
+			(at 212.09 63.5 0)
+			(hide yes)
+			(show_name no)
+			(do_not_autoplace no)
+			(effects
+				(font
+					(size 1.27 1.27)
+				)
+			)
+		)
 		(pin "2"
 		)
@@
 			)
 		)
-		(property "Footprint" "Connector_JST:JST_XH_B2B-XH-AM_1x02_P2.50mm_Vertical"
+		(property "Footprint" "Connector_JST:JST_PH_B2B-PH-SM4-TB_1x02-1MP_P2.00mm_Vertical"
 			(at 264.16 77.47 0)
 			(hide yes)
@@
 			(at 264.16 77.47 0)
 			(hide yes)
+			(show_name no)
+			(do_not_autoplace no)
+			(effects
+				(font
+					(size 1.27 1.27)
+				)
+			)
+		)
+		(property "mouser" "306-B2BPHSM4TBLFSN"
+			(at 264.16 77.47 0)
+			(hide yes)

Commit message: all
Parts:
- J8: footprint (none) -> Connector_Wire:SolderWirePad_1x01_SMD_1x2mm; mouser (none) -> n/a
Changed lines of the file:
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@@
 			)
 		)
-		(property "Footprint" ""
+		(property "Footprint" "Connector_Wire:SolderWirePad_1x01_SMD_1x2mm"
 			(at 217.17 105.41 0)
 			(hide yes)
@@
 			(at 217.17 105.41 0)
 			(hide yes)
+			(show_name no)
+			(do_not_autoplace no)
+			(effects
+				(font
+					(size 1.27 1.27)
+				)
+			)
+		)
+		(property "mouser" "n/a"
+			(at 217.17 105.41 0)
+			(hide yes)
