File: KB-01_kicad/KB-01/battery_charger.kicad_sch (KiCad schematic)
At the start: 37 parts, among them IC1 MAX17048G+T10, J12 Conn_01x01_Socket, J3 USB_C_Receptacle_USB2.0_14P, J4 Conn_01x02_MountingPin, J5 Conn_01x01_Socket, SW2 Power button, U1 BQ25895, U2 TS3USB30ERSWR, U3 TLV70430DBVR

Commit message: all
Parts:
- SW2: footprint Button_Switch_SMD:SW_Push_1P1T_NO_CK_KSC6xxJ -> Button_Switch_SMD:SW_SPST_EVQP7A; mouser 667-EVQP7B01P -> 667-EVQP7A01P
Connections:
- net GND: now also U3.4 (NC), U3.5 (NC)
- no-connect marks 2 -> 0
Other:
- note added: "MUX come with ESD protection"
Changed lines of the file:
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@@
 		)
 	)
+	(text "MUX come with ESD protection"
+		(exclude_from_sim no)
+		(at 96.012 42.672 0)
+		(effects
+			(font
+				(size 1.27 1.27)
+			)
+		)
+	)
 	(text "MAX17048 Fuel Gauge"
 		(exclude_from_sim no)
@@
 	)
 	(junction
+		(at 205.74 149.86)
+		(diameter 0)
+		(color 0 0 0 0)
+	)
+	(junction
 		(at 39.37 97.79)
 		(diameter 0)
@@
 	)
 	(junction
+		(at 196.85 149.86)
+		(diameter 0)
+		(color 0 0 0 0)
+	)
+	(junction
 		(at 153.67 45.72)
 		(diameter 0)
@@
 		(color 0 0 0 0)
 	)
-	(no_connect
-		(at 205.74 149.86)
-	)
-	(no_connect
-		(at 205.74 147.32)
-	)
 	(wire
 		(pts
@@
 	(wire
 		(pts
+			(xy 196.85 149.86) (xy 205.74 149.86)
+		)
+		(stroke
+			(width 0)
+			(type default)
+		)
+	)
+	(wire
+		(pts
 			(xy 142.24 53.34) (xy 142.24 55.88)
 		)
@@
 	(wire
 		(pts
+			(xy 205.74 147.32) (xy 205.74 149.86)
+		)
+		(stroke
+			(width 0)
+			(type default)
+		)
+	)
+	(wire
+		(pts
 			(xy 250.19 58.42) (xy 262.89 58.42)
 		)
@@
 	(wire
 		(pts
-			(xy 196.85 147.32) (xy 196.85 152.4)
+			(xy 196.85 147.32) (xy 196.85 149.86)
 		)
 		(stroke
@@
 	(wire
 		(pts
+			(xy 196.85 149.86) (xy 196.85 152.4)
+		)
+		(stroke
+			(width 0)
+			(type default)
+		)
+	)
+	(wire
+		(pts
 			(xy 125.73 100.33) (xy 125.73 106.68)
 		)
@@
 			)
 		)
-		(property "Footprint" "Button_Switch_SMD:SW_Push_1P1T_NO_CK_KSC6xxJ"
+		(property "Footprint" "Button_Switch_SMD:SW_SPST_EVQP7A"
 			(at 120.65 95.25 0)
 			(hide yes)
@@
 			)
 		)
-		(property "mouser" "667-EVQP7B01P"
+		(property "mouser" "667-EVQP7A01P"
 			(at 125.73 95.25 90)
 			(hide yes)
