File: KB-01_kicad/KB-01/gnss.kicad_sch (KiCad schematic)
At the start: 1 part, among them U3 L89_2.0

Commit message: all
Signed-off-by: syauqi-alias <syauqi_nur@yahoo.com>
Parts:
- removed U3: L89_2.0, L89_2.0:XCVR_L89_2.0, symbol L89_2.0:L89_2.0
- added C28, C29: 1uF, Capacitor_SMD:C_0603_1608Metric_Pad1.08x0.95mm_HandSolder, symbol Device:C
- added C30: 10nF, Capacitor_SMD:C_0603_1608Metric_Pad1.08x0.95mm_HandSolder, symbol Device:C
- added C31, C32: 56pF, Capacitor_SMD:C_0603_1608Metric_Pad1.08x0.95mm_HandSolder, symbol Device:C
- added L4: 27nH, Inductor_SMD:L_0603_1608Metric_Pad1.05x0.95mm_HandSolder, symbol Device:L
- added U3: TESEO-LIV3F, LCC-18_9P7X10P1_STM, symbol Teseo-LIV3F:TESEO-LIV3F
- added U7: TLV70033_SOT353, Package_TO_SOT_SMD:SOT-353_SC-70-5, symbol Regulator_Linear:TLV70033_SOT353
- added U8: MAX2659ELT+T, 21-0147-L611+2_MXM, symbol MAX2659ELT+T:MAX2659ELT+T
Connections:
- new net: C31.1, L4.2, U3.7 (VCC_IO), U3.8 (VCC)
- new net +5V: C29.1, U7.1 (IN)
- new net 3.3V_GNSS: C28.1, C30.1, L4.1, U7.5 (OUT)
- new net GND: C28.2, C29.2, C30.2, C31.2, C32.2, U7.2 (GND)
- new net GNSS_PSU_EN: U7.3 (EN)
- new net VCC_RF: C32.1, U3.14 (VCC_RF)
Other:
- note added: "960-FXP611.07.0092C"

Commit message: hi
Parts:
- added C33: 470pF, Capacitor_SMD:C_0402_1005Metric_Pad0.74x0.62mm_HandSolder, symbol Device:C
- added C34: 120pF, Capacitor_SMD:C_0402_1005Metric_Pad0.74x0.62mm_HandSolder, symbol Device:C
- added FL1: B39162B4327P810, B39162B4327P810:FIL_B39162B4327P810, symbol B39162B4327P810:B39162B4327P810
- added J5: Conn_Coaxial, Connector_Coaxial:U.FL_Hirose_U.FL-R-SMT-1_Vertical, symbol Connector:Conn_Coaxial
- added L5: 6.8nH, Inductor_SMD:L_0402_1005Metric_Pad0.77x0.64mm_HandSolder, symbol Device:L
- added R17: R, Resistor_SMD:R_0402_1005Metric_Pad0.72x0.64mm_HandSolder, symbol Device:R
- U8: footprint 21-0147-L611+2_MXM -> footprints:21-0147-L611&plus_2_MXM
Connections:
- net 3.3V_GNSS: no longer C28.1, U7.5 (OUT)
- net GND: now also U3.1 (GND), U3.10 (GND_RF), U3.12 (GND_RF), U8.1 (GND), U8.2 (GND), FL1.2 (GND), FL1.3 (GND__1), FL1.5 (GND__2), J5.2 (Ext)
- net VCC_RF: now also C28.1, U7.5 (OUT), U8.4 (VCC)
- net RF_IN: now reaches U3.11 (RF_IN)
- net RF_IN: now also C34.2
- net RF_EN: now reaches U3.13 (ANT_OFF)
- net RF_EN: now also U8.5 (*SHDN), R17.1
- net GNSS_TX: now reaches U3.2 (TX)
- net GNSS_RX: now reaches U3.3 (RX)
- net at U8.3 (RFIN): now also L5.2
- net at U8.6 (RFOUT): now also FL1.1 (INPUT)
- new net: C33.1, J5.1 (In)
- new net: C33.2, L5.1
- new net: C34.1, FL1.4 (OUTPUT)
Other:
- moved on the sheet: C28, C29, C30, C31, C32, L4, U3, U7, U8

Commit message: update gnss
Parts:
- added D3: LED, LED_SMD:LED_0603_1608Metric_Pad1.05x0.95mm_HandSolder, symbol Device:LED
- added D4: D_Schottky, symbol Device:D_Schottky
- added Q1: MMBT3904, Package_TO_SOT_SMD:SOT-23, symbol Transistor_BJT:MMBT3904
- added R18: 330, Resistor_SMD:R_0402_1005Metric_Pad0.72x0.64mm_HandSolder, symbol Device:R
- R17: value R -> 10k
Connections:
- net 3.3V_GNSS: now also C28.1, U7.5 (OUT), D4.2 (A), R18.1
- net GND: now also R17.2, Q1.2 (E)
- net VCC_RF: no longer C28.1, U7.5 (OUT)
- net GNSS_SDA: now reaches U3.16 (SDA)
- net GNSS_SCL: now reaches U3.17 (SCL)
- net GNSS_PPS: now reaches U3.4 (PPS)
- net GNSS_PPS: now also Q1.1 (B)
- net GNSS_WAKEUP: now reaches U3.5 (WAKE_UP)
- net GNSS_Vbatt: now reaches U3.6 (VBATT)
- net GNSS_Vbatt: now also D4.1 (K)
- net GNSS_RSTn: now reaches U3.9 (SYS_RSTN)
- new net: D3.2 (A), R18.2
- new net: D3.1 (K), Q1.3 (C)
Other:
- note added: "RF Front-end"
- moved on the sheet: C30, C31, C32, C33, C34, FL1, J5, L4, L5, R17, U3, U8

Commit message: up
Parts:
- added D5: SM15T36CA, Diode_SMD:D_SMA, symbol Diode:SM15T36CA
Connections:
- net GND: now also D5.2 (A2)
- net at C33.1, J5.1 (In): now also D5.1 (A1)
Changed lines of the file:
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@@
 	)
 	(junction
+		(at 66.04 149.86)
+		(diameter 0)
+		(color 0 0 0 0)
+	)
+	(junction
 		(at 111.76 85.09)
 		(diameter 0)
@@
 	)
 	(junction
+		(at 69.85 137.16)
+		(diameter 0)
+		(color 0 0 0 0)
+	)
+	(junction
 		(at 215.9 142.24)
 		(diameter 0)
@@
 	(wire
 		(pts
-			(xy 68.58 137.16) (xy 76.2 137.16)
+			(xy 68.58 137.16) (xy 69.85 137.16)
 		)
 		(stroke
@@
 	(wire
 		(pts
+			(xy 69.85 149.86) (xy 66.04 149.86)
+		)
+		(stroke
+			(width 0)
+			(type default)
+		)
+	)
+	(wire
+		(pts
 			(xy 107.95 77.47) (xy 113.03 77.47)
 		)
@@
 	(wire
 		(pts
-			(xy 63.5 142.24) (xy 63.5 146.05)
+			(xy 66.04 149.86) (xy 66.04 153.67)
 		)
 		(stroke
@@
 	(wire
 		(pts
+			(xy 66.04 149.86) (xy 63.5 149.86)
+		)
+		(stroke
+			(width 0)
+			(type default)
+		)
+	)
+	(wire
+		(pts
 			(xy 215.9 139.7) (xy 215.9 137.16)
 		)
@@
 	(wire
 		(pts
+			(xy 69.85 137.16) (xy 69.85 139.7)
+		)
+		(stroke
+			(width 0)
+			(type default)
+		)
+	)
+	(wire
+		(pts
 			(xy 168.91 72.39) (xy 172.72 72.39)
 		)
@@
 	(wire
 		(pts
+			(xy 69.85 137.16) (xy 76.2 137.16)
+		)
+		(stroke
+			(width 0)
+			(type default)
+		)
+	)
+	(wire
+		(pts
 			(xy 182.88 92.71) (xy 182.88 80.01)
 		)
@@
 	(wire
 		(pts
+			(xy 63.5 149.86) (xy 63.5 142.24)
+		)
+		(stroke
+			(width 0)
+			(type default)
+		)
+	)
+	(wire
+		(pts
 			(xy 256.54 45.72) (xy 256.54 40.64)
 		)
@@
 	(wire
 		(pts
+			(xy 69.85 147.32) (xy 69.85 149.86)
+		)
+		(stroke
+			(width 0)
+			(type default)
+		)
+	)
+	(wire
+		(pts
 			(xy 172.72 95.25) (xy 172.72 93.98)
 		)
@@
 	)
 	(symbol
+		(lib_id "Diode:SM15T36CA")
+		(at 69.85 143.51 270)
+		(unit 1)
+		(exclude_from_sim no)
+		(in_bom yes)
+		(on_board yes)
+		(dnp no)
+		(fields_autoplaced yes)
+		(property "Reference" "D5"
+			(at 72.39 142.2399 90)
+			(effects
+				(font
+					(size 1.27 1.27)
+				)
+				(justify left)
+			)
+		)
+		(property "Value" "SM15T36CA"
+			(at 72.39 144.7799 90)
+			(effects
+				(font
+					(size 1.27 1.27)
+				)
+				(justify left)
+			)
+		)
+		(property "Footprint" "Diode_SMD:D_SMA"
+			(at 61.214 144.018 0)
+			(effects
+				(font
+					(size 1.27 1.27)
+				)
+				(hide yes)
+			)
+		)
+		(property "Datasheet" "https://www.st.com/resource/en/datasheet/sm15t36a.pdf"
+			(at 63.246 143.51 0)
+			(effects
+				(font
+					(size 1.27 1.27)
+				)
+				(hide yes)
+			)
+		)
+		(property "Description" "1500W (10/1000 μs) Bidirectional TVS Diode, VRM = 30.8V (IRM = 0.2 μA at 25°C), VBR = 34.2 ... 37.8V, 'BEV' marking, SMC"
+			(at 65.278 143.51 0)
+			(effects
+				(font
+					(size 1.27 1.27)
+				)
+				(hide yes)
+			)
+		)
+		(pin "1"
+		)
+		(pin "2"
+		)
+		(instances
+			(project ""
+				(path "/e6144e29-1dc4-45a8-93e7-988a20131b94/0be82c74-fb54-4d7f-bce1-28060d710cf9"
+					(reference "D5")
+					(unit 1)
+				)
+			)
+		)
+	)
+	(symbol
 		(lib_id "power:GND")
 		(at 93.98 95.25 0)
@@
 	(symbol
 		(lib_id "power:GND")
-		(at 63.5 146.05 0)
+		(at 66.04 153.67 0)
 		(unit 1)
 		(exclude_from_sim no)
@@
 		(fields_autoplaced yes)
 		(property "Reference" "#PWR036"
-			(at 63.5 152.4 0)
+			(at 66.04 160.02 0)
 			(effects
 				(font
@@
 		)
 		(property "Value" "GND"
-			(at 63.5 151.13 0)
+			(at 66.04 158.75 0)
 			(effects
 				(font
@@
 		)
 		(property "Footprint" ""
-			(at 63.5 146.05 0)
+			(at 66.04 153.67 0)
 			(effects
 				(font
@@
 		)
 		(property "Datasheet" ""
-			(at 63.5 146.05 0)
+			(at 66.04 153.67 0)
 			(effects
 				(font
@@
 		)
 		(property "Description" "Power symbol creates a global label with name \"GND\" , ground"
-			(at 63.5 146.05 0)
+			(at 66.04 153.67 0)
 			(effects
 				(font

Commit message: up
Parts:
- removed D4: D_Schottky, symbol Device:D_Schottky
- added C1: 56pF, Capacitor_SMD:C_0402_1005Metric_Pad0.74x0.62mm_HandSolder, symbol Device:C
- added C43: 10uF, Capacitor_SMD:C_0603_1608Metric_Pad1.08x0.95mm_HandSolder, symbol Device:C
- added C44: 100nF, Capacitor_SMD:C_0603_1608Metric_Pad1.08x0.95mm_HandSolder, symbol Device:C
- added D6: SM15T36CA, Diode_SMD:D_SMA, symbol Diode:SM15T36CA
- added J1: Conn_Coaxial, Connector_Coaxial:U.FL_Hirose_U.FL-R-SMT-1_Vertical, symbol Connector:Conn_Coaxial
- added U1: TESEO-LIV4F, TESEO-LIV4F:XCVR_TESEO-LIV4F, symbol TESEO-LIV4F:TESEO-LIV4F
- C30, C31, C32, C33, C34, D5, FL1, J5, L4, L5, R17, U3, U8: now not fitted; now left out of the parts list
- U7: value TLV70033_SOT353 -> TLV773_SOT353
Connections:
- net 3.3V_GNSS: now also C43.1, C44.1, U1.6 (VBAT), U1.8 (VCC)
- net GND: now also C43.2, C44.2, D6.2 (A2), J1.2 (Ext), U1.1 (GND), U1.10 (GND_RF), U1.12 (GND_RF); no longer U3.10 (GND_RF), U3.12 (GND_RF)
- net GNSS_PPS: now also U1.4 (PPS)
- net GNSS_RSTn: now also U1.9 (~{RESET})
- net GNSS_RX: now also U1.3 (UART-RX)
- net GNSS_SCL: now also U1.17 (I2C_SCL)
- net GNSS_SDA: now also U1.16 (I2C_SDA)
- net GNSS_TX: now also U1.2 (UART-TX)
- net GNSS_WAKEUP: now also U1.5 (WAKEUP)
- net +5V renamed +5v
- new net: U3.10 (GND_RF), U3.12 (GND_RF)
- new net: C1.1, D6.1 (A1), J1.1 (In)
- new net: C1.2, U1.11 (RF_IN)
- new net: U1.13 (RESERVED), U1.15 (RESERVED), U1.7 (RESERVED)
- no-connect marks 0 -> 2
Other:
- moved on the sheet: C28, C29

Commit message: all
Connections:
- net GNSS_SCL: no longer U1.17 (I2C_SCL)
- net GNSS_SDA: no longer U1.16 (I2C_SDA)
- no-connect marks 2 -> 4
Changed lines of the file:
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@@
+	)
+	(no_connect
+		(at 156.21 41.91)
 	)
 	(no_connect
@@
 		(at 115.57 36.83)
 	)
+	(no_connect
+		(at 156.21 39.37)
+	)
 	(wire
 		(pts
@@
 	(wire
 		(pts
-			(xy 156.21 39.37) (xy 161.29 39.37)
-		)
-		(stroke
-			(width 0)
-			(type default)
-		)
-	)
-	(wire
-		(pts
 			(xy 102.87 96.52) (xy 107.95 96.52)
 		)
@@
 		(pts
 			(xy 234.95 151.13) (xy 243.84 151.13)
-		)
-		(stroke
-			(width 0)
-			(type default)
-		)
-	)
-	(wire
-		(pts
-			(xy 156.21 41.91) (xy 161.29 41.91)
 		)
 		(stroke
@@
 		(effects
 			(font
-				(size 1.27 1.27)
-			)
-			(justify left)
-		)
-	)
-	(hierarchical_label "GNSS_SCL"
-		(shape input)
-		(at 161.29 39.37 0)
-		(effects
-			(font
-				(size 1.27 1.27)
-			)
-			(justify left)
-		)
-	)
-	(hierarchical_label "GNSS_SDA"
-		(shape input)
-		(at 161.29 41.91 0)
-		(effects
-			(font

Commit message: all
Parts:
- renumbered C1 to C51

Commit message: all
Parts:
- C43: value 10uF -> 10uF 6.3V; mouser (none) -> 81-GRM188R60J106ME47
- C44: value 100nF -> 100nF 6.3V; mouser (none) -> 581-KGM15AR70J104KT
- C51: value 56pF -> 56pF 50V; mouser (none) -> 81-GRM1555C1H560JA1J
- D6: mouser (none) -> 511-SM15T36CAY
- U11: renamed from U1; footprint TESEO-LIV4F:XCVR_TESEO-LIV4F -> TESEO-LIV4FTR:TESEOLIV4FTR; mouser (none) -> 511-TESEO-LIV4FTR
- renumbered J1 to J10
Other:
- note added: "Passive antenna"
