File: KB-01_kicad/KB-01/gnss.kicad_sch (KiCad schematic)
At the start: 25 parts, among them J10 Conn_Coaxial, J5 Conn_Coaxial, Q1 MMBT3904, U11 TESEO-LIV4F, U3 TESEO-LIV3F, U7 TLV773_SOT353, U8 MAX2659ELT+T

Commit message: all
Parts:
- C28, C29: value 1uF -> 1uF 16V; mouser (none) -> 187-CL10B105KO8NNNC
- D3: value LED -> LED Red; mouser (none) -> 755-SML-D12L8WT86
- Q1: mouser (none) -> 621-MMBT3904T-F
Changed lines of the file:
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@@
 			)
 		)
-		(property "Value" "1uF"
+		(property "Value" "1uF 16V"
 			(at 260.35 41.9099 0)
 			(show_name no)
@@
 			)
 		)
+		(property "mouser" "187-CL10B105KO8NNNC"
+			(at 256.54 40.64 0)
+			(hide yes)
+			(show_name no)
+			(do_not_autoplace no)
+			(effects
+				(font
+					(size 1.27 1.27)
+				)
+			)
+		)
 		(pin "1"
 		)
@@
 			)
 		)
-		(property "Value" "LED"
+		(property "Value" "LED Red"
 			(at 238.76 85.4074 90)
 			(show_name no)
@@
 			)
 		)
+		(property "mouser" "755-SML-D12L8WT86"
+			(at 234.95 82.55 90)
+			(hide yes)
+			(show_name no)
+			(do_not_autoplace no)
+			(effects
+				(font
+					(size 1.27 1.27)
+				)
+			)
+		)
 		(pin "1"
 		)
@@
 			)
 		)
+		(property "mouser" "621-MMBT3904T-F"
+			(at 232.41 93.98 0)
+			(hide yes)
+			(show_name no)
+			(do_not_autoplace no)
+			(effects
+				(font
+					(size 1.27 1.27)
+				)
+			)
+		)
 		(pin "1"
 		)
@@
 			)
 		)
-		(property "Value" "1uF"
+		(property "Value" "1uF 16V"
 			(at 234.95 41.9099 0)
 			(show_name no)
@@
 			)
 		)
+		(property "mouser" "187-CL10B105KO8NNNC"
+			(at 231.14 40.64 0)
+			(hide yes)
+			(show_name no)
+			(do_not_autoplace no)
+			(effects
+				(font
+					(size 1.27 1.27)
+				)
+			)
+		)
 		(pin "1"
 		)
@@
 		)
 	)
-	(embedded_fonts no)
 )

Commit message: all
Parts:
- added R1: 4.7k, Resistor_SMD:R_0603_1608Metric_Pad0.98x0.95mm_HandSolder, symbol Device:R
- added R31: 10k, Resistor_SMD:R_0603_1608Metric_Pad0.98x0.95mm_HandSolder, symbol Device:R
- J10: mouser (none) -> 798-U.FL-R-SMT-110
- R18: mouser (none) -> 754-RG1608P-331-BT5
Connections:
- net GND: now also R31.2
- net GNSS_PPS: now also R1.1; no longer Q1.1 (B)
- new net: Q1.1 (B), R1.2, R31.1

Commit message: all
Parts:
- R18: renamed from R1; mouser 652-CR0603FX-4701ELF -> 667-ERJ-3GEYJ472V
- R19: renamed from R31; mouser 71-CRCW060310K0FKECC -> 71-CRCW060310K0FKEE
- renumbered C44 to C24, C43 to C25, C29 to C26, C28 to C27, C51 to C28, C32 to C29, C34 to C32, D6 to D5, D3 to D6, D5 to D7, J10 to J6, J5 to J7, L4 to L3, L5 to L4, R18 to R17, R17 to R20, U7 to U5, U11 to U6, U3 to U7
Connections:
- net GND: now also U7.10 (GND_RF), U7.12 (GND_RF)

Commit message: all
Parts:
- added J15: Conn_Coaxial, Connector_Coaxial:SMA_Molex_73251-2120_EdgeMount_Horizontal, symbol Connector:Conn_Coaxial
- C28, J6: now not fitted
- D5: footprint Diode_SMD:D_SMA -> Diode_SMD:D_0201_0603Metric_Pad0.64x0.40mm_HandSolder; mouser 511-SM15T36CAY -> 511-ESDL031-1BF4
- R17: footprint Resistor_SMD:R_0402_1005Metric_Pad0.72x0.64mm_HandSolder -> Resistor_SMD:R_0603_1608Metric_Pad0.98x0.95mm_HandSolder
Connections:
- net GND: now also J15.2 (Ext)
- net at C28.1, D5.1 (A1), J6.1 (In): now also C28.2, U6.11 (RF_IN), J15.1 (In)
Other:
- note added: "Use SMA instead for helical antenna"
- moved on the sheet: D5
Changed lines of the file:
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@@
 		)
 	)
+	(text "Use SMA instead for helical antenna"
+		(exclude_from_sim no)
+		(at 62.484 31.496 0)
+		(effects
+			(font
+				(size 1.27 1.27)
+			)
+		)
+	)
 	(text "RF Front-end"
 		(exclude_from_sim no)
@@
 	)
 	(junction
+		(at 101.6 41.91)
+		(diameter 0)
+		(color 0 0 0 0)
+	)
+	(junction
 		(at 246.38 45.72)
 		(diameter 0)
@@
 	)
 	(junction
+		(at 80.01 46.99)
+		(diameter 0)
+		(color 0 0 0 0)
+	)
+	(junction
 		(at 78.74 156.21)
 		(diameter 0)
@@
 	(wire
 		(pts
+			(xy 101.6 46.99) (xy 101.6 41.91)
+		)
+		(stroke
+			(width 0)
+			(type default)
+		)
+	)
+	(wire
+		(pts
 			(xy 106.68 106.68) (xy 107.95 106.68)
 		)
@@
 	(wire
 		(pts
-			(xy 97.79 41.91) (xy 115.57 41.91)
+			(xy 97.79 41.91) (xy 101.6 41.91)
 		)
 		(stroke
@@
 	(wire
 		(pts
+			(xy 80.01 46.99) (xy 80.01 48.26)
+		)
+		(stroke
+			(width 0)
+			(type default)
+		)
+	)
+	(wire
+		(pts
 			(xy 74.93 41.91) (xy 80.01 41.91)
 		)
@@
 	(wire
 		(pts
+			(xy 53.34 34.29) (xy 80.01 34.29)
+		)
+		(stroke
+			(width 0)
+			(type default)
+		)
+	)
+	(wire
+		(pts
 			(xy 172.72 106.68) (xy 163.83 106.68)
 		)
@@
 	(wire
 		(pts
+			(xy 101.6 41.91) (xy 115.57 41.91)
+		)
+		(stroke
+			(width 0)
+			(type default)
+		)
+	)
+	(wire
+		(pts
 			(xy 231.14 45.72) (xy 231.14 44.45)
 		)
@@
 	(wire
 		(pts
-			(xy 80.01 53.34) (xy 80.01 58.42)
+			(xy 80.01 55.88) (xy 80.01 58.42)
 		)
 		(stroke
@@
 	(wire
 		(pts
+			(xy 80.01 46.99) (xy 101.6 46.99)
+		)
+		(stroke
+			(width 0)
+			(type default)
+		)
+	)
+	(wire
+		(pts
 			(xy 78.74 156.21) (xy 78.74 158.75)
 		)
@@
 	(wire
 		(pts
+			(xy 48.26 46.99) (xy 48.26 58.42)
+		)
+		(stroke
+			(width 0)
+			(type default)
+		)
+	)
+	(wire
+		(pts
 			(xy 165.1 33.02) (xy 177.8 33.02)
 		)
@@
 	(wire
 		(pts
+			(xy 53.34 41.91) (xy 53.34 34.29)
+		)
+		(stroke
+			(width 0)
+			(type default)
+		)
+	)
+	(wire
+		(pts
 			(xy 102.87 99.06) (xy 107.95 99.06)
 		)
@@
 	(wire
 		(pts
+			(xy 80.01 34.29) (xy 80.01 41.91)
+		)
+		(stroke
+			(width 0)
+			(type default)
+		)
+	)
+	(wire
+		(pts
 			(xy 177.8 116.84) (xy 177.8 104.14)
 		)
@@
 	(wire
 		(pts
-			(xy 80.01 41.91) (xy 80.01 45.72)
+			(xy 80.01 41.91) (xy 80.01 46.99)
 		)
 		(stroke
@@
 	(wire
 		(pts
+			(xy 48.26 58.42) (xy 69.85 58.42)
+		)
+		(stroke
+			(width 0)
+			(type default)
+		)
+	)
+	(wire
+		(pts
 			(xy 167.64 111.76) (xy 167.64 119.38)
 		)
@@
 			)
 		)
-		(property "Footprint" "Resistor_SMD:R_0402_1005Metric_Pad0.72x0.64mm_HandSolder"
+		(property "Footprint" "Resistor_SMD:R_0603_1608Metric_Pad0.98x0.95mm_HandSolder"
 			(at 233.172 72.39 90)
 			(hide yes)
@@
 	)
 	(symbol
+		(lib_id "Connector:Conn_Coaxial")
+		(at 48.26 41.91 0)
+		(mirror y)
+		(unit 1)
+		(body_style 1)
+		(exclude_from_sim no)
+		(in_bom yes)
+		(on_board yes)
+		(in_pos_files yes)
+		(dnp no)
+		(property "Reference" "J15"
+			(at 44.45 40.9331 0)
+			(show_name no)
+			(do_not_autoplace no)
+			(effects
+				(font
+					(size 1.27 1.27)
+				)
+				(justify left)
+			)
+		)
+		(property "Value" "Conn_Coaxial"
+			(at 44.45 43.4731 0)
+			(show_name no)
+			(do_not_autoplace no)
+			(effects
+				(font
+					(size 1.27 1.27)
+				)
+				(justify left)
+			)
+		)
+		(property "Footprint" "Connector_Coaxial:SMA_Molex_73251-2120_EdgeMount_Horizontal"
+			(at 48.26 41.91 0)
+			(hide yes)
+			(show_name no)
+			(do_not_autoplace no)
+			(effects
+				(font
+					(size 1.27 1.27)
+				)
+			)
+		)
+		(property "Datasheet" ""
+			(at 48.26 41.91 0)
+			(hide yes)
+			(show_name no)
+			(do_not_autoplace no)
+			(effects
+				(font
+					(size 1.27 1.27)
+				)
+			)
+		)
+		(property "Description" "coaxial connector (BNC, SMA, SMB, SMC, Cinch/RCA, LEMO, ...)"
+			(at 48.26 41.91 0)
+			(hide yes)
+			(show_name no)
+			(do_not_autoplace no)
+			(effects
+				(font
+					(size 1.27 1.27)
+				)
+			)
+		)
+		(property "SNAPEDA_PN" ""
+			(at 48.26 41.91 0)
+			(hide yes)
+			(show_name no)
+			(do_not_autoplace no)
+			(effects
+				(font
+					(size 1.27 1.27)
+				)
+			)
+		)
+		(property "mouser" "538-73251-2120"
+			(at 48.26 41.91 0)
+			(hide yes)
+			(show_name no)
+			(do_not_autoplace no)
+			(effects
+				(font
+					(size 1.27 1.27)
+				)
+			)
+		)
+		(pin "2"
+		)
+		(pin "1"
+		)
+		(instances
+			(project "KB-01"
+				(path "/e6144e29-1dc4-45a8-93e7-988a20131b94/0be82c74-fb54-4d7f-bce1-28060d710cf9"
+					(reference "J15")
+					(unit 1)
+				)
+			)
+		)
+	)
+	(symbol
 		(lib_id "power:GND")
 		(at 69.85 63.5 0)
@@
 	(symbol
 		(lib_id "Diode:SM15T36CA")
-		(at 80.01 49.53 270)
+		(at 80.01 52.07 270)
 		(unit 1)
 		(body_style 1)
@@
 		(fields_autoplaced yes)
 		(property "Reference" "D5"
-			(at 82.55 48.2599 90)
+			(at 82.55 50.7999 90)
 			(show_name no)
 			(do_not_autoplace no)
@@
 		)
 		(property "Value" "SM15T36CA"
-			(at 82.55 50.7999 90)
+			(at 82.55 53.3399 90)
 			(show_name no)
 			(do_not_autoplace no)
@@
 			)
 		)
-		(property "Footprint" "Diode_SMD:D_SMA"
-			(at 71.374 50.038 0)
+		(property "Footprint" "Diode_SMD:D_0201_0603Metric_Pad0.64x0.40mm_HandSolder"
+			(at 71.374 52.578 0)
 			(hide yes)
 			(show_name no)
@@
 		)
 		(property "Datasheet" "https://www.st.com/resource/en/datasheet/sm15t36a.pdf"
-			(at 73.406 49.53 0)
+			(at 73.406 52.07 0)
 			(hide yes)
 			(show_name no)
@@
 		)
 		(property "Description" "1500W (10/1000 μs) Bidirectional TVS Diode, VRM = 30.8V (IRM = 0.2 μA at 25°C), VBR = 34.2 ... 37.8V, 'BEV' marking, SMC"
-			(at 75.438 49.53 0)
+			(at 75.438 52.07 0)
 			(hide yes)
 			(show_name no)
@@
 		)
 		(property "SNAPEDA_PN" ""
-			(at 80.01 49.53 90)
+			(at 80.01 52.07 90)
 			(hide yes)
 			(show_name no)
@@
 			)
 		)
-		(property "mouser" "511-SM15T36CAY"
-			(at 80.01 49.53 90)
+		(property "mouser" "511-ESDL031-1BF4 "
+			(at 80.01 52.07 90)
 			(hide yes)
 			(show_name no)
@@
 		(exclude_from_sim no)
 		(in_bom yes)
-		(on_board yes)
+		(on_board no)
 		(in_pos_files yes)
-		(dnp no)
+		(dnp yes)
 		(fields_autoplaced yes)
 		(property "Reference" "C28"
@@
 		(exclude_from_sim no)
 		(in_bom yes)
-		(on_board yes)
+		(on_board no)
 		(in_pos_files yes)
-		(dnp no)
+		(dnp yes)
 		(property "Reference" "J6"
 			(at 66.04 40.9331 0)
