File: KB-01_kicad/KB-01/CM5_GPIO.kicad_sch (KiCad schematic)
At the start: 1 part

Commit message: up
Parts:
- added BT1: Battery_Cell, CM5IO:BatteryHolder_Keystone_3034_1x20mm, symbol Device:Battery_Cell
- added D4: LED Red, LED_SMD:LED_0603_1608Metric, symbol Device:LED
- added D7: LED Green, LED_SMD:LED_0603_1608Metric, symbol Device:LED
- added J7: Conn_01x03, Connector_PinHeader_2.54mm:PinHeader_1x03_P2.54mm_Vertical, symbol Connector_Generic:Conn_01x03
- added R20, R21: 1k, Resistor_SMD:R_0402_1005Metric, symbol Device:R
- added SW1: Right angle Tact button, Button_Switch_THT:SW_Tactile_SPST_Angled_PTS645Vx58-2LFS, symbol Switch:SW_Push
- added TP3, TP5: TestPoint, TestPoint:TestPoint_Pad_2.0x2.0mm, symbol Connector:TestPoint
- added U13: 74LVC1G07SE-7, Package_TO_SOT_SMD:SOT-353_SC-70-5, symbol CM5IO:74LVC1G07_copy
Connections:
- net GND: now reaches Module1.1 (GND)
- net GND: now also Module1.13 (GND), Module1.14 (GND), Module1.2 (GND), Module1.22 (GND), Module1.23 (GND), Module1.32 (GND), Module1.33 (GND), Module1.42 (GND), Module1.43 (GND), Module1.52 (GND), Module1.53 (GND), Module1.59 (GND), Module1.60 (GND), Module1.65 (GND), Module1.66 (GND), Module1.7 (GND), Module1.71 (GND), Module1.74 (GND), Module1.8 (GND), Module1.98 (GND), BT1.2 (-), J7.2 (Pin_2), SW1.2, U13.3 (GND)
- net TRD0_N: now reaches Module1.10 (Ethernet_Pair0_N)
- net CAM_GPIO1: now reaches Module1.100 (CAM_GPIO1)
- net TRD0_P: now reaches Module1.12 (Ethernet_Pair0_P)
- net TACHO: now reaches Module1.16 (FAN_TACHO)
- net SYNC_OUT: now reaches Module1.18 (Ethernet_SYNC_OUT(3.3v))
- net PWM: now reaches Module1.19 (FAN_PWM)
- net EEPROM_nWP: now reaches Module1.20 (EEPROM_nWP)
- net at Module1.21 (LED_nACT): now also R21.2
- net I2C1_SDA: now reaches Module1.24 (GPIO26)
- net GPIO21: now reaches Module1.25 (GPIO21)
- net GPIO19: now reaches Module1.26 (GPIO19)
- net GPIO20: now reaches Module1.27 (GPIO20)
- net UART4_RX: now reaches Module1.28 (GPIO13)
- net GPIO16: now reaches Module1.29 (GPIO16)
- net GPIO6: now reaches Module1.30 (GPIO6)
- net UART4_TX: now reaches Module1.31 (GPIO12)
- net GPIO5: now reaches Module1.34 (GPIO5)
- net I2C0_SCL: now reaches Module1.35 (ID_SC)
- net I2C0_SDA: now reaches Module1.36 (ID_SD)
- net GPIO7: now reaches Module1.37 (GPIO7)
- net SPI0_SCLK: now reaches Module1.38 (GPIO11)
- net SPI0_CSn(0): now reaches Module1.39 (GPIO8)
- net TRD1_P: now reaches Module1.4 (Ethernet_Pair1_P)
- net SPI0_SIO(1): now reaches Module1.40 (GPIO9)
- net GPIO25: now reaches Module1.41 (GPIO25)
- net SPI0_SIO(0): now reaches Module1.44 (GPIO10)
- net GPIO24: now reaches Module1.45 (GPIO24)
- net GPIO22: now reaches Module1.46 (GPIO22)
- net GPIO23: now reaches Module1.47 (GPIO23)
- net GPIO27: now reaches Module1.48 (GPIO27)
- net GPIO18: now reaches Module1.49 (GPIO18)
- net GPIO17: now reaches Module1.50 (GPIO17)
- net UART4_RTS: now reaches Module1.51 (GPIO15)
- net GPIO4: now reaches Module1.54 (GPIO4)
- net UART4_CTS: now reaches Module1.55 (GPIO14)
- net I2C1_SCL: now reaches Module1.56 (GPIO3)
- net SD_CLK: now reaches Module1.57 (SD_CLK)
- net GPIO2: now reaches Module1.58 (GPIO2)
- net TRD1_N: now reaches Module1.6 (Ethernet_Pair1_N)
- net SD_DAT3: now reaches Module1.61 (SD_DAT3)
- net SD_CMD: now reaches Module1.62 (SD_CMD)
- net SD_DAT0: now reaches Module1.63 (SD_DAT0)
- net SD_DAT1: now reaches Module1.67 (SD_DAT1)
- net SD_DAT2: now reaches Module1.69 (SD_DAT2)
- net SD_PWR_ON: now reaches Module1.75 (SD_PWR_ON)
- net VBAT: now reaches Module1.76 (VBAT)
- net VBAT: now also BT1.1 (+)
- net +5v: now reaches Module1.77 (+5v_(Input))
- net +5v: now also Module1.79 (+5v_(Input)), Module1.81 (+5v_(Input)), Module1.83 (+5v_(Input)), Module1.85 (+5v_(Input)), Module1.87 (+5v_(Input))
- net GPIO_VREF: now reaches Module1.78 (GPIO_VREF(1.8v/3.3v_Input))
- net SCL0: now reaches Module1.80 (SCL0)
- net SDA0: now reaches Module1.82 (SDA0)
- net +3.3v: now reaches Module1.84 (+3.3v_(Output))
- net +3.3v: now also Module1.86 (+3.3v_(Output)), D4.2 (A), D7.2 (A), U13.5 (VCC)
- net +1.8v: now reaches Module1.88 (+1.8v_(Output))
- net +1.8v: now also Module1.90 (+1.8v_(Output))
- net WL_nDis: now reaches Module1.89 (WiFi_nDisable)
- net WL_nDis: now also J7.1 (Pin_1)
- net BT_nDis: now reaches Module1.91 (BT_nDisable)
- net BT_nDis: now also J7.3 (Pin_3)
- net PWR_BUT: now reaches Module1.92 (PWR_BUT)
- net PWR_BUT: now also SW1.1
- net nRPIBOOT: now reaches Module1.93 (nRPIBOOT)
- net CC1: now reaches Module1.94 (CC1)
- net nPWR_LED: now reaches Module1.95 (LED_nPWR)
- net nPWR_LED: now also U13.2
- net CC2: now reaches Module1.96 (CC2)
- net CAM_GPIO0: now reaches Module1.97 (CAM_GPIO0)
- net PMIC_ENABLE: now reaches Module1.99 (PMIC_ENABLE)
- new net: D4.1 (K), R20.1, TP5.1
- new net: R20.2, U13.4
- new net: D7.1 (K), R21.1, TP3.1
- no-connect marks 0 -> 5
Other:
- note added: "Activity LED"
- note added: "I2C for display dont use"
- note added: "Not Fitted header"
- note added: "PWR LED"

Commit message: everything
Parts:
- removed J7: Conn_01x03, Connector_PinHeader_2.54mm:PinHeader_1x03_P2.54mm_Vertical, symbol Connector_Generic:Conn_01x03
- removed U13: 74LVC1G07SE-7, Package_TO_SOT_SMD:SOT-353_SC-70-5, symbol CM5IO:74LVC1G07_copy
- added J4: Conn_01x03, Connector_PinHeader_2.54mm:PinHeader_1x03_P2.54mm_Vertical, symbol Connector_Generic:Conn_01x03
Connections:
- net GPIO2 is gone; now on net I2C1_SDA: Module1.58 (GPIO2)
- net BT_nDis: now also J4.3 (Pin_3)
- net GND: now also J4.2 (Pin_2)
- net I2C1_SDA: no longer Module1.24 (GPIO26)
- net WL_nDis: now also J4.1 (Pin_1)
- net nPWR_LED: now also R20.2
- net TRD2_P: now reaches Module1.11 (Ethernet_Pair2_P)
- net ETH_LEDY: now reaches Module1.15 (Ethernet_nLED3(3.3v))
- net ETH_LEDG: now reaches Module1.17 (Ethernet_nLED2(3.3v))
- net TRD3_P: now reaches Module1.3 (Ethernet_Pair3_P)
- net TRD3_N: now reaches Module1.5 (Ethernet_Pair3_N)
- net TRD2_N: now reaches Module1.9 (Ethernet_Pair2_N)
- net GPIO16 renamed GNSS_RSTn
- net GPIO17 renamed BQ_CE
- net GPIO20 renamed GNSS_WAKEUP
- net GPIO21 renamed GNSS_PSU_EN
- net GPIO22 renamed FG_INT
- net GPIO23 renamed BMI270_INT1
- net GPIO24 renamed LIS2MDL_INT
- net GPIO25 renamed BMP390_INT
- net GPIO27 renamed BQ_INT
- net GPIO4 renamed I2C2_SDA
- net GPIO5 renamed I2C2_SCL
- net GPIO6 renamed I2C3_SDA
- net GPIO7 renamed I2C3_SCL
- net I2C0_SCL renamed ID_SC
- net I2C0_SDA renamed ID_SD
- net SPI0_SCLK renamed SPIO_SCLK
- net SPI0_SIO(1) renamed SPIO_SIO(1)
- net UART4_CTS renamed UART0_TX
- net UART4_RTS renamed UART0_RX
- net UART4_RX renamed GPIO13
- net UART4_TX renamed GPIO12
- new net BMI270_INT2: Module1.24 (GPIO26)
Other:
- note added: "For MIPI"
- note added: "Has internal 1.8k pull-up"
- note added: "Leave unconnected"
- note removed: "I2C for display dont use"
- moved on the sheet: BT1, Module1A, SW1, TP3, TP5

Commit message: all
Connections:
- net I2C3_SCL renamed GPIO7
- net I2C3_SDA renamed GPIO6
- net VBAT renamed Coin_bat
Changed lines of the file:
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@@
+		)
+	)
+	(hierarchical_label "GPIO19"
+		(shape input)
+		(at 92.71 59.69 180)
+		(effects
+			(font
+				(size 1.27 1.27)
+			)
+			(justify right)
 		)
 	)
@@
 		)
 	)
+	(hierarchical_label "GPIO18"
+		(shape input)
+		(at 182.88 90.17 0)
+		(effects
+			(font
+				(size 1.27 1.27)
+			)
+			(justify left)
+		)
+	)
 	(hierarchical_label "ID_SC"
 		(shape output)
@@
 		)
 	)
-	(hierarchical_label "I2C3_SDA"
+	(hierarchical_label "I2C1_SCL"
+		(shape input)
+		(at 92.71 97.79 180)
+		(effects
+			(font
+				(size 1.27 1.27)
+			)
+			(justify right)
+		)
+	)
+	(hierarchical_label "+3.3v"
+		(shape output)
+		(at 93.98 133.35 180)
+		(effects
+			(font
+				(size 1.27 1.27)
+			)
+			(justify right)
+		)
+	)
+	(hierarchical_label "UART0_TX"
+		(shape input)
+		(at 182.88 97.79 0)
+		(effects
+			(font
+				(size 1.27 1.27)
+			)
+			(justify left)
+		)
+	)
+	(hierarchical_label "SDA0"
+		(shape output)
+		(at 93.98 130.81 180)
+		(effects
+			(font
+				(size 1.27 1.27)
+			)
+			(justify right)
+		)
+	)
+	(hierarchical_label "GPIO7"
+		(shape output)
+		(at 182.88 74.93 0)
+		(effects
+			(font
+				(size 1.27 1.27)
+			)
+			(justify left)
+		)
+	)
+	(hierarchical_label "I2C2_SDA"
+		(shape input)
+		(at 92.71 95.25 180)
+		(effects
+			(font
+				(size 1.27 1.27)
+			)
+			(justify right)
+		)
+	)
+	(hierarchical_label "LIS2MDL_INT"
+		(shape input)
+		(at 182.88 85.09 0)
+		(effects
+			(font
+				(size 1.27 1.27)
+			)
+			(justify left)
+		)
+	)
+	(hierarchical_label "BMI270_INT1"
+		(shape input)
+		(at 182.88 87.63 0)
+		(effects
+			(font
+				(size 1.27 1.27)
+			)
+			(justify left)
+		)
+	)
+	(hierarchical_label "GNSS_PSU_EN"
+		(shape input)
+		(at 182.88 59.69 0)
+		(effects
+			(font
+				(size 1.27 1.27)
+			)
+			(justify left)
+		)
+	)
+	(hierarchical_label "I2C1_SDA"
+		(shape input)
+		(at 92.71 100.33 180)
+		(effects
+			(font
+				(size 1.27 1.27)
+			)
+			(justify right)
+		)
+	)
+	(hierarchical_label "BMI270_INT2"
+		(shape input)
+		(at 92.71 57.15 180)
+		(effects
+			(font
+				(size 1.27 1.27)
+			)
+			(justify right)
+		)
+	)
+	(hierarchical_label "SPIO_SCLK"
+		(shape input)
+		(at 92.71 74.93 180)
+		(effects
+			(font
+				(size 1.27 1.27)
+			)
+			(justify right)
+		)
+	)
+	(hierarchical_label "Coin_bat"
+		(shape output)
+		(at 52.07 92.71 0)
+		(effects
+			(font
+				(size 1.27 1.27)
+			)
+			(justify left)
+		)
+	)
+	(hierarchical_label "CC2"
+		(shape output)
+		(at 93.98 148.59 180)
+		(effects
+			(font
+				(size 1.27 1.27)
+			)
+			(justify right)
+		)
+	)
+	(hierarchical_label "GPIO_VREF"
+		(shape output)
+		(at 93.98 125.73 180)
+		(effects
+			(font
+				(size 1.27 1.27)
+			)
+			(justify right)
+		)
+	)
+	(hierarchical_label "BMP390_INT"
+		(shape input)
+		(at 182.88 80.01 0)
+		(effects
+			(font
+				(size 1.27 1.27)
+			)
+			(justify left)
+		)
+	)
+	(hierarchical_label "UART0_RX"
+		(shape input)
+		(at 182.88 92.71 0)
+		(effects
+			(font
+				(size 1.27 1.27)
+			)
+			(justify left)
+		)
+	)
+	(hierarchical_label "CC1"
+		(shape output)
+		(at 93.98 146.05 180)
+		(effects
+			(font
+				(size 1.27 1.27)
+			)
+			(justify right)
+		)
+	)
+	(hierarchical_label "CAM_GPIO0"
+		(shape output)
+		(at 185.42 151.13 0)
+		(effects
+			(font
+				(size 1.27 1.27)
+			)
+			(justify left)
+		)
+	)
+	(hierarchical_label "I2C2_SCL"
+		(shape input)
+		(at 92.71 69.85 180)
+		(effects
+			(font
+				(size 1.27 1.27)
+			)
+			(justify right)
+		)
+	)
+	(hierarchical_label "GPIO12"
+		(shape input)
+		(at 182.88 67.31 0)
+		(effects
+			(font
+				(size 1.27 1.27)
+			)
+			(justify left)
+		)
+	)
+	(hierarchical_label "GPIO13"
+		(shape input)
+		(at 92.71 62.23 180)
+		(effects
+			(font
+				(size 1.27 1.27)
+			)
+			(justify right)
+		)
+	)
+	(hierarchical_label "FG_INT"
+		(shape input)
+		(at 92.71 85.09 180)
+		(effects
+			(font
+				(size 1.27 1.27)
+			)
+			(justify right)
+		)
+	)
+	(hierarchical_label "GPIO6"
 		(shape input)
 		(at 92.71 64.77 180)
 		(effects
 			(font
-				(size 1.27 1.27)
-			)
-			(justify right)
-		)
-	)
-	(hierarchical_label "I2C1_SCL"
-		(shape input)
-		(at 92.71 97.79 180)
-		(effects
-			(font
-				(size 1.27 1.27)
-			)
-			(justify right)
-		)
-	)
-	(hierarchical_label "+3.3v"
-		(shape output)
-		(at 93.98 133.35 180)
-		(effects
-			(font
-				(size 1.27 1.27)
-			)
-			(justify right)
-		)
-	)
-	(hierarchical_label "UART0_TX"
-		(shape input)
-		(at 182.88 97.79 0)
-		(effects
-			(font
-				(size 1.27 1.27)
-			)
-			(justify left)
-		)
-	)
-	(hierarchical_label "SDA0"
-		(shape output)
-		(at 93.98 130.81 180)
-		(effects
-			(font
-				(size 1.27 1.27)
-			)
-			(justify right)
-		)
-	)
-	(hierarchical_label "I2C2_SDA"
-		(shape input)
-		(at 92.71 95.25 180)
-		(effects
-			(font
-				(size 1.27 1.27)
-			)
-			(justify right)
-		)
-	)
-	(hierarchical_label "LIS2MDL_INT"
-		(shape input)
-		(at 182.88 85.09 0)
-		(effects
-			(font
-				(size 1.27 1.27)
-			)
-			(justify left)
-		)
-	)
-	(hierarchical_label "BMI270_INT1"
-		(shape input)
-		(at 182.88 87.63 0)
-		(effects
-			(font
-				(size 1.27 1.27)
-			)
-			(justify left)
-		)
-	)
-	(hierarchical_label "GNSS_PSU_EN"
-		(shape input)
-		(at 182.88 59.69 0)
-		(effects
-			(font
-				(size 1.27 1.27)
-			)
-			(justify left)
-		)
-	)
-	(hierarchical_label "I2C1_SDA"
-		(shape input)
-		(at 92.71 100.33 180)
-		(effects
-			(font
-				(size 1.27 1.27)
-			)
-			(justify right)
-		)
-	)
-	(hierarchical_label "BMI270_INT2"
-		(shape input)
-		(at 92.71 57.15 180)
-		(effects
-			(font
-				(size 1.27 1.27)
-			)
-			(justify right)
-		)
-	)
-	(hierarchical_label "SPIO_SCLK"
-		(shape input)
-		(at 92.71 74.93 180)
-		(effects
-			(font
-				(size 1.27 1.27)
-			)
-			(justify right)
-		)
-	)
-	(hierarchical_label "I2C3_SCL"
-		(shape input)
-		(at 182.88 74.93 0)
-		(effects
-			(font
-				(size 1.27 1.27)
-			)
-			(justify left)
-		)
-	)
-	(hierarchical_label "CC2"
-		(shape output)
-		(at 93.98 148.59 180)
-		(effects
-			(font
-				(size 1.27 1.27)
-			)
-			(justify right)
-		)
-	)
-	(hierarchical_label "GPIO_VREF"
-		(shape output)
-		(at 93.98 125.73 180)
-		(effects
-			(font
-				(size 1.27 1.27)
-			)
-			(justify right)
-		)
-	)
-	(hierarchical_label "BMP390_INT"
-		(shape input)
-		(at 182.88 80.01 0)
-		(effects
-			(font
-				(size 1.27 1.27)
-			)
-			(justify left)
-		)
-	)
-	(hierarchical_label "UART0_RX"
-		(shape input)
-		(at 182.88 92.71 0)
-		(effects
-			(font
-				(size 1.27 1.27)
-			)
-			(justify left)
-		)
-	)
-	(hierarchical_label "CC1"
-		(shape output)
-		(at 93.98 146.05 180)
-		(effects
-			(font
-				(size 1.27 1.27)
-			)
-			(justify right)
-		)
-	)
-	(hierarchical_label "CAM_GPIO0"
-		(shape output)
-		(at 185.42 151.13 0)
-		(effects
-			(font
-				(size 1.27 1.27)
-			)
-			(justify left)
-		)
-	)
-	(hierarchical_label "I2C2_SCL"
-		(shape input)
-		(at 92.71 69.85 180)
-		(effects
-			(font
-				(size 1.27 1.27)
-			)
-			(justify right)
-		)
-	)
-	(hierarchical_label "FG_INT"
-		(shape input)
-		(at 92.71 85.09 180)
-		(effects
-			(font

Commit message: all
Parts:
- D7: mouser (none) -> 859-LTST-C190KGKT
Changed lines of the file:
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@@
+			)
+		)
+		(property "mouser" "859-LTST-C190KGKT"
+			(at 185.42 35.56 90)
+			(hide yes)
+			(show_name no)
+			(do_not_autoplace no)
+			(effects
+				(font
+					(size 1.27 1.27)
+				)
 			)
 		)

Commit message: all
Parts:
- added C41: 0.1F, Capacitor_SMD:CP_Elec_10x10.5, symbol Device:C_Polarized
- added C56: 100nF 6.3V, Capacitor_SMD:C_0603_1608Metric_Pad1.08x0.95mm_HandSolder, symbol Device:C
- D4: mouser (none) -> 755-SML-D12L8WT86
Connections:
- net Coin_bat: now also C41.1, C56.1
- net GND: now also C41.2, C56.2
Other:
- note added: "Use supercap instead"
- moved on the sheet: BT1

Commit message: all
Parts:
- C41: value 0.1F -> 0.1F 5.5V; mouser (none) -> 80-FC0V104ZFTBR24
- R20, R21: footprint Resistor_SMD:R_0402_1005Metric -> Resistor_SMD:R_0603_1608Metric_Pad0.98x0.95mm_HandSolder; mouser (none) -> 652-CR0603FX-1001ELF
- SW1: footprint Button_Switch_THT:SW_Tactile_SPST_Angled_PTS645Vx58-2LFS -> Button_Switch_SMD:SW_SPST_EVQP7A; mouser (none) -> 667-EVQP7A01P
Changed lines of the file:
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@@
 			)
 		)
-		(property "Footprint" "Resistor_SMD:R_0402_1005Metric"
+		(property "Footprint" "Resistor_SMD:R_0603_1608Metric_Pad0.98x0.95mm_HandSolder"
 			(at 183.642 48.26 90)
 			(hide yes)
@@
 		)
 		(property "SNAPEDA_PN" ""
+			(at 185.42 48.26 0)
+			(hide yes)
+			(show_name no)
+			(do_not_autoplace no)
+			(effects
+				(font
+					(size 1.27 1.27)
+				)
+			)
+		)
+		(property "mouser" "652-CR0603FX-1001ELF "
 			(at 185.42 48.26 0)
 			(hide yes)
@@
 			)
 		)
-		(property "Footprint" "Button_Switch_THT:SW_Tactile_SPST_Angled_PTS645Vx58-2LFS"
+		(property "Footprint" "Button_Switch_SMD:SW_SPST_EVQP7A"
 			(at 48.26 71.12 0)
 			(hide yes)
@@
 		)
 		(property "SNAPEDA_PN" ""
+			(at 43.18 71.12 90)
+			(hide yes)
+			(show_name no)
+			(do_not_autoplace no)
+			(effects
+				(font
+					(size 1.27 1.27)
+				)
+			)
+		)
+		(property "mouser" "667-EVQP7A01P"
 			(at 43.18 71.12 90)
 			(hide yes)
@@
 			)
 		)
-		(property "Footprint" "Resistor_SMD:R_0402_1005Metric"
+		(property "Footprint" "Resistor_SMD:R_0603_1608Metric_Pad0.98x0.95mm_HandSolder"
 			(at 41.402 48.26 90)
 			(hide yes)
@@
 		)
 		(property "SNAPEDA_PN" ""
+			(at 43.18 48.26 0)
+			(hide yes)
+			(show_name no)
+			(do_not_autoplace no)
+			(effects
+				(font
+					(size 1.27 1.27)
+				)
+			)
+		)
+		(property "mouser" "652-CR0603FX-1001ELF "
 			(at 43.18 48.26 0)
 			(hide yes)
@@
 			)
 		)
-		(property "Value" "0.1F"
+		(property "Value" "0.1F 5.5V"
 			(at 36.83 110.8709 0)
 			(show_name no)
@@
 			(at 33.02 110.49 0)
 			(hide yes)
+			(show_name no)
+			(do_not_autoplace no)
+			(effects
+				(font
+					(size 1.27 1.27)
+				)
+			)
+		)
+		(property "mouser" "80-FC0V104ZFTBR24"
+			(at 33.02 110.49 0)
+			(hide yes)
