File: KB-01_kicad/KB-01/CM5_GPIO.kicad_sch (KiCad schematic)
At the start: 12 parts, among them J4 Conn_01x03, SW1 Right angle Tact button

Commit message: all
Parts:
- added J11: Conn_02x07_Odd_Even, Connector_PinHeader_1.00mm:PinHeader_2x07_P1.00mm_Vertical_SMD, symbol Connector_Generic:Conn_02x07_Odd_Even
- Module1: mouser (none) -> 798-DF40C100DS0.4V58
- renumbered C56 to C1, C41 to C2, D7 to D1, D4 to D2, J4 to J2, R20 to R3, R21 to R4, TP3 to TP1, TP5 to TP2
Connections:
- net GPIO_VREF is gone; now on net +3.3v: Module1.78 (GPIO_VREF(1.8v/3.3v_Input))
- net EEPROM_nWP: now also J11.4 (Pin_4)
- net GND: now also J11.1 (Pin_1), J11.11 (Pin_11), J11.13 (Pin_13), J11.3 (Pin_3), J11.5 (Pin_5), J11.7 (Pin_7), J11.9 (Pin_9)
- net PMIC_ENABLE: now also J11.12 (Pin_12)
- net PWR_BUT: now also J11.14 (Pin_14)
- net SYNC_OUT: now also J11.6 (Pin_6)
- net nRPIBOOT: now also J11.2 (Pin_2)
- new net USBOTG: J11.10 (Pin_10)
- no-connect marks 5 -> 6
Other:
- note added: "Force RPIBOOT = Jumper Pins 1-2"
- note added: "GPIO Voltage select"

Commit message: all
Parts:
- C2: value 0.1F 5.5V -> 0.1F 3.5V
Connections:
- net Coin_bat renamed +3V_CHRG
Changed lines of the file:
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@@
 	(text "GPIO Voltage select\n"
 		(exclude_from_sim no)
-		(at 72.136 125.476 0)
+		(at 86.106 126.238 0)
 		(effects
 			(font
@@
 	(wire
 		(pts
+			(xy 91.44 123.19) (xy 107.95 123.19)
+		)
+		(stroke
+			(width 0)
+			(type default)
+		)
+	)
+	(wire
+		(pts
 			(xy 92.71 49.53) (xy 107.95 49.53)
 		)
@@
 	(wire
 		(pts
-			(xy 93.98 123.19) (xy 107.95 123.19)
-		)
-		(stroke
-			(width 0)
-			(type solid)
-		)
-	)
-	(wire
-		(pts
 			(xy 168.91 133.35) (xy 168.91 135.89)
 		)
@@
 	(wire
 		(pts
+			(xy 91.44 120.65) (xy 91.44 123.19)
+		)
+		(stroke
+			(width 0)
+			(type default)
+		)
+	)
+	(wire
+		(pts
 			(xy 168.91 90.17) (xy 182.88 90.17)
 		)
@@
 	)
 	(symbol
+		(lib_id "power:+3V3")
+		(at 91.44 120.65 0)
+		(unit 1)
+		(body_style 1)
+		(exclude_from_sim no)
+		(in_bom yes)
+		(on_board yes)
+		(in_pos_files yes)
+		(dnp no)
+		(property "Reference" "#PWR090"
+			(at 91.44 124.46 0)
+			(hide yes)
+			(show_name no)
+			(do_not_autoplace no)
+			(effects
+				(font
+					(size 1.27 1.27)
+				)
+			)
+		)
+		(property "Value" "+3V_CHRG"
+			(at 91.44 116.586 0)
+			(show_name no)
+			(do_not_autoplace no)
+			(effects
+				(font
+					(size 1.27 1.27)
+				)
+			)
+		)
+		(property "Footprint" ""
+			(at 91.44 120.65 0)
+			(hide yes)
+			(show_name no)
+			(do_not_autoplace no)
+			(effects
+				(font
+					(size 1.27 1.27)
+				)
+			)
+		)
+		(property "Datasheet" ""
+			(at 91.44 120.65 0)
+			(hide yes)
+			(show_name no)
+			(do_not_autoplace no)
+			(effects
+				(font
+					(size 1.27 1.27)
+				)
+			)
+		)
+		(property "Description" "Power symbol creates a global label with name \"+3V3\""
+			(at 91.44 120.65 0)
+			(hide yes)
+			(show_name no)
+			(do_not_autoplace no)
+			(effects
+				(font
+					(size 1.27 1.27)
+				)
+			)
+		)
+		(pin "1"
+		)
+		(instances
+			(project "KB-01"
+				(path "/e6144e29-1dc4-45a8-93e7-988a20131b94/e0fc78fc-72bd-4488-afe4-0929818a7c1a"
+					(reference "#PWR090")
+					(unit 1)
+				)
+			)
+		)
+	)
+	(symbol
 		(lib_id "Connector:TestPoint")
 		(at 191.77 41.91 270)
@@
 		(exclude_from_sim no)
 		(in_bom yes)
-		(on_board yes)
+		(on_board no)
 		(in_pos_files yes)
 		(dnp no)
@@
 		(exclude_from_sim no)
 		(in_bom yes)
-		(on_board yes)
+		(on_board no)
 		(in_pos_files yes)
 		(dnp no)
@@
 			)
 		)
-		(property "Value" "0.1F 5.5V"
+		(property "Value" "0.1F 3.5V"
 			(at 36.83 110.8709 0)
 			(show_name no)

Commit message: all
Parts:
- added C58: 10uF 6.3V, Resistor_SMD:R_0603_1608Metric_Pad0.98x0.95mm_HandSolder, symbol Device:C
- added J14: Micro_SD_Card_Det, CM5IO:SDCARD_MOLEX_503398-1892, symbol Connector:Micro_SD_Card_Det2
- added R36: 10K 1%, Resistor_SMD:R_0603_1608Metric_Pad0.98x0.95mm_HandSolder, symbol Device:R
- added U18: RT9742GGJ5 / NCP380HSN10AAT1G, Package_TO_SOT_SMD:SOT-23-5, symbol CM5IO:RT9742GGJ5
- BT1, C1, C2: now not fitted
Connections:
- net +3.3v: now also R36.1, U18.5 (IN)
- net GND: now also C58.2, J14.11 (SHIELD), J14.6 (VSS), U18.2 (GND)
- net SD_CLK: now also J14.5 (CLK)
- net SD_CMD: now also J14.3 (CMD)
- net SD_DAT0: now also J14.7 (DAT0)
- net SD_DAT1: now also J14.8 (DAT1)
- net SD_DAT2: now also J14.1 (DAT2)
- net SD_DAT3: now also J14.2 (DAT3/CD)
- net SD_PWR_ON: now also R36.2, U18.4 (EN)
- new net SD_PWR: C58.1, J14.4 (VDD), U18.1 (OUT)
- no-connect marks 6 -> 9
Other:
- note added: "CM5Lite SDCARD I/F"
- note added: "For display MIPI"
- note added: "R2 : Add R13 to support CM4Lite"
- note added: "Repurpose for wheel sensor"
- note added: "Vbat comes straight from battery pack"
- note removed: "For MIPI"
- note removed: "Use supercap instead"

Commit message: all
Other:
- note added: "R2 : Add R36 to support CM4Lite"
- note removed: "R2 : Add R13 to support CM4Lite"
Changed lines of the file:
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@@
 		)
 	)
-	(text "R2 : Add R13 to support CM4Lite"
+	(text "R2 : Add R36 to support CM4Lite"
 		(exclude_from_sim no)
 		(at 259.334 121.412 0)
@@
 		(exclude_from_sim no)
 		(in_bom no)
-		(on_board yes)
+		(on_board no)
 		(in_pos_files yes)
 		(dnp yes)
@@
 		(exclude_from_sim yes)
 		(in_bom no)
-		(on_board yes)
+		(on_board no)
 		(in_pos_files yes)
 		(dnp yes)
@@
 		(exclude_from_sim no)
 		(in_bom no)
-		(on_board yes)
+		(on_board no)
 		(in_pos_files yes)
 		(dnp yes)
