File: KB-01_kicad/KB-01/CM5_GPIO.kicad_sch (KiCad schematic)
At the start: 17 parts, among them J11 Conn_02x07_Odd_Even, J14 Micro_SD_Card_Det, J2 Conn_01x03, SW1 Right angle Tact button, U18 RT9742GGJ5 / NCP380HSN10AAT1G

Commit message: all
Parts:
- Module1: mouser 798-DF40C100DS0.4V58 -> 649-101642271004RLF
Changed lines of the file:
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@@
 			)
 		)
-		(property "mouser" "798-DF40C100DS0.4V58 "
+		(property "mouser" "649-101642271004RLF "
 			(at 140.97 85.09 0)
 			(hide yes)
