File: KB-01_kicad/KB-01/pcie-nvme.kicad_sch (KiCad schematic)
At the start: 20 parts, among them J1 Bus_M.2_Socket_M, M1 M.2 Solder Nut, M2 M.2 Screw, U4 ASEK-32.768KHZ-L-R-T, U5 AP3441SHE-7B

Commit message: all
Parts:
- J8: renamed from J1; footprint M.2 NGFF:121992304 -> CM5IO:M.2 M Key socket
- renumbered C8 to C34, C1 to C35, C2 to C36, C3 to C37, C4 to C38, C5 to C39, C6 to C40, C7 to C41, C9 to C42, D1 to D8, L1 to L5, M2 to M1, M1 to M2, R4 to R21, R30 to R22, R3 to R23, R2 to R24, U5 to U10, U4 to U9
Connections:
- net M.2_3v3: no longer J8.68 (SUSCLK), U9.3 (Out)
- new net: J8.68 (SUSCLK), U9.3 (Out)

Commit message: all
Connections:
- net GND: no longer J8.M2 (GND2242), J8.M3 (GND2260), J8.M4 (GND2280)
- no-connect marks 15 -> 18

Commit message: all
Parts:
- R22: mouser 708-RMCF0603FT10K0 -> 667-ERJ-3EKF1002V
- R24: value 2.2k 1% -> 2.2K 1%
Changed lines of the file:
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@@
 			)
 		)
-		(property "Value" "2.2k 1%"
+		(property "Value" "2.2K 1%"
 			(at 132.08 182.8799 0)
 			(show_name no)
@@
 			)
 		)
-		(property "mouser" "708-RMCF0603FT10K0"
+		(property "mouser" "667-ERJ-3EKF1002V"
 			(at 129.54 170.18 0)
 			(hide yes)
