File: KB-01_kicad/KB-01/CM5_high_speed.kicad_sch (KiCad schematic)
At the start: 1 part

Commit message: up
Parts:
- added J16, J6: Conn_01x22_Female, CM5IO:Hirose_FH12-22S-0.5SH_1x22-1MP_P0.50mm_Horizontal, symbol Connector:Conn_01x22_Socket
- added R19: 2.2K 1%, Resistor_SMD:R_0402_1005Metric, symbol Device:R
Connections:
- new net: J16.17 (Pin_17), R19.2
- new net +3.3v: J16.22 (Pin_22), J6.22 (Pin_22), R19.1
- new net CAM_GPIO0: J6.17 (Pin_17)
- new net CAM_GPIO1: J6.18 (Pin_18)
- new net DPHY0_C_N: J6.8 (Pin_8)
- new net DPHY0_C_P: J6.9 (Pin_9)
- new net DPHY0_D0_N: J6.2 (Pin_2)
- new net DPHY0_D0_P: J6.3 (Pin_3)
- new net DPHY0_D1_N: J6.5 (Pin_5)
- new net DPHY0_D1_P: J6.6 (Pin_6)
- new net DPHY0_D2_N: J6.11 (Pin_11)
- new net DPHY0_D2_P: J6.12 (Pin_12)
- new net DPHY0_D3_N: J6.14 (Pin_14)
- new net DPHY0_D3_P: J6.15 (Pin_15)
- new net DPHY1_C_N: J16.8 (Pin_8)
- new net DPHY1_C_P: J16.9 (Pin_9)
- new net DPHY1_D0_N: J16.2 (Pin_2)
- new net DPHY1_D0_P: J16.3 (Pin_3)
- new net DPHY1_D1_N: J16.5 (Pin_5)
- new net DPHY1_D1_P: J16.6 (Pin_6)
- new net DPHY1_D2_N: J16.11 (Pin_11)
- new net DPHY1_D2_P: J16.12 (Pin_12)
- new net DPHY1_D3_N: J16.14 (Pin_14)
- new net DPHY1_D3_P: J16.15 (Pin_15)
- new net GND: J16.1 (Pin_1), J16.10 (Pin_10), J16.13 (Pin_13), J16.16 (Pin_16), J16.19 (Pin_19), J16.4 (Pin_4), J16.7 (Pin_7), J6.1 (Pin_1), J6.10 (Pin_10), J6.13 (Pin_13), J6.16 (Pin_16), J6.19 (Pin_19), J6.4 (Pin_4), J6.7 (Pin_7)
- new net SCL0: J6.20 (Pin_20)
- new net SCL1: J16.20 (Pin_20)
- new net SDA0: J6.21 (Pin_21)
- new net SDA1: J16.21 (Pin_21)
- no-connect marks 0 -> 1
Other:
- note added: "DSI/CSI Connectors"

Commit message: up
Connections:
- net DPHY0_C_N: now also Module1.127 (MIPI0_C_N)
- net DPHY0_C_P: now also Module1.129 (MIPI0_C_P)
- net DPHY0_D0_N: now also Module1.115 (MIPI0_D0_N)
- net DPHY0_D0_P: now also Module1.117 (MIPI0_D0_P)
- net DPHY0_D1_N: now also Module1.121 (MIPI0_D1_N)
- net DPHY0_D1_P: now also Module1.123 (MIPI0_D1_P)
- net DPHY0_D2_N: now also Module1.133 (MIPI0_D2_N)
- net DPHY0_D2_P: now also Module1.135 (MIPI0_D2_P)
- net DPHY0_D3_N: now also Module1.139 (MIPI0_D3_N)
- net DPHY0_D3_P: now also Module1.141 (MIPI0_D3_P)
- net DPHY1_C_N: now also Module1.187 (MIPI1_C_N)
- net DPHY1_C_P: now also Module1.189 (MIPI1_C_P)
- net DPHY1_D0_N: now also Module1.175 (MIPI1_D0_N)
- net DPHY1_D0_P: now also Module1.177 (MIPI1_D0_P)
- net DPHY1_D1_N: now also Module1.181 (MIPI1_D1_N)
- net DPHY1_D1_P: now also Module1.183 (MIPI1_D1_P)
- net DPHY1_D2_N: now also Module1.193 (MIPI1_D2_N)
- net DPHY1_D2_P: now also Module1.195 (MIPI1_D2_P)
- net DPHY1_D3_N: now also Module1.194 (MIPI1_D3_N)
- net DPHY1_D3_P: now also Module1.196 (MIPI1_D3_P)
- net GND: now also Module1.107 (GND), Module1.108 (GND), Module1.113 (GND), Module1.114 (GND), Module1.119 (GND), Module1.120 (GND), Module1.125 (GND), Module1.126 (GND), Module1.131 (GND), Module1.132 (GND), Module1.137 (GND), Module1.138 (GND), Module1.144 (GND), Module1.150 (GND), Module1.155 (GND), Module1.156 (GND), Module1.161 (GND), Module1.162 (GND), Module1.167 (GND), Module1.168 (GND), Module1.173 (GND), Module1.174 (GND), Module1.179 (GND), Module1.180 (GND), Module1.185 (GND), Module1.186 (GND), Module1.191 (GND), Module1.192 (GND), Module1.197 (GND), Module1.198 (GND)
- net USBOTG_ID: now reaches Module1.101 (USB_OTG_ID)
- net PCIE_nCLKREQ: now reaches Module1.102 (PCIe_nCLKREQ)
- net USB2_N: now reaches Module1.103 (USB2_N)
- net PCIE_nWAKE: now reaches Module1.104 (PCIE_nWAKE)
- net USB2_P: now reaches Module1.105 (USB2_P)
- net PCIE_PWR_EN: now reaches Module1.106 (PCIE_PWR_EN)
- net PCIE_nRST: now reaches Module1.109 (PCIe_nRST)
- net PCIE_CLK_P: now reaches Module1.110 (PCIe_CLK_P)
- net VBUS_EN: now reaches Module1.111 (VBUS_EN)
- net PCIE_CLK_N: now reaches Module1.112 (PCIe_CLK_N)
- net PCIE_RX_P: now reaches Module1.116 (PCIe_RX_P)
- net PCIE_RX_N: now reaches Module1.118 (PCIe_RX_N)
- net PCIE_TX_P: now reaches Module1.122 (PCIe_TX_P)
- net PCIE_TX_N: now reaches Module1.124 (PCIe_TX_N)
Other:
- note added: "DSI0/CSI0 Connectors"
- note added: "DSI1/CSI1 Connectors"
- note removed: "DSI/CSI Connectors"
- moved on the sheet: Module1B

Commit message: everything
Parts:
- removed J16: Conn_01x22_Female, CM5IO:Hirose_FH12-22S-0.5SH_1x22-1MP_P0.50mm_Horizontal, symbol Connector:Conn_01x22_Socket
- removed R19: 2.2K 1%, Resistor_SMD:R_0402_1005Metric, symbol Device:R
Connections:
- net USB3-0-RX_N: now reaches Module1.128 (USB3-0-RX_N)
- net USB3-0-RX_P: now reaches Module1.130 (USB3-0-RX_P)
- net USB3-0-D_P: now reaches Module1.134 (USB3-0-D_P)
- net USB3-0-D_N: now reaches Module1.136 (USB3-0-D_N)
- net USB3-0-TX_N: now reaches Module1.140 (USB3-0-TX_N)
- net USB3-0-TX_P: now reaches Module1.142 (USB3-0-TX_P)
- net HDMI1_HOTPLUG: now reaches Module1.143 (HDMI1_HOTPLUG)
- net HDMI1_SDA: now reaches Module1.145 (HDMI1_SDA)
- net HDMI1_D2_P: now reaches Module1.146 (HDMI1_TX2_P)
- net HDMI1_SCL: now reaches Module1.147 (HDMI1_SCL)
- net HDMI1_D2_N: now reaches Module1.148 (HDMI1_TX2_N)
- net HDMI1_CEC: now reaches Module1.149 (HDMI1_CEC)
- net HDMI0_CEC: now reaches Module1.151 (HDMI0_CEC)
- net HDMI1_D1_P: now reaches Module1.152 (HDMI1_TX1_P)
- net HDMI0_HOTPLUG: now reaches Module1.153 (HDMI0_HOTPLUG)
- net HDMI1_D1_N: now reaches Module1.154 (HDMI1_TX1_N)
- net USB3-1-RX_N: now reaches Module1.157 (USB3-1-RX_N)
- net HDMI1_D0_P: now reaches Module1.158 (HDMI1_TX0_P)
- net USB3-1-RX_P: now reaches Module1.159 (USB3-1-RX_P)
- net HDMI1_D0_N: now reaches Module1.160 (HDMI1_TX0_N)
- net USB3-1-D_P: now reaches Module1.163 (USB3-1-D_P)
- net HDMI1_CK_P: now reaches Module1.164 (HDMI1_CLK_P)
- net USB3-1-D_N: now reaches Module1.165 (USB3-1-D_N)
- net HDMI1_CK_N: now reaches Module1.166 (HDMI1_CLK_N)
- net USB3-1-TX_N: now reaches Module1.169 (USB3-1-TX_N)
- net HDMI0_D2_P: now reaches Module1.170 (HDMI0_TX2_P)
- net USB3-1-TX_P: now reaches Module1.171 (USB3-1-TX_P)
- net HDMI0_D2_N: now reaches Module1.172 (HDMI0_TX2_N)
- net HDMI0_D1_P: now reaches Module1.176 (HDMI0_TX1_P)
- net HDMI0_D1_N: now reaches Module1.178 (HDMI0_TX1_N)
- net HDMI0_D0_P: now reaches Module1.182 (HDMI0_TX0_P)
- net HDMI0_D0_N: now reaches Module1.184 (HDMI0_TX0_N)
- net HDMI0_CK_P: now reaches Module1.188 (HDMI0_CLK_P)
- net HDMI0_CK_N: now reaches Module1.190 (HDMI0_CLK_N)
- net HDMI0_SDA: now reaches Module1.199 (HDMI0_SDA)
- net HDMI0_SCL: now reaches Module1.200 (HDMI0_SCL)
- no-connect marks 1 -> 0
Other:
- note removed: "DSI1/CSI1 Connectors"
- moved on the sheet: J6

Commit message: all
Connections:
- net CAM_GPIO0: no longer J6.17 (Pin_17)
- net CAM_GPIO1: no longer J6.18 (Pin_18)
- no-connect marks 0 -> 2

Commit message: all
Parts:
- J6: mouser (none) -> 798-FH12-22S-0.5SH55
Changed lines of the file:
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@@
+			)
+		)
+		(property "mouser" "798-FH12-22S-0.5SH55"
+			(at 242.57 91.44 0)
+			(hide yes)
+			(show_name no)
+			(do_not_autoplace no)
+			(effects
+				(font
+					(size 1.27 1.27)
+				)
 			)
 		)

Commit message: all
Parts:
- Module1: mouser (none) -> 798-DF40C100DS0.4V58
- renumbered J6 to J1
Connections:
- no-connect marks 2 -> 50
Changed lines of the file:
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@@
+	)
+	(no_connect
+		(at 39.37 157.48)
+	)
+	(no_connect
+		(at 38.1 68.58)
+	)
+	(no_connect
+		(at 133.35 129.54)
+	)
+	(no_connect
+		(at 133.35 137.16)
+	)
+	(no_connect
+		(at 39.37 76.2)
+	)
+	(no_connect
+		(at 39.37 152.4)
+	)
+	(no_connect
+		(at 133.35 96.52)
+	)
+	(no_connect
+		(at 39.37 99.06)
+	)
+	(no_connect
+		(at 39.37 83.82)
+	)
+	(no_connect
+		(at 39.37 111.76)
+	)
+	(no_connect
+		(at 133.35 114.3)
+	)
+	(no_connect
+		(at 39.37 134.62)
+	)
+	(no_connect
+		(at 133.35 134.62)
+	)
+	(no_connect
+		(at 133.35 111.76)
+	)
+	(no_connect
+		(at 229.87 106.68)
+	)
+	(no_connect
+		(at 229.87 109.22)
+	)
+	(no_connect
+		(at 133.35 142.24)
+	)
+	(no_connect
+		(at 39.37 121.92)
+	)
+	(no_connect
+		(at 133.35 104.14)
+	)
+	(no_connect
+		(at 133.35 119.38)
+	)
+	(no_connect
+		(at 133.35 91.44)
+	)
+	(no_connect
+		(at 39.37 142.24)
+	)
+	(no_connect
+		(at 39.37 73.66)
+	)
+	(no_connect
+		(at 133.35 121.92)
+	)
+	(no_connect
+		(at 133.35 127)
+	)
+	(no_connect
+		(at 39.37 129.54)
+	)
+	(no_connect
+		(at 39.37 91.44)
+	)
+	(no_connect
+		(at 39.37 104.14)
+	)
+	(no_connect
+		(at 39.37 114.3)
 	)
 	(no_connect
@@
 	)
 	(no_connect
+		(at 39.37 144.78)
+	)
+	(no_connect
+		(at 133.35 106.68)
+	)
+	(no_connect
+		(at 39.37 106.68)
+	)
+	(no_connect
+		(at 39.37 137.16)
+	)
+	(no_connect
+		(at 39.37 81.28)
+	)
+	(no_connect
+		(at 39.37 119.38)
+	)
+	(no_connect
 		(at 237.49 106.68)
+	)
+	(no_connect
+		(at 133.35 88.9)
+	)
+	(no_connect
+		(at 133.35 99.06)
+	)
+	(no_connect
+		(at 39.37 149.86)
+	)
+	(no_connect
+		(at 133.35 149.86)
+	)
+	(no_connect
+		(at 38.1 66.04)
+	)
+	(no_connect
+		(at 133.35 157.48)
+	)
+	(no_connect
+		(at 133.35 93.98)
+	)
+	(no_connect
+		(at 133.35 144.78)
+	)
+	(no_connect
+		(at 39.37 88.9)
+	)
+	(no_connect
+		(at 133.35 86.36)
+	)
+	(no_connect
+		(at 39.37 127)
+	)
+	(no_connect
+		(at 39.37 96.52)
+	)
+	(no_connect
+		(at 133.35 152.4)
 	)
 	(wire
@@
 		(in_pos_files yes)
 		(dnp no)
-		(property "Reference" "#PWR0130"
+		(property "Reference" "#PWR012"
 			(at 119.38 166.37 0)
 			(hide yes)
@@
 			(project "KB-01"
 				(path "/e6144e29-1dc4-45a8-93e7-988a20131b94/c056c83f-0013-49c8-b531-d86fefdb5c46"
-					(reference "#PWR0130")
+					(reference "#PWR012")
 					(unit 1)
 				)
@@
 		(in_pos_files yes)
 		(dnp no)
-		(property "Reference" "#PWR0131"
+		(property "Reference" "#PWR011"
 			(at 53.34 166.37 0)
 			(hide yes)
@@
 			(project "KB-01"
 				(path "/e6144e29-1dc4-45a8-93e7-988a20131b94/c056c83f-0013-49c8-b531-d86fefdb5c46"
-					(reference "#PWR0131")
+					(reference "#PWR011")
 					(unit 1)
 				)
@@
 		(in_pos_files yes)
 		(dnp no)
-		(property "Reference" "#PWR0134"
+		(property "Reference" "#PWR010"
 			(at 234.95 127 0)
 			(hide yes)
@@
 			(project "KB-01"
 				(path "/e6144e29-1dc4-45a8-93e7-988a20131b94/c056c83f-0013-49c8-b531-d86fefdb5c46"
-					(reference "#PWR0134")
+					(reference "#PWR010")
 					(unit 1)
 				)
@@
 		(in_pos_files yes)
 		(dnp no)
-		(property "Reference" "J6"
+		(property "Reference" "J1"
 			(at 219.71 62.23 0)
 			(show_name no)
@@
 			(project "KB-01"
 				(path "/e6144e29-1dc4-45a8-93e7-988a20131b94/c056c83f-0013-49c8-b531-d86fefdb5c46"
-					(reference "J6")
+					(reference "J1")
 					(unit 1)
 				)
@@
 			(at -53.34 93.98 0)
 			(hide yes)
+			(show_name no)
+			(do_not_autoplace no)
+			(effects
+				(font
+					(size 1.27 1.27)
+				)
+			)
+		)
+		(property "mouser" "798-DF40C100DS0.4V58 "
+			(at -53.34 93.98 0)
+			(hide yes)
