File: KB-01_kicad/KB-01/CM5_high_speed.kicad_sch (KiCad schematic)
At the start: 2 parts, among them J1 Conn_01x22_Female

Commit message: all
Parts:
- J1: value Conn_01x22_Female -> Conn_01x22_MountingPin; footprint CM5IO:Hirose_FH12-22S-0.5SH_1x22-1MP_P0.50mm_Horizontal -> (none); symbol Connector:Conn_01x22_Socket -> Connector_Generic_MountingPin:Conn_01x22_MountingPin; Field4 Mouser -> (none); Field5 798-FH12-22S-0.5SH55 -> (none); Field6 FH12-22S-0.5SH55 -> (none); Field7 Hirose -> (none); Part Description 22 Position FFC, FPC Connector Contacts, Bottom 0.020" (0.5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 -> (none); mouser 798-FH12-22S-0.5SH55 -> (none)
Connections:
- net GND: now also J1.MP (MountPin)
Changed lines of the file:
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@@
+	)
+	(junction
+		(at 234.95 111.76)
+		(diameter 0)
+		(color 0 0 0 0)
 	)
 	(junction
@@
 	)
 	(junction
-		(at 234.95 111.76)
-		(diameter 1.016)
+		(at 234.95 124.46)
+		(diameter 0)
 		(color 0 0 0 0)
 	)
@@
 	(wire
 		(pts
+			(xy 234.95 124.46) (xy 242.57 124.46)
+		)
+		(stroke
+			(width 0)
+			(type default)
+		)
+	)
+	(wire
+		(pts
 			(xy 119.38 101.6) (xy 119.38 109.22)
 		)
@@
 	(wire
 		(pts
+			(xy 234.95 124.46) (xy 234.95 129.54)
+		)
+		(stroke
+			(width 0)
+			(type solid)
+		)
+	)
+	(wire
+		(pts
 			(xy 237.49 66.04) (xy 234.95 66.04)
 		)
@@
 	(wire
 		(pts
-			(xy 234.95 111.76) (xy 234.95 120.65)
+			(xy 234.95 111.76) (xy 234.95 124.46)
 		)
 		(stroke
@@
 	(polyline
 		(pts
-			(xy 208.915 55.88) (xy 208.915 127.635)
+			(xy 208.915 55.88) (xy 208.28 137.16)
 		)
 		(stroke
@@
 	(polyline
 		(pts
-			(xy 254 127.635) (xy 208.915 127.635)
+			(xy 254 137.16) (xy 208.28 137.16)
 		)
 		(stroke
@@
 	(polyline
 		(pts
-			(xy 208.915 127.635) (xy 254 127.635)
+			(xy 254 128.27) (xy 254 137.16)
 		)
 		(stroke
@@
 	(symbol
 		(lib_id "power:GND")
-		(at 234.95 120.65 0)
+		(at 234.95 129.54 0)
 		(unit 1)
 		(body_style 1)
@@
 		(dnp no)
 		(property "Reference" "#PWR010"
-			(at 234.95 127 0)
+			(at 234.95 135.89 0)
 			(hide yes)
 			(show_name no)
@@
 		)
 		(property "Value" "GND"
-			(at 235.077 125.0442 0)
+			(at 235.077 133.9342 0)
 			(show_name no)
 			(do_not_autoplace no)
@@
 		)
 		(property "Footprint" ""
-			(at 234.95 120.65 0)
+			(at 234.95 129.54 0)
 			(hide yes)
 			(show_name no)
@@
 		)
 		(property "Datasheet" ""
-			(at 234.95 120.65 0)
+			(at 234.95 129.54 0)
 			(hide yes)
 			(show_name no)
@@
 		)
 		(property "Description" "Power symbol creates a global label with name \"GND\" , ground"
-			(at 234.95 120.65 0)
+			(at 234.95 129.54 0)
 			(hide yes)
 			(show_name no)
@@
 	)
 	(symbol
-		(lib_id "Connector:Conn_01x22_Socket")
+		(lib_id "Connector_Generic_MountingPin:Conn_01x22_MountingPin")
 		(at 242.57 91.44 0)
 		(unit 1)
@@
 		(dnp no)
 		(property "Reference" "J1"
-			(at 219.71 62.23 0)
+			(at 242.57 63.5 0)
+			(show_name no)
+			(do_not_autoplace no)
+			(effects
+				(font
+					(size 1.27 1.27)
+				)
+			)
+		)
+		(property "Value" "Conn_01x22_MountingPin"
+			(at 245.872 120.396 90)
 			(show_name no)
 			(do_not_autoplace no)
@@
 			)
 		)
-		(property "Value" "Conn_01x22_Female"
-			(at 224.155 62.23 0)
-			(show_name no)
-			(do_not_autoplace no)
-			(effects
-				(font
-					(size 1.27 1.27)
-				)
-				(justify left)
-			)
-		)
-		(property "Footprint" "CM5IO:Hirose_FH12-22S-0.5SH_1x22-1MP_P0.50mm_Horizontal"
+		(property "Footprint" ""
 			(at 242.57 91.44 0)
 			(hide yes)
@@
 			)
 		)
-		(property "Datasheet" "https://www.hirose.com/product/document?clcode=&productname=&series=FH12&documenttype=Catalog&lang=en&documentid=D31648_en"
+		(property "Datasheet" ""
 			(at 242.57 91.44 0)
 			(hide yes)
@@
 			)
 		)
-		(property "Description" ""
+		(property "Description" "Generic connectable mounting pin connector, single row, 01x22, script generated (kicad-library-utils/schlib/autogen/connector/)"
 			(at 242.57 91.44 0)
 			(hide yes)
@@
 			)
 		)
-		(property "Field4" "Mouser"
-			(at 242.57 91.44 0)
-			(hide yes)
-			(show_name no)
-			(do_not_autoplace no)
-			(effects
-				(font
-					(size 1.27 1.27)
-				)
-			)
-		)
-		(property "Field5" "798-FH12-22S-0.5SH55"
-			(at 242.57 91.44 0)
-			(hide yes)
-			(show_name no)
-			(do_not_autoplace no)
-			(effects
-				(font
-					(size 1.27 1.27)
-				)
-			)
-		)
-		(property "Field6" "FH12-22S-0.5SH55"
-			(at 242.57 91.44 0)
-			(hide yes)
-			(show_name no)
-			(do_not_autoplace no)
-			(effects
-				(font
-					(size 1.27 1.27)
-				)
-			)
-		)
-		(property "Field7" "Hirose"
-			(at 242.57 91.44 0)
-			(hide yes)
-			(show_name no)
-			(do_not_autoplace no)
-			(effects
-				(font
-					(size 1.27 1.27)
-				)
-			)
-		)
-		(property "Part Description" "22 Position FFC, FPC Connector Contacts, Bottom 0.020\" (0.50mm) Surface Mount, Right Angle"
-			(at 242.57 91.44 0)
-			(hide yes)
-			(show_name no)
-			(do_not_autoplace no)
-			(effects
-				(font
-					(size 1.27 1.27)
-				)
-			)
-		)
-		(property "mouser" "798-FH12-22S-0.5SH55"
-			(at 242.57 91.44 0)
-			(hide yes)
-			(show_name no)
-			(do_not_autoplace no)
-			(effects
-				(font
-					(size 1.27 1.27)
-				)
-			)
-		)
-		(property "SNAPEDA_PN" ""
-			(at 242.57 91.44 0)
-			(hide yes)
-			(show_name no)
-			(do_not_autoplace no)
-			(effects
-				(font
-					(size 1.27 1.27)
-				)
-			)
-		)
 		(pin "1"
 		)
@@
 		(pin "9"
 		)
+		(pin "MP"
+		)
 		(instances

Commit message: all
Parts:
- added J13: Conn_01x22_MountingPin, CM5IO:Hirose_FH12-22S-0.5SH_1x22-1MP_P0.50mm_Horizontal, symbol Connector_Generic_MountingPin:Conn_01x22_MountingPin
- added R37, R38: 2.2K 1%, Resistor_SMD:R_0603_1608Metric_Pad0.98x0.95mm_HandSolder, symbol Device:R
- J1: footprint (none) -> CM5IO:Hirose_FH12-22S-0.5SH_1x22-1MP_P0.50mm_Horizontal
Connections:
- net +3.3v: now also J13.22 (Pin_22), R37.1, R38.1
- net CAM_GPIO0: now also J13.17 (Pin_17)
- net DPHY1_C_N: now also J13.8 (Pin_8)
- net DPHY1_C_P: now also J13.9 (Pin_9)
- net DPHY1_D0_N: now also J13.2 (Pin_2)
- net DPHY1_D0_P: now also J13.3 (Pin_3)
- net DPHY1_D1_N: now also J13.5 (Pin_5)
- net DPHY1_D1_P: now also J13.6 (Pin_6)
- net DPHY1_D2_N: now also J13.11 (Pin_11)
- net DPHY1_D2_P: now also J13.12 (Pin_12)
- net DPHY1_D3_N: now also J13.14 (Pin_14)
- net DPHY1_D3_P: now also J13.15 (Pin_15)
- net GND: now also J13.1 (Pin_1), J13.10 (Pin_10), J13.13 (Pin_13), J13.16 (Pin_16), J13.19 (Pin_19), J13.4 (Pin_4), J13.7 (Pin_7), J13.MP (MountPin)
- new net ID_SC: J13.20 (Pin_20), R38.2
- new net ID_SD: J13.21 (Pin_21), R37.2
- no-connect marks 50 -> 49
Other:
- note added: "CSI1 Connectors"
- note added: "DSI0 Connectors"
- note removed: "DSI0/CSI0 Connectors"
- moved on the sheet: J1
