File: KB-01_kicad/KB-01/CM5_high_speed.kicad_sch (KiCad schematic)
At the start: 5 parts, among them J1 Conn_01x22_MountingPin, J13 Conn_01x22_MountingPin

Commit message: all
Parts:
- added H1, H2, H3, H4: MountingHole, MountingHole:MountingHole_2.7mm_M2.5_DIN965, symbol Mechanical:MountingHole
- J1: waveshare (none) -> https://www.waveshare.com/wiki/3.5inch_DSI_LCD_(E)

Commit message: all
Parts:
- Module1: mouser 798-DF40C100DS0.4V58 -> 649-101642271004RLF
Changed lines of the file:
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@@
 			)
 		)
-		(property "mouser" "798-DF40C100DS0.4V58 "
+		(property "mouser" "649-101642271004RLF "
 			(at -53.34 93.98 0)
 			(hide yes)
