File: KB-01_kicad/KB-01/sensors.kicad_sch (KiCad schematic)
At the start: 3 parts, among them U9 BMI270

Commit message: up
Parts:
- added C37, C38, C39, C41, C42: 100nF, Capacitor_SMD:C_0603_1608Metric_Pad1.08x0.95mm_HandSolder, symbol Device:C
- added C40: 220nF, Capacitor_SMD:C_0603_1608Metric_Pad1.08x0.95mm_HandSolder, symbol Device:C
- added U10: LIS2MDL, Package_LGA:LGA-12_2x2mm_P0.5mm, symbol Sensor_Magnetic:LIS2MDL
- added U11: BMP390L, BMP390L:XDCR_BMP390L, symbol BMP390L:BMP390L
- added U12: SHT40, Sensor_Humidity:Sensirion_DFN-4_1.5x1.5mm_P0.8mm_SHT4x_NoCentralPad, symbol Sensor_Humidity:SHT4x
Connections:
- net +3V3: now also C37.1, C38.1, C39.1, C41.1, C42.1, U10.10 (Vdd_IO), U10.3 (~{CS}), U10.9 (Vdd), U11.1 (VDDIO), U11.10 (VDD), U11.5 (SDO/DNC/SA0), U11.6 (~{CS}), U12.3 (VDD)
- net GND: now also C37.2, C38.2, C39.2, C40.2, C41.2, C42.2, U10.6 (GND), U10.8 (GND), U11.3 (VSS/GND), U11.8 (VSS/GND), U11.9 (VSS/GND), U12.4 (VSS)
- new net: C40.1, U10.5 (C1)
- new net BMP390_INT: U11.7 (INT/DNC)
- new net BMP390_SCK: U11.2 (SCK/SCL)
- new net BMP390_SDA: U11.4 (SDI/SDO/SDA)
- new net LIS2MDL_INT: U10.7 (DRDY)
- new net LIS2MDL_SCL: U10.1 (SCL/SPC)
- new net LIS2MDL_SDA: U10.4 (SDA/SDI/SDO)
- new net SHT40_SCK: U12.2 (SCL)
- new net SHT40_SDA: U12.1 (SDA)
Other:
- note added: "Barometer, I2C"
- note added: "Close as possible pin 5 and 6 Use low ESR (max 200 mOhm)"
- note added: "IMU, SPI"
- note added: "Magnetometer, I2C"
- note added: "Temp and humidity, I2C"
- note removed: "IMU"

Commit message: up
Connections:
- net +3V3 renamed +3.3v

Commit message: all
Parts:
- added C50: 0.1uF, symbol Device:C
- added J7: DRV5023AJ, Connector_Audio:Jack_3.5mm_CUI_SJ-3523-SMT_Horizontal, symbol Connector_Audio:AudioJack3
- added R29: 10k, symbol Device:R
Connections:
- net GND: now also C50.2, J7.T
- new net +3.3V: C50.1, J7.R, R29.1
- new net Wheel_sensor: J7.S, R29.2
Other:
- note added: "Hall effect Sensor Wheel speed"

Commit message: all
Parts:
- C50: value 0.1uF -> 0.1uF 10V; footprint (none) -> Capacitor_SMD:C_0603_1608Metric_Pad1.08x0.95mm_HandSolder; mouser (none) -> 963-LMF107B7104KAHT

Commit message: all
Connections:
- net +3.3V is gone; now on net +3.3v: C50.1, J7.R, R29.1
Changed lines of the file:
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@@
+		)
+	)
+	(hierarchical_label "+3.3v"
+		(shape output)
+		(at 149.86 91.44 0)
+		(effects
+			(font
+				(size 1.27 1.27)
+			)
+			(justify left)
 		)
 	)
@@
 		(shape output)
 		(at 64.77 106.68 0)
+		(effects
+			(font
+				(size 1.27 1.27)
+			)
+			(justify left)
+		)
+	)
+	(hierarchical_label "+3.3v"
+		(shape output)
+		(at 173.99 104.14 0)
 		(effects
 			(font
@@
 	)
 	(symbol
-		(lib_id "power:+3.3V")
-		(at 173.99 104.14 0)
-		(unit 1)
-		(body_style 1)
-		(exclude_from_sim no)
-		(in_bom yes)
-		(on_board yes)
-		(in_pos_files yes)
-		(dnp no)
-		(fields_autoplaced yes)
-		(property "Reference" "#PWR076"
-			(at 173.99 107.95 0)
-			(hide yes)
-			(show_name no)
-			(do_not_autoplace no)
-			(effects
-				(font
-					(size 1.27 1.27)
-				)
-			)
-		)
-		(property "Value" "+3.3V"
-			(at 173.99 99.06 0)
-			(show_name no)
-			(do_not_autoplace no)
-			(effects
-				(font
-					(size 1.27 1.27)
-				)
-			)
-		)
-		(property "Footprint" ""
-			(at 173.99 104.14 0)
-			(hide yes)
-			(show_name no)
-			(do_not_autoplace no)
-			(effects
-				(font
-					(size 1.27 1.27)
-				)
-			)
-		)
-		(property "Datasheet" ""
-			(at 173.99 104.14 0)
-			(hide yes)
-			(show_name no)
-			(do_not_autoplace no)
-			(effects
-				(font
-					(size 1.27 1.27)
-				)
-			)
-		)
-		(property "Description" "Power symbol creates a global label with name \"+3.3V\""
-			(at 173.99 104.14 0)
-			(hide yes)
-			(show_name no)
-			(do_not_autoplace no)
-			(effects
-				(font
-					(size 1.27 1.27)
-				)
-			)
-		)
-		(pin "1"
-		)
-		(instances
-			(project "KB-01"
-				(path "/e6144e29-1dc4-45a8-93e7-988a20131b94/8f8a2829-aad0-4226-9c36-d614fdf3c6c8"
-					(reference "#PWR076")
-					(unit 1)
-				)
-			)
-		)
-	)
-	(symbol
 		(lib_id "BMI270:BMI270")
 		(at 62.23 58.42 0)
@@
 					(unit 1)
 				)
-			)
-		)
-	)
-	(symbol
-		(lib_id "power:+3.3V")
-		(at 149.86 91.44 0)
-		(unit 1)
-		(body_style 1)
-		(exclude_from_sim no)
-		(in_bom yes)
-		(on_board yes)
-		(in_pos_files yes)
-		(dnp no)
-		(fields_autoplaced yes)
-		(property "Reference" "#PWR079"
-			(at 149.86 95.25 0)
-			(hide yes)
-			(show_name no)
-			(do_not_autoplace no)
-			(effects
-				(font
-					(size 1.27 1.27)
-				)
-			)
-		)
-		(property "Value" "+3.3V"
-			(at 149.86 86.36 0)
-			(show_name no)
-			(do_not_autoplace no)
-			(effects
-				(font
-					(size 1.27 1.27)
-				)
-			)
-		)
-		(property "Footprint" ""
-			(at 149.86 91.44 0)
-			(hide yes)
-			(show_name no)
-			(do_not_autoplace no)
-			(effects
-				(font
-					(size 1.27 1.27)
-				)
-			)
-		)
-		(property "Datasheet" ""
-			(at 149.86 91.44 0)
-			(hide yes)
-			(show_name no)
-			(do_not_autoplace no)
-			(effects
-				(font
-					(size 1.27 1.27)
-				)
-			)
-		)
-		(property "Description" "Power symbol creates a global label with name \"+3.3V\""
-			(at 149.86 91.44 0)
-			(hide yes)
-			(show_name no)
-			(do_not_autoplace no)
-			(effects
-				(font
-					(size 1.27 1.27)
-				)
-			)
-		)
-		(pin "1"
-		)
-		(instances
-			(project "KB-01"
-				(path "/e6144e29-1dc4-45a8-93e7-988a20131b94/8f8a2829-aad0-4226-9c36-d614fdf3c6c8"
-					(reference "#PWR079")
-					(unit 1)
-				)

Commit message: all
Parts:
- removed C41: 100nF, Capacitor_SMD:C_0603_1608Metric_Pad1.08x0.95mm_HandSolder, symbol Device:C
- removed U11: BMP390L, BMP390L:XDCR_BMP390L, symbol BMP390L:BMP390L
- added C52, C53: 100nF 6.3V, Capacitor_SMD:C_0603_1608Metric_Pad1.08x0.95mm_HandSolder, symbol Device:C
- added J9: AudioJack3_SwitchTR, Connector_Audio:Jack_3.5mm_CUI_SJ2-3593D-SMT_Horizontal, symbol Connector_Audio:AudioJack3_SwitchTR
- added U13: BMP581, BMP581:BMP581, symbol BMP581:BMP581
- C35, C36, C37, C38, C42: value 100nF -> 100nF 6.3V; mouser (none) -> 581-KGM15AR70J104KT
- C39: value 100nF -> 10uF 6.3V; mouser (none) -> 81-GRM188R60J106ME47
- C40: value 220nF -> 220nF 25V; mouser (none) -> 187-CL10B224KA8NNNC
- J7: mouser (none) -> 595-DRV5023AJELPGMQ1
- R29: footprint (none) -> Resistor_SMD:R_0603_1608Metric_Pad0.98x0.95mm_HandSolder; mouser (none) -> 71-CRCW060310K0FKEE
- U10: mouser (none) -> 511-LIS2MDLTR; mouser2 (none) -> 511-IIS2MDCTR
- U12: mouser (none) -> 403-SHT40-AD1B-R2
- U9: footprint BMI270:XDCR_BMI270 -> BMI270:BMI270; mouser (none) -> 262-BMI270
Connections:
- net +3.3v: now also C52.2, C53.1, J9.R, J9.RN, U13.1 (VDDIO), U13.10 (VDD), U13.5 (SDO), U13.6 (CSB); no longer J7.R
- net BMP390_INT: now also U13.7 (INT)
- net BMP390_SCK: now also U13.2 (SCK)
- net BMP390_SDA: now also U13.4 (SDI)
- net GND: now also C52.1, C53.2, J9.T, J9.TN, U13.3 (VSS_1), U13.8 (VSS_2), U13.9 (VSS_3); no longer J7.T
- net Wheel_sensor: now also J9.S; no longer J7.S
Other:
- note added: "IMU, 4-wire SPI"
- note removed: "IMU, SPI"
- moved on the sheet: U12

Commit message: all
Parts:
- renumbered C52 to C43, C35 to C44, C36 to C45, C42 to C46, C50 to C47, C37 to C48, C39 to C49, C38 to C50, C53 to C51, C40 to C52, J7 to J10, R29 to R25, U13 to U11, U9 to U12, U12 to U13, U10 to U14
Connections:
- no-connect marks 4 -> 7
Changed lines of the file:
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@@
 	)
 	(no_connect
+		(at 129.54 127)
+	)
+	(no_connect
 		(at 46.99 66.04)
 	)
 	(no_connect
+		(at 129.54 129.54)
+	)
+	(no_connect
+		(at 129.54 124.46)
+	)
+	(no_connect
 		(at 46.99 68.58)
 	)
@@
 		(dnp no)
 		(fields_autoplaced yes)
-		(property "Reference" "#PWR047"
+		(property "Reference" "#PWR077"
 			(at 40.64 128.27 0)
 			(hide yes)
@@
 			(project "KB-01"
 				(path "/e6144e29-1dc4-45a8-93e7-988a20131b94/8f8a2829-aad0-4226-9c36-d614fdf3c6c8"
-					(reference "#PWR047")
+					(reference "#PWR077")
 					(unit 1)
 				)
@@
 		(in_pos_files yes)
 		(dnp no)
-		(property "Reference" "C39"
+		(property "Reference" "C49"
 			(at 49.022 115.57 0)
 			(show_name no)
@@
 			(project "KB-01"
 				(path "/e6144e29-1dc4-45a8-93e7-988a20131b94/8f8a2829-aad0-4226-9c36-d614fdf3c6c8"
-					(reference "C39")
+					(reference "C49")
 					(unit 1)
 				)
@@
 		(dnp no)
 		(fields_autoplaced yes)
-		(property "Reference" "#PWR044"
+		(property "Reference" "#PWR071"
 			(at 91.44 58.42 0)
 			(hide yes)
@@
 			(project "KB-01"
 				(path "/e6144e29-1dc4-45a8-93e7-988a20131b94/8f8a2829-aad0-4226-9c36-d614fdf3c6c8"
-					(reference "#PWR044")
+					(reference "#PWR071")
 					(unit 1)
 				)
@@
 		(dnp no)
 		(fields_autoplaced yes)
-		(property "Reference" "U9"
+		(property "Reference" "U12"
 			(at 62.23 33.02 0)
 			(show_name no)
@@
 			(project "KB-01"
 				(path "/e6144e29-1dc4-45a8-93e7-988a20131b94/8f8a2829-aad0-4226-9c36-d614fdf3c6c8"
-					(reference "U9")
+					(reference "U12")
 					(unit 1)
 				)
@@
 		(dnp no)
 		(fields_autoplaced yes)
-		(property "Reference" "C42"
+		(property "Reference" "C46"
 			(at 177.8 62.2299 0)
 			(show_name no)
@@
 			(project "KB-01"
 				(path "/e6144e29-1dc4-45a8-93e7-988a20131b94/8f8a2829-aad0-4226-9c36-d614fdf3c6c8"
-					(reference "C42")
+					(reference "C46")
 					(unit 1)
 				)
@@
 		(dnp no)
 		(fields_autoplaced yes)
-		(property "Reference" "#PWR070"
+		(property "Reference" "#PWR072"
 			(at 173.99 76.2 0)
 			(hide yes)
@@
 			(project "KB-01"
 				(path "/e6144e29-1dc4-45a8-93e7-988a20131b94/8f8a2829-aad0-4226-9c36-d614fdf3c6c8"
-					(reference "#PWR070")
+					(reference "#PWR072")
 					(unit 1)
 				)
@@
 		(dnp no)
 		(fields_autoplaced yes)
-		(property "Reference" "C50"
+		(property "Reference" "C47"
 			(at 162.56 106.6799 0)
 			(show_name no)
@@
 			(project "KB-01"
 				(path "/e6144e29-1dc4-45a8-93e7-988a20131b94/8f8a2829-aad0-4226-9c36-d614fdf3c6c8"
-					(reference "C50")
+					(reference "C47")
 					(unit 1)
 				)
@@
 		(dnp no)
 		(fields_autoplaced yes)
-		(property "Reference" "C38"
+		(property "Reference" "C50"
 			(at 88.9 114.2999 0)
 			(show_name no)
@@
 			(project "KB-01"
 				(path "/e6144e29-1dc4-45a8-93e7-988a20131b94/8f8a2829-aad0-4226-9c36-d614fdf3c6c8"
-					(reference "C38")
+					(reference "C50")
 					(unit 1)
 				)
@@
 		(dnp no)
 		(fields_autoplaced yes)
-		(property "Reference" "U13"
+		(property "Reference" "U11"
 			(at 213.36 49.4598 0)
 			(show_name no)
@@
 			(project "KB-01"
 				(path "/e6144e29-1dc4-45a8-93e7-988a20131b94/8f8a2829-aad0-4226-9c36-d614fdf3c6c8"
-					(reference "U13")
+					(reference "U11")
 					(unit 1)
 				)
@@
 		(dnp no)
 		(fields_autoplaced yes)
-		(property "Reference" "#PWR077"
+		(property "Reference" "#PWR069"
 			(at 213.36 44.45 0)
 			(hide yes)
@@
 			(project "KB-01"
 				(path "/e6144e29-1dc4-45a8-93e7-988a20131b94/8f8a2829-aad0-4226-9c36-d614fdf3c6c8"
-					(reference "#PWR077")
+					(reference "#PWR069")
 					(unit 1)
 				)
@@
 		(in_pos_files yes)
 		(dnp no)
-		(property "Reference" "U12"
+		(property "Reference" "U13"
 			(at 223.52 116.078 0)
 			(show_name no)
@@
 			(project "KB-01"
 				(path "/e6144e29-1dc4-45a8-93e7-988a20131b94/8f8a2829-aad0-4226-9c36-d614fdf3c6c8"
-					(reference "U12")
+					(reference "U13")
 					(unit 1)
 				)
@@
 		(dnp no)
 		(fields_autoplaced yes)
-		(property "Reference" "#PWR050"
+		(property "Reference" "#PWR080"
 			(at 81.28 157.48 0)
 			(hide yes)
@@
 			(project "KB-01"
 				(path "/e6144e29-1dc4-45a8-93e7-988a20131b94/8f8a2829-aad0-4226-9c36-d614fdf3c6c8"
-					(reference "#PWR050")
+					(reference "#PWR080")
 					(unit 1)
 				)
@@
 		(dnp no)
 		(fields_autoplaced yes)
-		(property "Reference" "#PWR045"
+		(property "Reference" "#PWR073"
 			(at 81.28 86.36 0)
 			(hide yes)
@@
 			(project "KB-01"
 				(path "/e6144e29-1dc4-45a8-93e7-988a20131b94/8f8a2829-aad0-4226-9c36-d614fdf3c6c8"
-					(reference "#PWR045")
+					(reference "#PWR073")
 					(unit 1)
 				)
@@
 		(dnp no)
 		(fields_autoplaced yes)
-		(property "Reference" "C40"
+		(property "Reference" "C52"
 			(at 85.09 138.4299 0)
 			(show_name no)
@@
 			(project "KB-01"
 				(path "/e6144e29-1dc4-45a8-93e7-988a20131b94/8f8a2829-aad0-4226-9c36-d614fdf3c6c8"
-					(reference "C40")
+					(reference "C52")
 					(unit 1)
 				)
@@
 		(dnp no)
 		(fields_autoplaced yes)
-		(property "Reference" "C35"
+		(property "Reference" "C44"
 			(at 88.9 43.1799 0)
 			(show_name no)
@@
 			(project "KB-01"
 				(path "/e6144e29-1dc4-45a8-93e7-988a20131b94/8f8a2829-aad0-4226-9c36-d614fdf3c6c8"
-					(reference "C35")
+					(reference "C44")
 					(unit 1)
 				)
@@
 		(dnp no)
 		(fields_autoplaced yes)
-		(property "Reference" "#PWR046"
+		(property "Reference" "#PWR079"
 			(at 66.04 157.48 0)
 			(hide yes)
@@
 			(project "KB-01"
 				(path "/e6144e29-1dc4-45a8-93e7-988a20131b94/8f8a2829-aad0-4226-9c36-d614fdf3c6c8"
-					(reference "#PWR046")
+					(reference "#PWR079")
 					(unit 1)
 				)
@@
 		(dnp no)
 		(fields_autoplaced yes)
-		(property "Reference" "C52"
+		(property "Reference" "C43"
 			(at 189.23 27.94 90)
 			(show_name no)
@@
 			(project "KB-01"
 				(path "/e6144e29-1dc4-45a8-93e7-988a20131b94/8f8a2829-aad0-4226-9c36-d614fdf3c6c8"
-					(reference "C52")
+					(reference "C43")
 					(unit 1)
 				)
@@
 		(dnp no)
 		(fields_autoplaced yes)
-		(property "Reference" "C36"
+		(property "Reference" "C45"
 			(at 101.6 43.1799 0)
 			(show_name no)
@@
 			(project "KB-01"
 				(path "/e6144e29-1dc4-45a8-93e7-988a20131b94/8f8a2829-aad0-4226-9c36-d614fdf3c6c8"
-					(reference "C36")
+					(reference "C45")
 					(unit 1)
 				)
@@
 		(dnp no)
 		(fields_autoplaced yes)
-		(property "Reference" "#PWR056"
+		(property "Reference" "#PWR078"
 			(at 233.68 146.05 0)
 			(hide yes)
@@
 			(project "KB-01"
 				(path "/e6144e29-1dc4-45a8-93e7-988a20131b94/8f8a2829-aad0-4226-9c36-d614fdf3c6c8"
-					(reference "#PWR056")
+					(reference "#PWR078")
 					(unit 1)
 				)
@@
 		(in_pos_files yes)
 		(dnp no)
-		(property "Reference" "U10"
+		(property "Reference" "U14"
 			(at 71.12 116.078 0)
 			(show_name no)
@@
 			(project "KB-01"
 				(path "/e6144e29-1dc4-45a8-93e7-988a20131b94/8f8a2829-aad0-4226-9c36-d614fdf3c6c8"
-					(reference "U10")
+					(reference "U14")
 					(unit 1)
 				)
@@
 		(dnp no)
 		(fields_autoplaced yes)
-		(property "Reference" "R29"
+		(property "Reference" "R25"
 			(at 152.4 95.2499 0)
 			(show_name no)
@@
 			(project "KB-01"
 				(path "/e6144e29-1dc4-45a8-93e7-988a20131b94/8f8a2829-aad0-4226-9c36-d614fdf3c6c8"
-					(reference "R29")
+					(reference "R25")
 					(unit 1)
 				)
@@
 		(dnp no)
 		(fields_autoplaced yes)
-		(property "Reference" "J7"
+		(property "Reference" "J10"
 			(at 122.555 118.11 0)
 			(show_name no)
@@
 			(project "KB-01"
 				(path "/e6144e29-1dc4-45a8-93e7-988a20131b94/8f8a2829-aad0-4226-9c36-d614fdf3c6c8"
-					(reference "J7")
+					(reference "J10")
 					(unit 1)
 				)
@@
 		(dnp no)
 		(fields_autoplaced yes)
-		(property "Reference" "#PWR073"
+		(property "Reference" "#PWR074"
 			(at 193.04 86.36 0)
 			(hide yes)
@@
 			(project "KB-01"
 				(path "/e6144e29-1dc4-45a8-93e7-988a20131b94/8f8a2829-aad0-4226-9c36-d614fdf3c6c8"
-					(reference "#PWR073")
+					(reference "#PWR074")
 					(unit 1)
 				)
@@
 		(in_pos_files yes)
 		(dnp no)
-		(property "Reference" "#PWR048"
+		(property "Reference" "#PWR076"
 			(at 85.09 127 0)
 			(hide yes)
@@
 			(project "KB-01"
 				(path "/e6144e29-1dc4-45a8-93e7-988a20131b94/8f8a2829-aad0-4226-9c36-d614fdf3c6c8"
-					(reference "#PWR048")
+					(reference "#PWR076")
 					(unit 1)
 				)
@@
 		(dnp no)
 		(fields_autoplaced yes)
-		(property "Reference" "C37"
+		(property "Reference" "C48"
 			(at 38.1 114.2999 0)
 			(show_name no)
@@
 			(project "KB-01"
 				(path "/e6144e29-1dc4-45a8-93e7-988a20131b94/8f8a2829-aad0-4226-9c36-d614fdf3c6c8"
-					(reference "C37")
+					(reference "C48")
 					(unit 1)
 				)
@@
 		(dnp no)
 		(fields_autoplaced yes)
-		(property "Reference" "C53"
+		(property "Reference" "C51"
 			(at 246.38 125.7299 0)
 			(show_name no)
@@
 			(project "KB-01"
 				(path "/e6144e29-1dc4-45a8-93e7-988a20131b94/8f8a2829-aad0-4226-9c36-d614fdf3c6c8"
-					(reference "C53")
+					(reference "C51")
 					(unit 1)
 				)
@@
 		(dnp no)
 		(fields_autoplaced yes)
-		(property "Reference" "#PWR071"
+		(property "Reference" "#PWR070"
 			(at 182.88 45.72 0)
 			(hide yes)
@@
 			(project "KB-01"
 				(path "/e6144e29-1dc4-45a8-93e7-988a20131b94/8f8a2829-aad0-4226-9c36-d614fdf3c6c8"
-					(reference "#PWR071")
+					(reference "#PWR070")
 					(unit 1)
 				)
