File: KB-01_kicad/KB-01/5v_boost_conv.kicad_sch (KiCad schematic)
At the start: 1 part, among them U2 TPS61022

Commit message: all
Signed-off-by: syauqi-alias <syauqi_nur@yahoo.com>
Parts:
- added C20, C21, C22, C23, C25, C27: 22uF 16V, Capacitor_SMD:C_0603_1608Metric_Pad1.08x0.95mm_HandSolder, symbol Device:C
- added C24: 47uF 16V, Capacitor_SMD:C_0603_1608Metric_Pad1.08x0.95mm_HandSolder, symbol Device:C
- added C26: 0.1uF 16V, Capacitor_SMD:C_0603_1608Metric_Pad1.08x0.95mm_HandSolder, symbol Device:C
- added L3: 1uH 21.8A, Inductor_SMD:L_Coilcraft_XAL7030-102, symbol Device:L
- added R15: 750k, Resistor_SMD:R_0603_1608Metric_Pad0.98x0.95mm_HandSolder, symbol Device:R
- added R16: 100k, Resistor_SMD:R_0603_1608Metric_Pad0.98x0.95mm_HandSolder, symbol Device:R
Connections:
- net GND: now reaches U2.1 (GND)
- net GND: now also C20.2, C21.2, C22.2, C23.2, C24.2, C25.2, C26.2, C27.2, R16.2
- net at U2.2 (SW): now also L3.2
- net +5V: now reaches U2.3 (VOUT)
- net +5V: now also C20.1, C21.1, C22.1, C23.1, C24.1, R15.1
- net at U2.4 (FB): now also R15.2, R16.1
- net BST_EN: now reaches U2.5 (EN)
- net BST_MODE: now reaches U2.6 (MODE)
- net BST_VIN: now reaches U2.7 (VIN)
- net BST_VIN: now also C25.1, C26.1, C27.1, L3.1
Other:
- note added: "5.1V 8A Max"
- moved on the sheet: U2

Commit message: up
Connections:
- net +5V renamed +5v
Changed lines of the file:
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@@
-	(wire
-		(pts
-			(xy 232.41 93.98) (xy 232.41 99.06)
-		)
-		(stroke
-			(width 0)
-			(type default)
-		)
-	)
 	(wire
 		(pts
@@
 		(pts
 			(xy 186.69 114.3) (xy 199.39 114.3)
+		)
+		(stroke
+			(width 0)
+			(type default)
+		)
+	)
+	(wire
+		(pts
+			(xy 232.41 92.71) (xy 232.41 99.06)
 		)
 		(stroke
@@
 			)
 			(justify right)
+		)
+	)
+	(hierarchical_label "+5v"
+		(shape input)
+		(at 232.41 92.71 0)
+		(effects
+			(font
+				(size 1.27 1.27)
+			)
+			(justify left)
 		)
 	)
@@
 					(unit 1)
 				)
-			)
-		)
-	)
-	(symbol
-		(lib_id "power:+5V")
-		(at 232.41 93.98 0)
-		(unit 1)
-		(exclude_from_sim no)
-		(in_bom yes)
-		(on_board yes)
-		(dnp no)
-		(fields_autoplaced yes)
-		(property "Reference" "#PWR028"
-			(at 232.41 97.79 0)
-			(effects
-				(font
-					(size 1.27 1.27)
-				)
-				(hide yes)
-			)
-		)
-		(property "Value" "+5V"
-			(at 232.41 88.9 0)
-			(effects
-				(font
-					(size 1.27 1.27)
-				)
-			)
-		)
-		(property "Footprint" ""
-			(at 232.41 93.98 0)
-			(effects
-				(font
-					(size 1.27 1.27)
-				)
-				(hide yes)
-			)
-		)
-		(property "Datasheet" ""
-			(at 232.41 93.98 0)
-			(effects
-				(font
-					(size 1.27 1.27)
-				)
-				(hide yes)
-			)
-		)
-		(property "Description" "Power symbol creates a global label with name \"+5V\""
-			(at 232.41 93.98 0)
-			(effects
-				(font
-					(size 1.27 1.27)
-				)
-				(hide yes)
-			)
-		)
-		(pin "1"
-		)
-		(instances
-			(project ""
-				(path "/e6144e29-1dc4-45a8-93e7-988a20131b94/f9d53241-b903-4597-892d-d58932656724"
-					(reference "#PWR028")
-					(unit 1)
-				)

Commit message: everything
Connections:
- net BST_EN is gone; now on net BST_VIN: U2.5 (EN)
- net BST_MODE is gone; now on net GND: U2.6 (MODE)
Other:
- moved on the sheet: C25, C26, C27
Changed lines of the file:
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@@
+	)
+	(junction
+		(at 80.01 87.63)
+		(diameter 0)
+		(color 0 0 0 0)
 	)
 	(junction
@@
 	)
 	(junction
-		(at 88.9 95.25)
-		(diameter 0)
-		(color 0 0 0 0)
-	)
-	(junction
 		(at 212.09 99.06)
 		(diameter 0)
@@
 	)
 	(junction
-		(at 115.57 87.63)
+		(at 106.68 87.63)
+		(diameter 0)
+		(color 0 0 0 0)
+	)
+	(junction
+		(at 120.65 87.63)
 		(diameter 0)
 		(color 0 0 0 0)
@@
 	)
 	(junction
-		(at 102.87 87.63)
-		(diameter 0)
-		(color 0 0 0 0)
-	)
-	(junction
 		(at 130.81 87.63)
 		(diameter 0)
@@
 	)
 	(junction
-		(at 102.87 95.25)
+		(at 93.98 95.25)
 		(diameter 0)
 		(color 0 0 0 0)
@@
 	)
 	(junction
-		(at 88.9 87.63)
-		(diameter 0)
-		(color 0 0 0 0)
-	)
-	(junction
 		(at 212.09 114.3)
 		(diameter 0)
@@
 	)
 	(junction
+		(at 135.89 109.22)
+		(diameter 0)
+		(color 0 0 0 0)
+	)
+	(junction
+		(at 80.01 95.25)
+		(diameter 0)
+		(color 0 0 0 0)
+	)
+	(junction
+		(at 93.98 87.63)
+		(diameter 0)
+		(color 0 0 0 0)
+	)
+	(junction
 		(at 158.75 99.06)
 		(diameter 0)
@@
 	(wire
 		(pts
-			(xy 102.87 95.25) (xy 115.57 95.25)
-		)
-		(stroke
-			(width 0)
-			(type default)
-		)
-	)
-	(wire
-		(pts
 			(xy 158.75 116.84) (xy 158.75 120.65)
 		)
@@
 	(wire
 		(pts
+			(xy 93.98 95.25) (xy 106.68 95.25)
+		)
+		(stroke
+			(width 0)
+			(type default)
+		)
+	)
+	(wire
+		(pts
+			(xy 120.65 87.63) (xy 120.65 99.06)
+		)
+		(stroke
+			(width 0)
+			(type default)
+		)
+	)
+	(wire
+		(pts
 			(xy 120.65 99.06) (xy 125.73 99.06)
 		)
@@
 	(wire
 		(pts
-			(xy 81.28 87.63) (xy 88.9 87.63)
-		)
-		(stroke
-			(width 0)
-			(type default)
-		)
-	)
-	(wire
-		(pts
-			(xy 135.89 106.68) (xy 135.89 121.92)
+			(xy 72.39 87.63) (xy 80.01 87.63)
+		)
+		(stroke
+			(width 0)
+			(type default)
+		)
+	)
+	(wire
+		(pts
+			(xy 135.89 106.68) (xy 135.89 109.22)
 		)
 		(stroke
@@
 	(wire
 		(pts
-			(xy 88.9 95.25) (xy 88.9 101.6)
+			(xy 80.01 95.25) (xy 80.01 101.6)
 		)
 		(stroke
@@
 	(wire
 		(pts
-			(xy 102.87 87.63) (xy 115.57 87.63)
-		)
-		(stroke
-			(width 0)
-			(type default)
-		)
-	)
-	(wire
-		(pts
 			(xy 199.39 106.68) (xy 199.39 114.3)
 		)
@@
 	(wire
 		(pts
-			(xy 88.9 87.63) (xy 102.87 87.63)
+			(xy 120.65 101.6) (xy 120.65 109.22)
 		)
 		(stroke
@@
 	(wire
 		(pts
-			(xy 88.9 95.25) (xy 102.87 95.25)
+			(xy 93.98 87.63) (xy 106.68 87.63)
 		)
 		(stroke
@@
 	(wire
 		(pts
-			(xy 115.57 87.63) (xy 130.81 87.63)
+			(xy 135.89 109.22) (xy 135.89 121.92)
 		)
 		(stroke
@@
 	(wire
 		(pts
+			(xy 120.65 109.22) (xy 135.89 109.22)
+		)
+		(stroke
+			(width 0)
+			(type default)
+		)
+	)
+	(wire
+		(pts
+			(xy 106.68 87.63) (xy 120.65 87.63)
+		)
+		(stroke
+			(width 0)
+			(type default)
+		)
+	)
+	(wire
+		(pts
 			(xy 172.72 114.3) (xy 186.69 114.3)
 		)
@@
 	(wire
 		(pts
+			(xy 80.01 95.25) (xy 93.98 95.25)
+		)
+		(stroke
+			(width 0)
+			(type default)
+		)
+	)
+	(wire
+		(pts
 			(xy 172.72 99.06) (xy 186.69 99.06)
 		)
@@
 	(wire
 		(pts
+			(xy 80.01 87.63) (xy 93.98 87.63)
+		)
+		(stroke
+			(width 0)
+			(type default)
+		)
+	)
+	(wire
+		(pts
 			(xy 132.08 87.63) (xy 130.81 87.63)
 		)
@@
 	(wire
 		(pts
+			(xy 120.65 87.63) (xy 130.81 87.63)
+		)
+		(stroke
+			(width 0)
+			(type default)
+		)
+	)
+	(wire
+		(pts
 			(xy 186.69 99.06) (xy 199.39 99.06)
 		)
@@
 			(width 0)
 			(type default)
-		)
-	)
-	(hierarchical_label "BST_EN"
-		(shape input)
-		(at 120.65 99.06 180)
-		(effects
-			(font
-				(size 1.27 1.27)
-			)
-			(justify right)
 		)
 	)
@@
 	(hierarchical_label "BST_VIN"
 		(shape input)
-		(at 81.28 87.63 180)
-		(effects
-			(font
-				(size 1.27 1.27)
-			)
-			(justify right)
-		)
-	)
-	(hierarchical_label "BST_MODE"
-		(shape input)
-		(at 120.65 101.6 180)
+		(at 72.39 87.63 180)
 		(effects
 			(font
@@
 	(symbol
 		(lib_id "Device:C")
-		(at 115.57 91.44 0)
+		(at 106.68 91.44 0)
 		(unit 1)
 		(exclude_from_sim no)
@@
 		(dnp no)
 		(property "Reference" "C26"
-			(at 119.38 90.1699 0)
+			(at 110.49 90.1699 0)
 			(effects
 				(font
@@
 		)
 		(property "Value" "0.1uF 16V"
-			(at 117.348 94.234 0)
+			(at 108.458 94.234 0)
 			(effects
 				(font
@@
 		)
 		(property "Footprint" "Capacitor_SMD:C_0603_1608Metric_Pad1.08x0.95mm_HandSolder"
-			(at 116.5352 95.25 0)
+			(at 107.6452 95.25 0)
 			(effects
 				(font
@@
 		)
 		(property "Datasheet" "~"
-			(at 115.57 91.44 0)
+			(at 106.68 91.44 0)
 			(effects
 				(font
@@
 		)
 		(property "Description" "Unpolarized capacitor"
-			(at 115.57 91.44 0)
+			(at 106.68 91.44 0)
 			(effects
 				(font
@@
 	(symbol
 		(lib_id "power:GND")
-		(at 88.9 101.6 0)
+		(at 80.01 101.6 0)
 		(unit 1)
 		(exclude_from_sim no)
@@
 		(fields_autoplaced yes)
 		(property "Reference" "#PWR029"
-			(at 88.9 107.95 0)
+			(at 80.01 107.95 0)
 			(effects
 				(font
@@
 		)
 		(property "Value" "GND"
-			(at 88.9 106.68 0)
+			(at 80.01 106.68 0)
 			(effects
 				(font
@@
 		)
 		(property "Footprint" ""
-			(at 88.9 101.6 0)
+			(at 80.01 101.6 0)
 			(effects
 				(font
@@
 		)
 		(property "Datasheet" ""
-			(at 88.9 101.6 0)
+			(at 80.01 101.6 0)
 			(effects
 				(font
@@
 		)
 		(property "Description" "Power symbol creates a global label with name \"GND\" , ground"
-			(at 88.9 101.6 0)
+			(at 80.01 101.6 0)
 			(effects
 				(font
@@
 	(symbol
 		(lib_id "Device:C")
-		(at 102.87 91.44 0)
+		(at 93.98 91.44 0)
 		(unit 1)
 		(exclude_from_sim no)
@@
 		(dnp no)
 		(property "Reference" "C25"
-			(at 106.68 90.1699 0)
+			(at 97.79 90.1699 0)
 			(effects
 				(font
@@
 		)
 		(property "Value" "22uF 16V"
-			(at 104.14 93.98 0)
+			(at 95.25 93.98 0)
 			(effects
 				(font
@@
 		)
 		(property "Footprint" "Capacitor_SMD:C_0603_1608Metric_Pad1.08x0.95mm_HandSolder"
-			(at 103.8352 95.25 0)
+			(at 94.9452 95.25 0)
 			(effects
 				(font
@@
 		)
 		(property "Datasheet" "~"
-			(at 102.87 91.44 0)
+			(at 93.98 91.44 0)
 			(effects
 				(font
@@
 		)
 		(property "Description" "Unpolarized capacitor"
-			(at 102.87 91.44 0)
+			(at 93.98 91.44 0)
 			(effects
 				(font
@@
 	(symbol
 		(lib_id "Device:C")
-		(at 88.9 91.44 0)
+		(at 80.01 91.44 0)
 		(unit 1)
 		(exclude_from_sim no)
@@
 		(dnp no)
 		(property "Reference" "C27"
-			(at 92.71 90.1699 0)
+			(at 83.82 90.1699 0)
 			(effects
 				(font
@@
 		)
 		(property "Value" "22uF 16V"
-			(at 90.678 93.98 0)
+			(at 81.788 93.98 0)
 			(effects
 				(font
@@
 		)
 		(property "Footprint" "Capacitor_SMD:C_0603_1608Metric_Pad1.08x0.95mm_HandSolder"
-			(at 89.8652 95.25 0)
+			(at 80.9752 95.25 0)
 			(effects
 				(font
@@
 		)
 		(property "Datasheet" "~"
-			(at 88.9 91.44 0)
+			(at 80.01 91.44 0)
 			(effects
 				(font
@@
 		)
 		(property "Description" "Unpolarized capacitor"
-			(at 88.9 91.44 0)
-			(effects
-				(font
+			(at 80.01 91.44 0)
+			(effects
+				(font

Commit message: all
Other:
- moved on the sheet: C20, C21, C22, C23, C24, C25, C26, C27, L3, R15, R16, U2

Commit message: all
Parts:
- C20, C21, C22, C23, C25, C27: mouser (none) -> 81-ZRB18AR61C226ME1L
- C26: mouser (none) -> 581-0603YC104K4T4A
- R15: mouser (none) -> 603-AC0603FR-07750KL
- R16: mouser (none) -> 603-RT0603FRE13100KL
- U2: mouser (none) -> 595-TPS61022RWUT

Commit message: all
Parts:
- renumbered C27 to C16, C25 to C17, C26 to C18, C20 to C19, C21 to C20, C22 to C21, C23 to C22, C24 to C23, L3 to L2, U2 to U4
Changed lines of the file:
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@@
 		(in_pos_files yes)
 		(dnp no)
-		(property "Reference" "C24"
+		(property "Reference" "C23"
 			(at 231.14 96.5199 0)
 			(show_name no)
@@
 			(project "KB-01"
 				(path "/e6144e29-1dc4-45a8-93e7-988a20131b94/f9d53241-b903-4597-892d-d58932656724"
-					(reference "C24")
+					(reference "C23")
 					(unit 1)
 				)
@@
 		(in_pos_files yes)
 		(dnp no)
-		(property "Reference" "C20"
+		(property "Reference" "C19"
 			(at 179.07 96.5199 0)
 			(show_name no)
@@
 			(project "KB-01"
 				(path "/e6144e29-1dc4-45a8-93e7-988a20131b94/f9d53241-b903-4597-892d-d58932656724"
-					(reference "C20")
+					(reference "C19")
 					(unit 1)
 				)
@@
 		(dnp no)
 		(fields_autoplaced yes)
-		(property "Reference" "#PWR030"
+		(property "Reference" "#PWR048"
 			(at 138.43 123.19 0)
 			(hide yes)
@@
 			(project "KB-01"
 				(path "/e6144e29-1dc4-45a8-93e7-988a20131b94/f9d53241-b903-4597-892d-d58932656724"
-					(reference "#PWR030")
+					(reference "#PWR048")
 					(unit 1)
 				)
@@
 		(in_pos_files yes)
 		(dnp no)
-		(property "Reference" "C26"
+		(property "Reference" "C18"
 			(at 113.03 85.0899 0)
 			(show_name no)
@@
 			(project "KB-01"
 				(path "/e6144e29-1dc4-45a8-93e7-988a20131b94/f9d53241-b903-4597-892d-d58932656724"
-					(reference "C26")
+					(reference "C18")
 					(unit 1)
 				)
@@
 		(in_pos_files yes)
 		(dnp no)
-		(property "Reference" "C21"
+		(property "Reference" "C20"
 			(at 193.04 96.5199 0)
 			(show_name no)
@@
 			(project "KB-01"
 				(path "/e6144e29-1dc4-45a8-93e7-988a20131b94/f9d53241-b903-4597-892d-d58932656724"
-					(reference "C21")
+					(reference "C20")
 					(unit 1)
 				)
@@
 		(dnp no)
 		(fields_autoplaced yes)
-		(property "Reference" "L3"
+		(property "Reference" "L2"
 			(at 138.43 77.47 90)
 			(show_name no)
@@
 			(project "KB-01"
 				(path "/e6144e29-1dc4-45a8-93e7-988a20131b94/f9d53241-b903-4597-892d-d58932656724"
-					(reference "L3")
+					(reference "L2")
 					(unit 1)
 				)
@@
 		(dnp no)
 		(fields_autoplaced yes)
-		(property "Reference" "#PWR027"
+		(property "Reference" "#PWR046"
 			(at 201.93 118.11 0)
 			(hide yes)
@@
 			(project "KB-01"
 				(path "/e6144e29-1dc4-45a8-93e7-988a20131b94/f9d53241-b903-4597-892d-d58932656724"
-					(reference "#PWR027")
+					(reference "#PWR046")
 					(unit 1)
 				)
@@
 		(dnp no)
 		(fields_autoplaced yes)
-		(property "Reference" "#PWR029"
+		(property "Reference" "#PWR045"
 			(at 82.55 102.87 0)
 			(hide yes)
@@
 			(project "KB-01"
 				(path "/e6144e29-1dc4-45a8-93e7-988a20131b94/f9d53241-b903-4597-892d-d58932656724"
-					(reference "#PWR029")
+					(reference "#PWR045")
 					(unit 1)
 				)
@@
 		(dnp no)
 		(fields_autoplaced yes)
-		(property "Reference" "#PWR026"
+		(property "Reference" "#PWR047"
 			(at 161.29 121.92 0)
 			(hide yes)
@@
 			(project "KB-01"
 				(path "/e6144e29-1dc4-45a8-93e7-988a20131b94/f9d53241-b903-4597-892d-d58932656724"
-					(reference "#PWR026")
+					(reference "#PWR047")
 					(unit 1)
 				)
@@
 		(in_pos_files yes)
 		(dnp no)
-		(property "Reference" "C23"
+		(property "Reference" "C22"
 			(at 218.44 96.5199 0)
 			(show_name no)
@@
 			(project "KB-01"
 				(path "/e6144e29-1dc4-45a8-93e7-988a20131b94/f9d53241-b903-4597-892d-d58932656724"
-					(reference "C23")
+					(reference "C22")
 					(unit 1)
 				)
@@
 		(in_pos_files yes)
 		(dnp no)
-		(property "Reference" "C22"
+		(property "Reference" "C21"
 			(at 205.74 96.5199 0)
 			(show_name no)
@@
 			(project "KB-01"
 				(path "/e6144e29-1dc4-45a8-93e7-988a20131b94/f9d53241-b903-4597-892d-d58932656724"
-					(reference "C22")
+					(reference "C21")
 					(unit 1)
 				)
@@
 		(dnp no)
 		(fields_autoplaced yes)
-		(property "Reference" "U2"
+		(property "Reference" "U4"
 			(at 140.5733 101.6 0)
 			(show_name no)
@@
 			(project "KB-01"
 				(path "/e6144e29-1dc4-45a8-93e7-988a20131b94/f9d53241-b903-4597-892d-d58932656724"
-					(reference "U2")
+					(reference "U4")
 					(unit 1)
 				)
@@
 		(in_pos_files yes)
 		(dnp no)
-		(property "Reference" "C25"
+		(property "Reference" "C17"
 			(at 100.33 85.0899 0)
 			(show_name no)
@@
 			(project "KB-01"
 				(path "/e6144e29-1dc4-45a8-93e7-988a20131b94/f9d53241-b903-4597-892d-d58932656724"
-					(reference "C25")
+					(reference "C17")
 					(unit 1)
 				)
@@
 		(in_pos_files yes)
 		(dnp no)
-		(property "Reference" "C27"
+		(property "Reference" "C16"
 			(at 86.36 85.0899 0)
 			(show_name no)
@@
 			(project "KB-01"
 				(path "/e6144e29-1dc4-45a8-93e7-988a20131b94/f9d53241-b903-4597-892d-d58932656724"
-					(reference "C27")
-					(unit 1)
-				)
+					(reference "C16")
+					(unit 1)
+				)

Commit message: all
Parts:
- C23: footprint Capacitor_SMD:C_0603_1608Metric_Pad1.08x0.95mm_HandSolder -> Resistor_SMD:R_1206_3216Metric; mouser (none) -> 963-EMK316BBJ476ML-T
Changed lines of the file:
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@@
 			)
 		)
-		(property "Footprint" "Capacitor_SMD:C_0603_1608Metric_Pad1.08x0.95mm_HandSolder"
+		(property "Footprint" "Resistor_SMD:R_1206_3216Metric"
 			(at 228.2952 101.6 0)
 			(hide yes)
@@
 			(at 227.33 97.79 0)
 			(hide yes)
+			(show_name no)
+			(do_not_autoplace no)
+			(effects
+				(font
+					(size 1.27 1.27)
+				)
+			)
+		)
+		(property "mouser" "963-EMK316BBJ476ML-T"
+			(at 227.33 97.79 0)
+			(hide yes)
