File: KB-01_kicad/KB-01/KB-01.kicad_pcb (KiCad board)
At the start: 2 copper layers, 1 part

Commit message: all
Signed-off-by: syauqi-alias <syauqi_nur@yahoo.com>
Parts:
- added C1: 10uF, Capacitor_SMD:C_0603_1608Metric_Pad1.08x0.95mm_HandSolder, F.Cu at (77.8, 57.1)
- added C10: 47nF 16V, Capacitor_SMD:C_0603_1608Metric_Pad1.08x0.95mm_HandSolder, F.Cu at (77.8, 71.7)
- added C11: 10uF 16V, Capacitor_SMD:C_0603_1608Metric_Pad1.08x0.95mm_HandSolder, F.Cu at (77.8, 74.2)
- added C12: 10uF 16V, Capacitor_SMD:C_0603_1608Metric_Pad1.08x0.95mm_HandSolder, F.Cu at (77.8, 76.7)
- added C13: 4.7uF 16V, Capacitor_SMD:C_0603_1608Metric_Pad1.08x0.95mm_HandSolder, F.Cu at (77.8, 79.2)
- added C14: 10uF 16V, Capacitor_SMD:C_0603_1608Metric_Pad1.08x0.95mm_HandSolder, F.Cu at (77.8, 81.7)
- added C15: 22uF 16V, Capacitor_SMD:C_0603_1608Metric_Pad1.08x0.95mm_HandSolder, F.Cu at (82.1, 71.7)
- added C16: 22uF 16V, Capacitor_SMD:C_0603_1608Metric_Pad1.08x0.95mm_HandSolder, F.Cu at (82.1, 74.2)
- added C17: 1uF 25V, Capacitor_SMD:C_0603_1608Metric_Pad1.08x0.95mm_HandSolder, F.Cu at (82.1, 76.7)
- added C18: 0.1uF 16V, Capacitor_SMD:C_0603_1608Metric_Pad1.08x0.95mm_HandSolder, F.Cu at (82.1, 79.2)
- added C19: 0.1uF 16V, Capacitor_SMD:C_0603_1608Metric_Pad1.08x0.95mm_HandSolder, F.Cu at (82.1, 81.7)
- added C2: 10uF, Capacitor_SMD:C_0603_1608Metric_Pad1.08x0.95mm_HandSolder, F.Cu at (77.8, 59.7)
- added C20: 22uF 16V, Capacitor_SMD:C_0603_1608Metric_Pad1.08x0.95mm_HandSolder, F.Cu at (104.2, 71.7)
- added C21: 22uF 16V, Capacitor_SMD:C_0603_1608Metric_Pad1.08x0.95mm_HandSolder, F.Cu at (104.2, 74.2)
- added C22: 22uF 16V, Capacitor_SMD:C_0603_1608Metric_Pad1.08x0.95mm_HandSolder, F.Cu at (104.2, 76.7)
- added C23: 22uF 16V, Capacitor_SMD:C_0603_1608Metric_Pad1.08x0.95mm_HandSolder, F.Cu at (104.2, 79.2)
- added C24: 47uF 16V, Capacitor_SMD:C_0603_1608Metric_Pad1.08x0.95mm_HandSolder, F.Cu at (104.2, 81.7)
- added C25: 22uF 16V, Capacitor_SMD:C_0603_1608Metric_Pad1.08x0.95mm_HandSolder, F.Cu at (104.2, 84.2)
- added C26: 0.1uF 16V, Capacitor_SMD:C_0603_1608Metric_Pad1.08x0.95mm_HandSolder, F.Cu at (104.2, 86.8)
- added C27: 22uF 16V, Capacitor_SMD:C_0603_1608Metric_Pad1.08x0.95mm_HandSolder, F.Cu at (104.2, 89.3)
- added C28: 1uF, Capacitor_SMD:C_0603_1608Metric_Pad1.08x0.95mm_HandSolder, F.Cu at (105.0, 45.0)
- added C29: 1uF, Capacitor_SMD:C_0603_1608Metric_Pad1.08x0.95mm_HandSolder, F.Cu at (105.0, 47.5)
- added C3: 0.1uF 10V, Capacitor_SMD:C_0603_1608Metric_Pad1.08x0.95mm_HandSolder, F.Cu at (77.8, 62.2)
- added C30: 10nF, Capacitor_SMD:C_0603_1608Metric_Pad1.08x0.95mm_HandSolder, F.Cu at (105.0, 50.0)
- added C31: 56pF, Capacitor_SMD:C_0603_1608Metric_Pad1.08x0.95mm_HandSolder, F.Cu at (105.0, 52.5)
- added C32: 56pF, Capacitor_SMD:C_0603_1608Metric_Pad1.08x0.95mm_HandSolder, F.Cu at (105.0, 55.0)
- added C4: 4.7nF 10V, Capacitor_SMD:C_0603_1608Metric_Pad1.08x0.95mm_HandSolder, F.Cu at (77.8, 64.7)
- added C5: 10uF, Capacitor_SMD:C_0603_1608Metric_Pad1.08x0.95mm_HandSolder, F.Cu at (77.8, 67.2)
- added C6: 10uF, Capacitor_SMD:C_0603_1608Metric_Pad1.08x0.95mm_HandSolder, F.Cu at (82.1, 57.1)
- added C7: 10uF, Capacitor_SMD:C_0603_1608Metric_Pad1.08x0.95mm_HandSolder, F.Cu at (82.1, 59.7)
- added C8: 0.1uF 10V, Capacitor_SMD:C_0603_1608Metric_Pad1.08x0.95mm_HandSolder, F.Cu at (82.1, 62.2)
- added C9: 10uF, Capacitor_SMD:C_0603_1608Metric_Pad1.08x0.95mm_HandSolder, F.Cu at (82.1, 64.7)
- added D1: Green, Diode_SMD:D_0603_1608Metric_Pad1.05x0.95mm_HandSolder, F.Cu at (96.1, 64.2)
- added D2: Green, Diode_SMD:D_0603_1608Metric_Pad1.05x0.95mm_HandSolder, F.Cu at (96.5, 92.1)
- added J1: Bus_M.2_Socket_M, M.2 NGFF:121992304, F.Cu at (88.1, 49.9)
- added J2: Conn_01x02_Socket, Connector_JST:JST_XH_B2B-XH-AM_1x02_P2.50mm_Vertical, F.Cu at (91.1, 86.4)
- added J3: USB_C_Receptacle_USB2.0_14P, Connector_USB:USB_C_Receptacle_JAE_DX07S016JA1R1500, F.Cu at (81.6, 87.8)
- added J4: NTC (optional), Connector_Wire:SolderWire-0.1sqmm_1x01_D0.4mm_OD1mm, F.Cu at (96.1, 95.2)
- added L1: 2.2uH, CM5IO:L_Bourns_SRP5030CC, F.Cu at (92.7, 59.6)
- added L2: 1.0uH, Inductor_SMD:L_Coilcraft_XAL5030-XXX, F.Cu at (96.5, 74.1)
- added L3: 1uH 21.8A, Inductor_SMD:L_Coilcraft_XAL7030-102, F.Cu at (111.1, 75.2)
- added L4: 27nH, Inductor_SMD:L_0603_1608Metric_Pad1.05x0.95mm_HandSolder, F.Cu at (105.0, 57.5)
- added R1: 10k 1%, Resistor_SMD:R_0603_1608Metric_Pad0.98x0.95mm_HandSolder, F.Cu at (82.1, 67.2)
- added R10: 10K, Resistor_SMD:R_0603_1608Metric_Pad0.98x0.95mm_HandSolder, F.Cu at (90.8, 71.7)
- added R11: 10K, Resistor_SMD:R_0603_1608Metric_Pad0.98x0.95mm_HandSolder, F.Cu at (90.8, 74.2)
- added R12: 10K, Resistor_SMD:R_0603_1608Metric_Pad0.98x0.95mm_HandSolder, F.Cu at (90.8, 76.7)
- added R13: 10K, Resistor_SMD:R_0603_1608Metric_Pad0.98x0.95mm_HandSolder, F.Cu at (90.8, 79.2)
- added R14: 10K, Resistor_SMD:R_0603_1608Metric_Pad0.98x0.95mm_HandSolder, F.Cu at (90.8, 81.7)
- added R15: 750k, Resistor_SMD:R_0603_1608Metric_Pad0.98x0.95mm_HandSolder, F.Cu at (104.2, 91.8)
- added R16: 100k, Resistor_SMD:R_0603_1608Metric_Pad0.98x0.95mm_HandSolder, F.Cu at (104.2, 94.3)
- added R2: 2.2k 1%, Resistor_SMD:R_0603_1608Metric_Pad0.98x0.95mm_HandSolder, F.Cu at (86.5, 57.1)
- added R3: 100k 1%, Resistor_SMD:R_0603_1608Metric_Pad0.98x0.95mm_HandSolder, F.Cu at (86.5, 59.7)
- added R4: 1k, Resistor_SMD:R_0603_1608Metric_Pad0.98x0.95mm_HandSolder, F.Cu at (86.5, 62.2)
- added R5: 2.21K, Resistor_SMD:R_0603_1608Metric_Pad0.98x0.95mm_HandSolder, F.Cu at (86.5, 71.7)
- added R6: 5.1k, Resistor_SMD:R_0603_1608Metric_Pad0.98x0.95mm_HandSolder, F.Cu at (86.5, 74.2)
- added R7: 5.1k, Resistor_SMD:R_0603_1608Metric_Pad0.98x0.95mm_HandSolder, F.Cu at (86.5, 76.7)
- added R8: 133, Resistor_SMD:R_0603_1608Metric_Pad0.98x0.95mm_HandSolder, F.Cu at (86.5, 79.2)
- added R9: R, Resistor_SMD:R_0603_1608Metric_Pad0.98x0.95mm_HandSolder, F.Cu at (86.5, 81.7)
- added U1: BQ25895, Package_DFN_QFN:Texas_RTW_WQFN-24-1EP_4x4mm_P0.5mm_EP2.7x2.7mm_ThermalVias, F.Cu at (91.1, 94.0)
- added U2: TPS61022, Package_DFN_QFN:Texas_RWU0007A_VQFN-7_2x2mm_P0.5mm, F.Cu at (108.6, 81.8)
- added U4: ASEK-32.768KHZ-L-R-T, Crystal:Crystal_SMD_3225-4Pin_3.2x2.5mm, F.Cu at (91.3, 65.2)
- added U5: AP3441SHE-7B, Package_DFN_QFN:DFN-8-1EP_2x2mm_P0.5mm_EP1.05x1.75mm, F.Cu at (98.9, 57.8)
- added U6: TS3USB30ERSWR, Package_DFN_QFN:UQFN-10_1.4x1.8mm_P0.4mm, F.Cu at (94.8, 79.7)
- added U7: TLV70033_SOT353, Package_TO_SOT_SMD:SOT-353_SC-70-5, F.Cu at (109.5, 45.6)

Commit message: all
Parts:
- removed C29: 1uF, Capacitor_SMD:C_0603_1608Metric_Pad1.08x0.95mm_HandSolder
- removed C30: 10nF, Capacitor_SMD:C_0603_1608Metric_Pad1.08x0.95mm_HandSolder
- removed C31, C32: 56pF, Capacitor_SMD:C_0603_1608Metric_Pad1.08x0.95mm_HandSolder
- removed L3: 1uH 21.8A, Inductor_SMD:L_Coilcraft_XAL7030-102
- removed L4: 27nH, Inductor_SMD:L_0603_1608Metric_Pad1.05x0.95mm_HandSolder
- removed U7: TLV70033_SOT353, Package_TO_SOT_SMD:SOT-353_SC-70-5
- added C34: 0.1uF 10V, Capacitor_SMD:C_0603_1608Metric_Pad1.08x0.95mm_HandSolder, F.Cu at (62.7, 99.1)
- added C35: 10uF10V, Capacitor_SMD:C_0603_1608Metric_Pad1.08x0.95mm_HandSolder, F.Cu at (62.7, 101.6)
- added C36: 10uF10V, Capacitor_SMD:C_0603_1608Metric_Pad1.08x0.95mm_HandSolder, F.Cu at (62.7, 104.1)
- added C37: 0.1uF 10V, Capacitor_SMD:C_0603_1608Metric_Pad1.08x0.95mm_HandSolder, F.Cu at (62.7, 106.6)
- added C38: 4.7nF 10V, Capacitor_SMD:C_0603_1608Metric_Pad1.08x0.95mm_HandSolder, F.Cu at (62.7, 109.1)
- added C39: 10uF10V, Capacitor_SMD:C_0603_1608Metric_Pad1.08x0.95mm_HandSolder, F.Cu at (67.1, 99.1)
- added C40: 10uF10V, Capacitor_SMD:C_0603_1608Metric_Pad1.08x0.95mm_HandSolder, F.Cu at (67.1, 101.6)
- added C41: 10uF10V, Capacitor_SMD:C_0603_1608Metric_Pad1.08x0.95mm_HandSolder, F.Cu at (67.1, 104.1)
- added C42: 10uF10V, Capacitor_SMD:C_0603_1608Metric_Pad1.08x0.95mm_HandSolder, F.Cu at (67.1, 106.6)
- added C43: 100nF 6.3V, Capacitor_SMD:C_0603_1608Metric_Pad1.08x0.95mm_HandSolder, F.Cu at (111.7, 60.3)
- added C44: 100nF 6.3V, Capacitor_SMD:C_0603_1608Metric_Pad1.08x0.95mm_HandSolder, F.Cu at (111.7, 62.8)
- added C45: 100nF 6.3V, Capacitor_SMD:C_0603_1608Metric_Pad1.08x0.95mm_HandSolder, F.Cu at (111.7, 65.3)
- added C46: 100nF 6.3V, Capacitor_SMD:C_0603_1608Metric_Pad1.08x0.95mm_HandSolder, F.Cu at (111.7, 67.8)
- added C47: 0.1uF 10V, Capacitor_SMD:C_0603_1608Metric_Pad1.08x0.95mm_HandSolder, F.Cu at (111.7, 70.4)
- added C48: 100nF 6.3V, Capacitor_SMD:C_0603_1608Metric_Pad1.08x0.95mm_HandSolder, F.Cu at (111.7, 72.9)
- added C49: 10uF 6.3V, Capacitor_SMD:C_0603_1608Metric_Pad1.08x0.95mm_HandSolder, F.Cu at (116.0, 60.3)
- added C50: 100nF 6.3V, Capacitor_SMD:C_0603_1608Metric_Pad1.08x0.95mm_HandSolder, F.Cu at (116.0, 62.8)
- added C51: 100nF 6.3V, Capacitor_SMD:C_0603_1608Metric_Pad1.08x0.95mm_HandSolder, F.Cu at (116.0, 65.3)
- added C52: 220nF 25V, Capacitor_SMD:C_0603_1608Metric_Pad1.08x0.95mm_HandSolder, F.Cu at (116.0, 67.8)
- added C53: 100nF 6.3V, Capacitor_SMD:C_0603_1608Metric_Pad1.08x0.95mm_HandSolder, F.Cu at (38.2, 102.6)
- added C54: 100nF 6.3V, Capacitor_SMD:C_0603_1608Metric_Pad1.08x0.95mm_HandSolder, F.Cu at (38.2, 105.1)
- added C55: 100nF 6.3V, Capacitor_SMD:C_0603_1608Metric_Pad1.08x0.95mm_HandSolder, F.Cu at (38.2, 107.6)
- added C56: 100nF 6.3V, Capacitor_SMD:C_0603_1608Metric_Pad1.08x0.95mm_HandSolder, F.Cu at (38.2, 110.2)
- added C57: 100nF 6.3V, Capacitor_SMD:C_0603_1608Metric_Pad1.08x0.95mm_HandSolder, F.Cu at (38.2, 112.7)
- added D3: Green, Diode_SMD:D_0603_1608Metric_Pad1.05x0.95mm_HandSolder, F.Cu at (119.6, 52.5)
- added D4: BAT54-05W, Package_TO_SOT_SMD:SOT-323_SC-70, F.Cu at (112.3, 53.8)
- added D5: SM15T36CA, Diode_SMD:D_SMA, F.Cu at (120.9, 103.0)
- added D6: LED Red, LED_SMD:LED_0603_1608Metric_Pad1.05x0.95mm_HandSolder, F.Cu at (123.4, 90.4)
- added D8: Green, Diode_SMD:D_0603_1608Metric_Pad1.05x0.95mm_HandSolder, F.Cu at (81.1, 106.1)
- added D9: 1N4148W, Diode_SMD:D_SOD-123, F.Cu at (52.0, 111.1)
- added IC1: MAX17048G+T10, MAX17048G+T10:SON50P200X200X80-9N-D, F.Cu at (92.2, 41.1)
- added J11: Conn_02x07_Odd_Even, Connector_PinHeader_1.00mm:PinHeader_2x07_P1.00mm_Vertical_SMD, F.Cu at (107.8, 124.1)
- added J12: Conn_01x01_Socket, Connector_Wire:SolderWirePad_1x01_SMD_2x4mm, F.Cu at (121.8, 57.8)
- added J5: Conn_01x01_Socket, Connector_Wire:SolderWirePad_1x01_SMD_2x4mm, F.Cu at (119.3, 57.8)
- added J6: Conn_Coaxial, Connector_Coaxial:U.FL_Hirose_U.FL-R-SMT-1_Vertical, F.Cu at (106.7, 102.5)
- added J8: Bus_M.2_Socket_M, CM5IO:M.2 M Key socket, F.Cu at (149.5, 77.9)
- added J9: AudioJack3_SwitchTR, Connector_Audio:Jack_3.5mm_CUI_SJ2-3593D-SMT_Horizontal, F.Cu at (103.4, 68.6)
- added L5: 2.2uH, CM5IO:L_Bourns_SRP5030CC, F.Cu at (77.6, 101.5)
- added LS1: CMT-0502-03-SMT-TR, CMT-0502-03SMTTR:CMT050203SMTTR, F.Cu at (53.5, 105.4)
- added Q1: MMBT3904, Package_TO_SOT_SMD:SOT-23, F.Cu at (111.5, 101.7)
- added Q2: 2N7002, Package_TO_SOT_SMD:SOT-23, F.Cu at (56.1, 87.8)
- added R17: 330, Resistor_SMD:R_0402_1005Metric_Pad0.72x0.64mm_HandSolder, F.Cu at (122.8, 92.7)
- added R18: 4.7k, Resistor_SMD:R_0603_1608Metric_Pad0.98x0.95mm_HandSolder, F.Cu at (119.0, 96.9)
- added R19: 10k, Resistor_SMD:R_0603_1608Metric_Pad0.98x0.95mm_HandSolder, F.Cu at (119.0, 99.4)
- added R21: 1k, Resistor_SMD:R_0603_1608Metric_Pad0.98x0.95mm_HandSolder, F.Cu at (67.1, 109.1)
- added R22: 10K 1%, Resistor_SMD:R_0603_1608Metric_Pad0.98x0.95mm_HandSolder, F.Cu at (71.4, 99.1)
- added R23: 100k 1%, Resistor_SMD:R_0603_1608Metric_Pad0.98x0.95mm_HandSolder, F.Cu at (71.4, 101.6)
- added R24: 2.2k 1%, Resistor_SMD:R_0603_1608Metric_Pad0.98x0.95mm_HandSolder, F.Cu at (71.4, 104.1)
- added R25: 10k, Resistor_SMD:R_0603_1608Metric_Pad0.98x0.95mm_HandSolder, F.Cu at (116.0, 70.4)
- added R26: 10k, Resistor_SMD:R_0603_1608Metric_Pad0.98x0.95mm_HandSolder, F.Cu at (42.5, 102.6)
- added R27: 10k, Resistor_SMD:R_0603_1608Metric_Pad0.98x0.95mm_HandSolder, F.Cu at (42.5, 105.1)
- added R28: 10k, Resistor_SMD:R_0603_1608Metric_Pad0.98x0.95mm_HandSolder, F.Cu at (42.5, 107.6)
- added R29: 10k, Resistor_SMD:R_0603_1608Metric_Pad0.98x0.95mm_HandSolder, F.Cu at (42.5, 110.2)
- added R30: 10k, Resistor_SMD:R_0603_1608Metric_Pad0.98x0.95mm_HandSolder, F.Cu at (42.5, 112.7)
- added R31: 1k, Resistor_SMD:R_0603_1608Metric_Pad0.98x0.95mm_HandSolder, F.Cu at (46.9, 102.6)
- added R32: 1k, Resistor_SMD:R_0603_1608Metric_Pad0.98x0.95mm_HandSolder, F.Cu at (46.9, 105.1)
- added R33: 1k, Resistor_SMD:R_0603_1608Metric_Pad0.98x0.95mm_HandSolder, F.Cu at (46.9, 107.6)
- added R34: 180, Resistor_SMD:R_0603_1608Metric_Pad0.98x0.95mm_HandSolder, F.Cu at (46.9, 110.2)
- added R35: 10k, Resistor_SMD:R_0603_1608Metric_Pad0.98x0.95mm_HandSolder, F.Cu at (46.9, 112.7)
- added SW1: Right angle Tact button, Button_Switch_SMD:SW_SPST_EVQP7A, F.Cu at (121.5, 109.8)
- added SW2: Power button, Button_Switch_SMD:SW_Push_1P1T_NO_CK_KSC6xxJ, F.Cu at (115.4, 41.0)
- added SW3: RotaryEncoder_Switch_MP, Rotary_Encoder:RotaryEncoder_Bourns_Vertical_PEC12R-3x17F-Sxxxx, F.Cu at (37.6, 91.0)
- added SW4: SW_Push, PCM_Switch_Keyboard_Kailh:SW_Kailh_Choc_V2, F.Cu at (135.8, 37.8)
- added SW5: SW_Push, PCM_Switch_Keyboard_Kailh:SW_Kailh_Choc_V2, F.Cu at (135.8, 54.3)
- added TP1: TestPoint, TestPoint:TestPoint_Pad_2.0x2.0mm, F.Cu at (118.6, 121.6)
- added TP2: TestPoint, TestPoint:TestPoint_Pad_2.0x2.0mm, F.Cu at (118.6, 125.7)
- added TP3: TestPoint, TestPoint:TestPoint_Pad_1.0x1.0mm, F.Cu at (122.3, 29.0)
- added TP4: TestPoint, TestPoint:TestPoint_Pad_1.0x1.0mm, F.Cu at (122.3, 32.1)
- added U10: AP3441SHE-7B, Package_DFN_QFN:DFN-8-1EP_2x2mm_P0.5mm_EP1.05x1.75mm, F.Cu at (83.8, 99.8)
- added U11: BMP581, BMP581:BMP581, F.Cu at (118.2, 76.7)
- added U12: BMI270, BMI270:BMI270, F.Cu at (112.6, 76.9)
- added U13: SHT40, Sensor_Humidity:Sensirion_DFN-4_1.5x1.5mm_P0.8mm_SHT4x_NoCentralPad, F.Cu at (111.6, 81.2)
- added U14: LIS2MDL, Package_LGA:LGA-12_2x2mm_P0.5mm, F.Cu at (117.6, 81.2)
- added U3: TLV70430DBVR, TLV70430DBVR:DBV0005A_N, F.Cu at (90.6, 47.3)
- added U9: ASEK-32.768KHZ-L-R-T, Crystal:Crystal_SMD_3225-4Pin_3.2x2.5mm, F.Cu at (76.2, 107.1)
- C1: value 10uF -> 100nF 6.3V
- C10: value 47nF 16V -> 10uF 25V
- C11: value 10uF 16V -> 0.1uF 25V
- C12, C14: value 10uF 16V -> 4.7uF 16V
- C13: value 4.7uF 16V -> 1uF 25V
- C15: value 22uF 16V -> 0.1uF 25V
- C17: value 1uF 25V -> 22uF 16V
- C19: value 0.1uF 16V -> 22uF 16V
- C2: value 10uF -> 0.1F 5.5V; footprint Capacitor_SMD:C_0603_1608Metric_Pad1.08x0.95mm_HandSolder -> Capacitor_SMD:CP_Elec_10x10.5
- C23: value 22uF 16V -> 47uF 16V
- C24: value 47uF 16V -> 100nF 6.3V
- C25: value 22uF 16V -> 10uF 6.3V
- C26: value 0.1uF 16V -> 1uF 16V
- C27: value 22uF 16V -> 1uF 16V
- C28: value 1uF -> 56pF 50V; footprint Capacitor_SMD:C_0603_1608Metric_Pad1.08x0.95mm_HandSolder -> Capacitor_SMD:C_0402_1005Metric_Pad0.74x0.62mm_HandSolder
- C3, C8: value 0.1uF 10V -> 10uF 25V
- C4: value 4.7nF 10V -> 0.1uF 25V
- C5: value 10uF -> 1uF 25V
- C6: value 10uF -> 0.1uF 10V
- C7: value 10uF -> 47nF 25V
- C9: value 10uF -> 10uF 25V
- D1: value Green -> LED Green; footprint Diode_SMD:D_0603_1608Metric_Pad1.05x0.95mm_HandSolder -> LED_SMD:LED_0603_1608Metric
- D2: value Green -> LED Red; footprint Diode_SMD:D_0603_1608Metric_Pad1.05x0.95mm_HandSolder -> LED_SMD:LED_0603_1608Metric
- J1: value Bus_M.2_Socket_M -> Conn_01x22_Female; footprint M.2 NGFF:121992304 -> CM5IO:Hirose_FH12-22S-0.5SH_1x22-1MP_P0.50mm_Horizontal
- J2: value Conn_01x02_Socket -> Conn_01x03; footprint Connector_JST:JST_XH_B2B-XH-AM_1x02_P2.50mm_Vertical -> Connector_PinHeader_2.54mm:PinHeader_1x03_P2.54mm_Vertical
- J4: value NTC (optional) -> Conn_01x02_Socket; footprint Connector_Wire:SolderWire-0.1sqmm_1x01_D0.4mm_OD1mm -> Connector_JST:JST_PH_B2B-PH-SM4-TB_1x02-1MP_P2.00mm_Vertical
- L1: value 2.2uH -> 1.0uH; footprint CM5IO:L_Bourns_SRP5030CC -> Inductor_SMD:L_Coilcraft_XAL5030-XXX
- L2: value 1.0uH -> 1uH 21.8A; footprint Inductor_SMD:L_Coilcraft_XAL5030-XXX -> Inductor_SMD:L_Coilcraft_XAL7030-102
- R1: value 10k 1% -> 4.7k
- R10, R11, R12, R13, R14: value 10K -> 10k
- R2: value 2.2k 1% -> 4.7k
- R3: value 100k 1% -> 1k
- R8: value 133 -> 10k
- R9: value R -> 133
- U2: value TPS61022 -> TS3USB30ERSWR; footprint Package_DFN_QFN:Texas_RWU0007A_VQFN-7_2x2mm_P0.5mm -> Package_DFN_QFN:UQFN-10_1.4x1.8mm_P0.4mm
- U4: value ASEK-32.768KHZ-L-R-T -> TPS61022; footprint Crystal:Crystal_SMD_3225-4Pin_3.2x2.5mm -> Package_DFN_QFN:Texas_RWU0007A_VQFN-7_2x2mm_P0.5mm
- U5: value AP3441SHE-7B -> TLV773_SOT353; footprint Package_DFN_QFN:DFN-8-1EP_2x2mm_P0.5mm_EP1.05x1.75mm -> Package_TO_SOT_SMD:SOT-353_SC-70-5
- U6: value TS3USB30ERSWR -> TESEO-LIV4F; footprint Package_DFN_QFN:UQFN-10_1.4x1.8mm_P0.4mm -> TESEO-LIV4FTR:TESEOLIV4FTR
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Connections:
- C1 pad 1: +5V -> /CM5_GPIO/VBAT
- C10 pad 1: Net-(C10-Pad1) -> /Battery_charger/Fuel_G
- C10 pad 2: Net-(U1-BTST) -> GND
- C11 pad 1: /battery_charger/Vsys -> /Battery_charger/Fuel_G
- C12 pad 1: /battery_charger/Vsys -> Net-(U1-REGN)
- C13 pad 1: Net-(U1-REGN) -> Net-(D4-K)
- C14 pad 1: /battery_charger/Fuel_G -> +3V_CHRG
- C15 pad 1: Net-(U1-PMID) -> /Battery_charger/Fuel_G
- C16 pad 1: Net-(U1-PMID) -> /Battery_charger/Vsys
- C17 pad 1: VBUS -> /Battery_charger/Vsys
- C18 pad 1: /battery_charger/Fuel_G -> /Battery_charger/Vsys
- C19 pad 1: /battery_charger/Fuel_G -> +5V
- C2 pad 1: +5V -> /CM5_GPIO/VBAT
- C24 pad 1: +5V -> /GNSS/3.3V_GNSS
- C25 pad 1: /5v_boost_conv/BST_VIN -> /GNSS/3.3V_GNSS
- C26 pad 1: /5v_boost_conv/BST_VIN -> +5V
- C27 pad 1: /5v_boost_conv/BST_VIN -> /GNSS/3.3V_GNSS
- C28 pad 1: /gnss/3.3V_GNSS -> Net-(D5-A1)
- C28 pad 2: GND -> Net-(U6-RF_IN)
- C3 pad 1: +5V -> Net-(U1-PMID)
- C4 pad 1: /pcie-nvme/M.2_3v3 -> Net-(U1-PMID)
- C4 pad 2: /pcie-nvme/FB -> GND
- C5 pad 1: /pcie-nvme/M.2_3v3 -> VBUS
- C6 pad 1: /pcie-nvme/M.2_3v3 -> +3V_CHRG
- C7 pad 1: /pcie-nvme/M.2_3v3 -> Net-(C7-Pad1)
- C7 pad 2: GND -> Net-(U1-BTST)
- C8 pad 1: /pcie-nvme/M.2_3v3 -> /Battery_charger/Vsys
- C9 pad 1: /pcie-nvme/M.2_3v3 -> /Battery_charger/Vsys
- D1 pad 2: /pcie-nvme/M.2_3v3 -> +3V3
- D2 pad 2: Net-(D2-A) -> +3V3
- J1 pad 10: Net-(J1-DAS/~{DSS}/~{LED1}) -> GND
- J1 pad 11: unconnected-(J1-PERn3-Pad11) -> /CM5_high_speed/DPHY0_D2_N
- J1 pad 12: /pcie-nvme/M.2_3v3 -> /CM5_high_speed/DPHY0_D2_P
- J1 pad 13: unconnected-(J1-PERp3-Pad13) -> GND
- J1 pad 14: /pcie-nvme/M.2_3v3 -> /CM5_high_speed/DPHY0_D3_N
- J1 pad 15: GND -> /CM5_high_speed/DPHY0_D3_P
- J1 pad 16: /pcie-nvme/M.2_3v3 -> GND
- J1 pad 18: /pcie-nvme/M.2_3v3 -> unconnected-(J1-Pin_18-Pad18)
- J1 pad 19: unconnected-(J1-PETp2-Pad19) -> GND
- J1 pad 2: /pcie-nvme/M.2_3v3 -> /CM5_high_speed/DPHY0_D0_N
- J1 pad 20: unconnected-(J1-NC-Pad20) -> /CM5_high_speed/SCL0
- J1 pad 21: GND -> /CM5_high_speed/SDA0
- J1 pad 22: unconnected-(J1-NC-Pad22) -> +3V3
- J1 pad 3: GND -> /CM5_high_speed/DPHY0_D0_P
- J1 pad 4: /pcie-nvme/M.2_3v3 -> GND
- J1 pad 5: unconnected-(J1-PETn3-Pad5) -> /CM5_high_speed/DPHY0_D1_N
- J1 pad 6: unconnected-(J1-NC-Pad6) -> /CM5_high_speed/DPHY0_D1_P
- J1 pad 7: unconnected-(J1-PETp3-Pad7) -> GND
- J1 pad 8: unconnected-(J1-NC-Pad8) -> /CM5_high_speed/DPHY0_C_N
- J1 pad 9: GND -> /CM5_high_speed/DPHY0_C_P
- J2 pad 1: /battery_charger/Fuel_G -> /CM5_GPIO/WL_nDis
- J3 pad A6: /battery_charger/USB_D+ -> /Battery_charger/USB_D+
- J3 pad A7: /battery_charger/USB_D- -> /Battery_charger/USB_D-
- J3 pad B6: /battery_charger/USB_D+ -> /Battery_charger/USB_D+
- J3 pad B7: /battery_charger/USB_D- -> /Battery_charger/USB_D-
- J4 pad 1: Net-(J4-Pin_1) -> /Battery_charger/Fuel_G
- L1 pad 1: Net-(U5-LX) -> Net-(C7-Pad1)
- L1 pad 2: /pcie-nvme/M.2_3v3 -> /Battery_charger/Vsys
- L2 pad 1: Net-(C10-Pad1) -> /Battery_charger/Vsys
- L2 pad 2: /battery_charger/Vsys -> Net-(U4-SW)
- Module1 pad 1: unconnected-(Module1A-GND-Pad1) -> GND
- Module1 pad 10: unconnected-(Module1A-Ethernet_Pair0_N-Pad10) -> /CM5_GPIO/TRD0_N
- Module1 pad 100: unconnected-(Module1A-CAM_GPIO1-Pad100) -> /CM5_GPIO/CAM_GPIO1
- Module1 pad 101: unconnected-(Module1B-USB_OTG_ID-Pad101) -> /CM5_GPIO/USBOTG
- Module1 pad 102: unconnected-(Module1B-PCIe_nCLKREQ-Pad102) -> /CM5_high_speed/PCIE_nCLKREQ
- Module1 pad 103: unconnected-(Module1B-USB2_N-Pad103) -> /Battery_charger/MUX_D-
- Module1 pad 104: unconnected-(Module1B-PCIE_nWAKE-Pad104) -> /CM5_high_speed/PCIE_nWAKE
- Module1 pad 105: unconnected-(Module1B-USB2_P-Pad105) -> /Battery_charger/MUX_D+
- Module1 pad 106: unconnected-(Module1B-PCIE_PWR_EN-Pad106) -> /CM5_high_speed/PCIE_PWR_EN
- Module1 pad 107: unconnected-(Module1B-GND-Pad107) -> GND
- Module1 pad 108: unconnected-(Module1B-GND-Pad108) -> GND
- Module1 pad 109: unconnected-(Module1B-PCIe_nRST-Pad109) -> /CM5_high_speed/PCIE_nRST
- Module1 pad 11: unconnected-(Module1A-Ethernet_Pair2_P-Pad11) -> /CM5_GPIO/TRD2_P
- Module1 pad 110: unconnected-(Module1B-PCIe_CLK_P-Pad110) -> /CM5_high_speed/PCIE_CLK_P
- Module1 pad 111: unconnected-(Module1B-VBUS_EN-Pad111) -> /CM5_high_speed/VBUS_EN
- Module1 pad 112: unconnected-(Module1B-PCIe_CLK_N-Pad112) -> /CM5_high_speed/PCIE_CLK_N
- Module1 pad 113: unconnected-(Module1B-GND-Pad113) -> GND
- Module1 pad 114: unconnected-(Module1B-GND-Pad114) -> GND
- Module1 pad 115: unconnected-(Module1B-MIPI0_D0_N-Pad115) -> /CM5_high_speed/DPHY0_D0_N
- Module1 pad 116: unconnected-(Module1B-PCIe_RX_P-Pad116) -> /CM5_high_speed/PCIE_RX_P
- Module1 pad 117: unconnected-(Module1B-MIPI0_D0_P-Pad117) -> /CM5_high_speed/DPHY0_D0_P
- Module1 pad 118: unconnected-(Module1B-PCIe_RX_N-Pad118) -> /CM5_high_speed/PCIE_RX_N
- Module1 pad 119: unconnected-(Module1B-GND-Pad119) -> GND
- Module1 pad 12: unconnected-(Module1A-Ethernet_Pair0_P-Pad12) -> /CM5_GPIO/TRD0_P
- Module1 pad 120: unconnected-(Module1B-GND-Pad120) -> GND
- Module1 pad 121: unconnected-(Module1B-MIPI0_D1_N-Pad121) -> /CM5_high_speed/DPHY0_D1_N
- Module1 pad 122: unconnected-(Module1B-PCIe_TX_P-Pad122) -> /CM5_high_speed/PCIE_TX_P
- Module1 pad 123: unconnected-(Module1B-MIPI0_D1_P-Pad123) -> /CM5_high_speed/DPHY0_D1_P
- Module1 pad 124: unconnected-(Module1B-PCIe_TX_N-Pad124) -> /CM5_high_speed/PCIE_TX_N
- Module1 pad 125: unconnected-(Module1B-GND-Pad125) -> GND
- Module1 pad 126: unconnected-(Module1B-GND-Pad126) -> GND
- Module1 pad 127: unconnected-(Module1B-MIPI0_C_N-Pad127) -> /CM5_high_speed/DPHY0_C_N
- Module1 pad 128: unconnected-(Module1B-USB3-0-RX_N-Pad128) -> /CM5_high_speed/USB3-0-RX_N
- Module1 pad 129: unconnected-(Module1B-MIPI0_C_P-Pad129) -> /CM5_high_speed/DPHY0_C_P
- Module1 pad 13: unconnected-(Module1A-GND-Pad13) -> GND
- Module1 pad 130: unconnected-(Module1B-USB3-0-RX_P-Pad130) -> /CM5_high_speed/USB3-0-RX_P
- Module1 pad 131: unconnected-(Module1B-GND-Pad131) -> GND
- Module1 pad 132: unconnected-(Module1B-GND-Pad132) -> GND
- Module1 pad 133: unconnected-(Module1B-MIPI0_D2_N-Pad133) -> /CM5_high_speed/DPHY0_D2_N
- Module1 pad 134: unconnected-(Module1B-USB3-0-D_P-Pad134) -> /CM5_high_speed/USB3-0-D_P
- Module1 pad 135: unconnected-(Module1B-MIPI0_D2_P-Pad135) -> /CM5_high_speed/DPHY0_D2_P
- Module1 pad 136: unconnected-(Module1B-USB3-0-D_N-Pad136) -> /CM5_high_speed/USB3-0-D_N
- Module1 pad 137: unconnected-(Module1B-GND-Pad137) -> GND
- Module1 pad 138: unconnected-(Module1B-GND-Pad138) -> GND
- Module1 pad 139: unconnected-(Module1B-MIPI0_D3_N-Pad139) -> /CM5_high_speed/DPHY0_D3_N
- Module1 pad 14: unconnected-(Module1A-GND-Pad14) -> GND
- Module1 pad 140: unconnected-(Module1B-USB3-0-TX_N-Pad140) -> /CM5_high_speed/USB3-0-TX_N
- Module1 pad 141: unconnected-(Module1B-MIPI0_D3_P-Pad141) -> /CM5_high_speed/DPHY0_D3_P
- Module1 pad 142: unconnected-(Module1B-USB3-0-TX_P-Pad142) -> /CM5_high_speed/USB3-0-TX_P
- Module1 pad 143: unconnected-(Module1B-HDMI1_HOTPLUG-Pad143) -> /CM5_high_speed/HDMI1_HOTPLUG
- Module1 pad 144: unconnected-(Module1B-GND-Pad144) -> GND
- Module1 pad 145: unconnected-(Module1B-HDMI1_SDA-Pad145) -> /CM5_high_speed/HDMI1_SDA
- Module1 pad 146: unconnected-(Module1B-HDMI1_TX2_P-Pad146) -> /CM5_high_speed/HDMI1_D2_P
- Module1 pad 147: unconnected-(Module1B-HDMI1_SCL-Pad147) -> /CM5_high_speed/HDMI1_SCL
- Module1 pad 148: unconnected-(Module1B-HDMI1_TX2_N-Pad148) -> /CM5_high_speed/HDMI1_D2_N
- Module1 pad 149: unconnected-(Module1B-HDMI1_CEC-Pad149) -> /CM5_high_speed/HDMI1_CEC
- Module1 pad 15: unconnected-(Module1A-Ethernet_nLED3(3.3v)-Pad15) -> /CM5_GPIO/ETH_LEDY
- Module1 pad 150: unconnected-(Module1B-GND-Pad150) -> GND
- Module1 pad 151: unconnected-(Module1B-HDMI0_CEC-Pad151) -> /CM5_high_speed/HDMI0_CEC
- Module1 pad 152: unconnected-(Module1B-HDMI1_TX1_P-Pad152) -> /CM5_high_speed/HDMI1_D1_P
- Module1 pad 153: unconnected-(Module1B-HDMI0_HOTPLUG-Pad153) -> /CM5_high_speed/HDMI0_HOTPLUG
- Module1 pad 154: unconnected-(Module1B-HDMI1_TX1_N-Pad154) -> /CM5_high_speed/HDMI1_D1_N
- Module1 pad 155: unconnected-(Module1B-GND-Pad155) -> GND
- Module1 pad 156: unconnected-(Module1B-GND-Pad156) -> GND
- Module1 pad 157: unconnected-(Module1B-USB3-1-RX_N-Pad157) -> /CM5_high_speed/USB3-1-RX_N
- Module1 pad 158: unconnected-(Module1B-HDMI1_TX0_P-Pad158) -> /CM5_high_speed/HDMI1_D0_P
- Module1 pad 159: unconnected-(Module1B-USB3-1-RX_P-Pad159) -> /CM5_high_speed/USB3-1-RX_P
- Module1 pad 16: unconnected-(Module1A-FAN_TACHO-Pad16) -> /CM5_GPIO/TACHO
- Module1 pad 160: unconnected-(Module1B-HDMI1_TX0_N-Pad160) -> /CM5_high_speed/HDMI1_D0_N
- Module1 pad 161: unconnected-(Module1B-GND-Pad161) -> GND
- Module1 pad 162: unconnected-(Module1B-GND-Pad162) -> GND
- Module1 pad 163: unconnected-(Module1B-USB3-1-D_P-Pad163) -> /CM5_high_speed/USB3-1-D_P
- Module1 pad 164: unconnected-(Module1B-HDMI1_CLK_P-Pad164) -> /CM5_high_speed/HDMI1_CK_P
- Module1 pad 165: unconnected-(Module1B-USB3-1-D_N-Pad165) -> /CM5_high_speed/USB3-1-D_N
- Module1 pad 166: unconnected-(Module1B-HDMI1_CLK_N-Pad166) -> /CM5_high_speed/HDMI1_CK_N
- Module1 pad 167: unconnected-(Module1B-GND-Pad167) -> GND
- Module1 pad 168: unconnected-(Module1B-GND-Pad168) -> GND
- Module1 pad 169: unconnected-(Module1B-USB3-1-TX_N-Pad169) -> /CM5_high_speed/USB3-1-TX_N
- Module1 pad 17: unconnected-(Module1A-Ethernet_nLED2(3.3v)-Pad17) -> /CM5_GPIO/ETH_LEDG
- Module1 pad 170: unconnected-(Module1B-HDMI0_TX2_P-Pad170) -> /CM5_high_speed/HDMI0_D2_P
- Module1 pad 171: unconnected-(Module1B-USB3-1-TX_P-Pad171) -> /CM5_high_speed/USB3-1-TX_P
- Module1 pad 172: unconnected-(Module1B-HDMI0_TX2_N-Pad172) -> /CM5_high_speed/HDMI0_D2_N
- Module1 pad 173: unconnected-(Module1B-GND-Pad173) -> GND
- Module1 pad 174: unconnected-(Module1B-GND-Pad174) -> GND
- Module1 pad 175: unconnected-(Module1B-MIPI1_D0_N-Pad175) -> /CM5_high_speed/DPHY1_D0_N
- Module1 pad 176: unconnected-(Module1B-HDMI0_TX1_P-Pad176) -> /CM5_high_speed/HDMI0_D1_P
- Module1 pad 177: unconnected-(Module1B-MIPI1_D0_P-Pad177) -> /CM5_high_speed/DPHY1_D0_P
- Module1 pad 178: unconnected-(Module1B-HDMI0_TX1_N-Pad178) -> /CM5_high_speed/HDMI0_D1_N
- Module1 pad 179: unconnected-(Module1B-GND-Pad179) -> GND
- Module1 pad 18: unconnected-(Module1A-Ethernet_SYNC_OUT(3.3v)-Pad18) -> /CM5_GPIO/SYNC_OUT
- Module1 pad 180: unconnected-(Module1B-GND-Pad180) -> GND
- Module1 pad 181: unconnected-(Module1B-MIPI1_D1_N-Pad181) -> /CM5_high_speed/DPHY1_D1_N
- Module1 pad 182: unconnected-(Module1B-HDMI0_TX0_P-Pad182) -> /CM5_high_speed/HDMI0_D0_P
- Module1 pad 183: unconnected-(Module1B-MIPI1_D1_P-Pad183) -> /CM5_high_speed/DPHY1_D1_P
- Module1 pad 184: unconnected-(Module1B-HDMI0_TX0_N-Pad184) -> /CM5_high_speed/HDMI0_D0_N
- Module1 pad 185: unconnected-(Module1B-GND-Pad185) -> GND
- Module1 pad 186: unconnected-(Module1B-GND-Pad186) -> GND
- Module1 pad 187: unconnected-(Module1B-MIPI1_C_N-Pad187) -> /CM5_high_speed/DPHY1_C_N
- Module1 pad 188: unconnected-(Module1B-HDMI0_CLK_P-Pad188) -> /CM5_high_speed/HDMI0_CK_P
- Module1 pad 189: unconnected-(Module1B-MIPI1_C_P-Pad189) -> /CM5_high_speed/DPHY1_C_P
- Module1 pad 19: unconnected-(Module1A-FAN_PWM-Pad19) -> /CM5_GPIO/PWM
- Module1 pad 190: unconnected-(Module1B-HDMI0_CLK_N-Pad190) -> /CM5_high_speed/HDMI0_CK_N
- Module1 pad 191: unconnected-(Module1B-GND-Pad191) -> GND
- Module1 pad 192: unconnected-(Module1B-GND-Pad192) -> GND
- Module1 pad 193: unconnected-(Module1B-MIPI1_D2_N-Pad193) -> /CM5_high_speed/DPHY1_D2_N
- Module1 pad 194: unconnected-(Module1B-MIPI1_D3_N-Pad194) -> /CM5_high_speed/DPHY1_D3_N
- Module1 pad 195: unconnected-(Module1B-MIPI1_D2_P-Pad195) -> /CM5_high_speed/DPHY1_D2_P
- Module1 pad 196: unconnected-(Module1B-MIPI1_D3_P-Pad196) -> /CM5_high_speed/DPHY1_D3_P
- Module1 pad 197: unconnected-(Module1B-GND-Pad197) -> GND
- Module1 pad 198: unconnected-(Module1B-GND-Pad198) -> GND
- Module1 pad 199: unconnected-(Module1B-HDMI0_SDA-Pad199) -> /CM5_high_speed/HDMI0_SDA
- Module1 pad 2: unconnected-(Module1A-GND-Pad2) -> GND
- Module1 pad 20: unconnected-(Module1A-EEPROM_nWP-Pad20) -> /CM5_GPIO/EEPROM_nWP
- Module1 pad 200: unconnected-(Module1B-HDMI0_SCL-Pad200) -> /CM5_high_speed/HDMI0_SCL
- Module1 pad 21: unconnected-(Module1A-LED_nACT-Pad21) -> Net-(Module1A-LED_nACT)
- Module1 pad 22: unconnected-(Module1A-GND-Pad22) -> GND
- Module1 pad 23: unconnected-(Module1A-GND-Pad23) -> GND
- Module1 pad 24: unconnected-(Module1A-GPIO26-Pad24) -> /CM5_GPIO/GPIO26
- Module1 pad 25: unconnected-(Module1A-GPIO21-Pad25) -> /CM5_GPIO/GPIO21
- Module1 pad 26: unconnected-(Module1A-GPIO19-Pad26) -> /CM5_GPIO/GPIO19
- Module1 pad 27: unconnected-(Module1A-GPIO20-Pad27) -> /CM5_GPIO/GPIO20
- Module1 pad 28: unconnected-(Module1A-GPIO13-Pad28) -> /CM5_GPIO/GPIO13
- Module1 pad 29: unconnected-(Module1A-GPIO16-Pad29) -> /CM5_GPIO/GPIO16
- Module1 pad 3: unconnected-(Module1A-Ethernet_Pair3_P-Pad3) -> /CM5_GPIO/TRD3_P
- Module1 pad 30: unconnected-(Module1A-GPIO6-Pad30) -> /CM5_GPIO/GPIO6
- Module1 pad 31: unconnected-(Module1A-GPIO12-Pad31) -> /CM5_GPIO/GPIO12
- Module1 pad 32: unconnected-(Module1A-GND-Pad32) -> GND
- Module1 pad 33: unconnected-(Module1A-GND-Pad33) -> GND
- Module1 pad 34: unconnected-(Module1A-GPIO5-Pad34) -> /CM5_GPIO/GPIO5
- Module1 pad 35: unconnected-(Module1A-ID_SC-Pad35) -> /CM5_GPIO/ID_SC
- Module1 pad 36: unconnected-(Module1A-ID_SD-Pad36) -> /CM5_GPIO/ID_SD
- Module1 pad 37: unconnected-(Module1A-GPIO7-Pad37) -> /CM5_GPIO/GPIO7
- Module1 pad 38: unconnected-(Module1A-GPIO11-Pad38) -> /CM5_GPIO/GPIO11
- Module1 pad 39: unconnected-(Module1A-GPIO8-Pad39) -> /CM5_GPIO/GPIO8
- Module1 pad 4: unconnected-(Module1A-Ethernet_Pair1_P-Pad4) -> /CM5_GPIO/TRD1_P
- Module1 pad 40: unconnected-(Module1A-GPIO9-Pad40) -> /CM5_GPIO/GPIO9
- Module1 pad 41: unconnected-(Module1A-GPIO25-Pad41) -> /CM5_GPIO/GPIO25
- Module1 pad 42: unconnected-(Module1A-GND-Pad42) -> GND
- Module1 pad 43: unconnected-(Module1A-GND-Pad43) -> GND
- Module1 pad 44: unconnected-(Module1A-GPIO10-Pad44) -> /CM5_GPIO/GPIO10
- Module1 pad 45: unconnected-(Module1A-GPIO24-Pad45) -> /CM5_GPIO/GPIO24
- Module1 pad 46: unconnected-(Module1A-GPIO22-Pad46) -> /CM5_GPIO/GPIO22
- Module1 pad 47: unconnected-(Module1A-GPIO23-Pad47) -> /CM5_GPIO/GPIO23
- Module1 pad 48: unconnected-(Module1A-GPIO27-Pad48) -> /CM5_GPIO/GPIO27
- Module1 pad 49: unconnected-(Module1A-GPIO18-Pad49) -> /CM5_GPIO/GPIO18
- Module1 pad 5: unconnected-(Module1A-Ethernet_Pair3_N-Pad5) -> /CM5_GPIO/TRD3_N
- Module1 pad 50: unconnected-(Module1A-GPIO17-Pad50) -> /CM5_GPIO/GPIO17
- Module1 pad 51: unconnected-(Module1A-GPIO15-Pad51) -> /CM5_GPIO/GPIO15
- Module1 pad 52: unconnected-(Module1A-GND-Pad52) -> GND
- Module1 pad 53: unconnected-(Module1A-GND-Pad53) -> GND
- Module1 pad 54: unconnected-(Module1A-GPIO4-Pad54) -> /CM5_GPIO/GPIO4
- Module1 pad 55: unconnected-(Module1A-GPIO14-Pad55) -> /CM5_GPIO/GPIO14
- Module1 pad 56: unconnected-(Module1A-GPIO3-Pad56) -> /CM5_GPIO/GPIO3
- Module1 pad 57: unconnected-(Module1A-SD_CLK-Pad57) -> /CM5_GPIO/SD_CLK
- Module1 pad 58: unconnected-(Module1A-GPIO2-Pad58) -> /CM5_GPIO/GPIO2
- Module1 pad 59: unconnected-(Module1A-GND-Pad59) -> GND
- Module1 pad 6: unconnected-(Module1A-Ethernet_Pair1_N-Pad6) -> /CM5_GPIO/TRD1_N
- Module1 pad 60: unconnected-(Module1A-GND-Pad60) -> GND
- Module1 pad 61: unconnected-(Module1A-SD_DAT3-Pad61) -> /CM5_GPIO/SD_DAT3
- Module1 pad 62: unconnected-(Module1A-SD_CMD-Pad62) -> /CM5_GPIO/SD_CMD
- Module1 pad 63: unconnected-(Module1A-SD_DAT0-Pad63) -> /CM5_GPIO/SD_DAT0
- Module1 pad 65: unconnected-(Module1A-GND-Pad65) -> GND
- Module1 pad 66: unconnected-(Module1A-GND-Pad66) -> GND
- Module1 pad 67: unconnected-(Module1A-SD_DAT1-Pad67) -> /CM5_GPIO/SD_DAT1
- Module1 pad 69: unconnected-(Module1A-SD_DAT2-Pad69) -> /CM5_GPIO/SD_DAT2
- Module1 pad 7: unconnected-(Module1A-GND-Pad7) -> GND
- Module1 pad 71: unconnected-(Module1A-GND-Pad71) -> GND
- Module1 pad 74: unconnected-(Module1A-GND-Pad74) -> GND
- Module1 pad 75: unconnected-(Module1A-SD_PWR_ON-Pad75) -> /CM5_GPIO/SD_PWR_ON
- Module1 pad 76: unconnected-(Module1A-VBAT-Pad76) -> /CM5_GPIO/VBAT
- Module1 pad 77: unconnected-(Module1A-+5v_(Input)-Pad77) -> +5V
- Module1 pad 78: unconnected-(Module1A-GPIO_VREF(1.8v/3.3v_Input)-Pad78) -> +3V3
- Module1 pad 79: unconnected-(Module1A-+5v_(Input)-Pad79) -> +5V
- Module1 pad 8: unconnected-(Module1A-GND-Pad8) -> GND
- Module1 pad 80: unconnected-(Module1A-SCL0-Pad80) -> /CM5_high_speed/SCL0
- Module1 pad 81: unconnected-(Module1A-+5v_(Input)-Pad81) -> +5V
- Module1 pad 82: unconnected-(Module1A-SDA0-Pad82) -> /CM5_high_speed/SDA0
- Module1 pad 83: unconnected-(Module1A-+5v_(Input)-Pad83) -> +5V
- Module1 pad 84: unconnected-(Module1A-+3.3v_(Output)-Pad84) -> +3V3
- Module1 pad 85: unconnected-(Module1A-+5v_(Input)-Pad85) -> +5V
- Module1 pad 86: unconnected-(Module1A-+3.3v_(Output)-Pad86) -> +3V3
- Module1 pad 87: unconnected-(Module1A-+5v_(Input)-Pad87) -> +5V
- Module1 pad 88: unconnected-(Module1A-+1.8v_(Output)-Pad88) -> /CM5_GPIO/+1.8v
- Module1 pad 89: unconnected-(Module1A-WiFi_nDisable-Pad89) -> /CM5_GPIO/WL_nDis
- Module1 pad 9: unconnected-(Module1A-Ethernet_Pair2_N-Pad9) -> /CM5_GPIO/TRD2_N
- Module1 pad 90: unconnected-(Module1A-+1.8v_(Output)-Pad90) -> /CM5_GPIO/+1.8v
- Module1 pad 91: unconnected-(Module1A-BT_nDisable-Pad91) -> /CM5_GPIO/BT_nDis
- Module1 pad 92: unconnected-(Module1A-PWR_BUT-Pad92) -> /CM5_GPIO/PWR_BUT
- Module1 pad 93: unconnected-(Module1A-nRPIBOOT-Pad93) -> /CM5_GPIO/nRPIBOOT
- Module1 pad 94: unconnected-(Module1A-CC1-Pad94) -> /CM5_GPIO/CC1
- Module1 pad 95: unconnected-(Module1A-LED_nPWR-Pad95) -> /CM5_GPIO/nPWR_LED
- Module1 pad 96: unconnected-(Module1A-CC2-Pad96) -> /CM5_GPIO/CC2
- Module1 pad 97: unconnected-(Module1A-CAM_GPIO0-Pad97) -> /CM5_GPIO/CAM_GPIO0
- Module1 pad 98: unconnected-(Module1A-GND-Pad98) -> GND
- Module1 pad 99: unconnected-(Module1A-PMIC_ENABLE-Pad99) -> /CM5_GPIO/PMIC_ENABLE
- R1 pad 1: /pcie-nvme/M.2_3v3 -> +3V3
- R1 pad 2: /pcie-nvme/FB -> /CM5_GPIO/GPIO5
- R10 pad 1: +3V3 -> /Battery_charger/SEL
- R10 pad 2: /battery_charger/INT -> +3V_CHRG
- R11 pad 1: /battery_charger/OTG -> /CM5_GPIO/GPIO17
- R12 pad 1: /battery_charger/CE -> Net-(U1-REGN)
- R12 pad 2: GND -> Net-(J5-Pin_1)
- R13 pad 1: Net-(U1-REGN) -> Net-(J5-Pin_1)
- R13 pad 2: Net-(J4-Pin_1) -> GND
- R14 pad 1: Net-(J4-Pin_1) -> +3V_CHRG
- R14 pad 2: GND -> /CM5_GPIO/GPIO22
- R15 pad 2: Net-(U2-FB) -> Net-(U4-FB)
- R16 pad 1: Net-(U2-FB) -> Net-(U4-FB)
- R2 pad 1: /pcie-nvme/FB -> +3V3
- R2 pad 2: GND -> /CM5_GPIO/GPIO4
- R3 pad 1: /pcie-nvme/PCIE_PWR_EN -> Net-(D2-K)
- R3 pad 2: GND -> /CM5_GPIO/nPWR_LED
- R4 pad 2: Net-(J1-DAS/~{DSS}/~{LED1}) -> Net-(Module1A-LED_nACT)
- R5 pad 1: Net-(D2-A) -> Net-(D3-A)
- R5 pad 2: /battery_charger/Vsys -> /Battery_charger/Vsys
- R8 pad 1: Net-(U1-ILIM) -> +3V_CHRG
- R8 pad 2: GND -> /CM5_GPIO/GPIO27
- R9 pad 1: /battery_charger/SEL -> Net-(U1-ILIM)
- R9 pad 2: +3V3 -> GND
- U1 pad 11: Net-(J4-Pin_1) -> Net-(J5-Pin_1)
- U1 pad 12: /battery_charger/RESET -> /Battery_charger/RESET
- U1 pad 13: /battery_charger/Fuel_G -> /Battery_charger/Fuel_G
- U1 pad 14: /battery_charger/Fuel_G -> /Battery_charger/Fuel_G
- U1 pad 15: /battery_charger/Vsys -> /Battery_charger/Vsys
- U1 pad 16: /battery_charger/Vsys -> /Battery_charger/Vsys
- U1 pad 19: Net-(C10-Pad1) -> Net-(C7-Pad1)
- U1 pad 2: /battery_charger/CHG_D+ -> /Battery_charger/CHG_D+
- U1 pad 20: Net-(C10-Pad1) -> Net-(C7-Pad1)
- U1 pad 24: /battery_charger/SEL -> /Battery_charger/SEL
- U1 pad 3: /battery_charger/CHG_D- -> /Battery_charger/CHG_D-
- U1 pad 4: Net-(D2-K) -> Net-(D3-K)
- U1 pad 5: /battery_charger/SCL -> /CM5_GPIO/GPIO3
- U1 pad 6: /battery_charger/SDA -> /CM5_GPIO/GPIO2
- U1 pad 7: /battery_charger/INT -> /CM5_GPIO/GPIO27
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Other:
- copper layers 2 -> 6

Commit message: all
Parts:
- removed C1: 100nF 6.3V, Capacitor_SMD:C_0603_1608Metric_Pad1.08x0.95mm_HandSolder
- removed C2: 0.1F 5.5V, Capacitor_SMD:CP_Elec_10x10.5
- C10, C11, C12, C13, C14, C15, C16, C17, C18, C19, C20, C21, C22, C23, C3, C34, C35, C36, C37, C38, C39, C4, C40, C41, C42, C5, C6, C7, C8, C9, D1, D2, D3, D4, D8, IC1, J11, J12, J2, J3, J5, J8, L1, L2, L5, R1, R10, R11, R12, R13, R14, R15, R16, R2, R21, R22, R23, R24, R3, R4, R5, R6, R7, R8, R9, SW1, SW2, TP1, TP2, TP3, TP4, U1, U10, U2, U3, U4, U9: moved to B.Cu
- J1: value Conn_01x22_Female -> Conn_01x22_MountingPin
- J4: value Conn_01x02_Socket -> Conn_01x02_MountingPin; moved to B.Cu
- moved C3 118.6 mm to (115.4, 146.3), turned to 90 degrees
- moved C4 115.8 mm to (112.9, 146.3), turned to 90 degrees
- moved C11 113.8 mm to (115.4, 141.9), turned to 90 degrees
- moved C5 113.0 mm to (110.4, 146.3), turned to 90 degrees
- moved C12 111.0 mm to (112.9, 141.9), turned to 90 degrees
- moved C6 110.3 mm to (107.9, 146.3), turned to 90 degrees
- moved IC1 110.0 mm to (104.2, 150.5), turned to 90 degrees
- moved R8 109.1 mm to (115.4, 137.6), turned to 90 degrees
- moved C13 108.3 mm to (110.4, 141.9), turned to 90 degrees
- moved C7 107.6 mm to (105.4, 146.3), turned to 90 degrees
- moved R9 106.4 mm to (112.9, 137.6), turned to 90 degrees
- moved C14 105.7 mm to (107.9, 141.9), turned to 90 degrees
- moved C8 105.0 mm to (102.9, 146.3), turned to 90 degrees
- moved U3 104.9 mm to (98.0, 152.0), turned to 90 degrees
- moved R10 103.8 mm to (110.4, 137.6), turned to 90 degrees
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Connections:
- J1 pad MP: (no net) -> GND
- J4 pad MP: (no net) -> GND
- Module1 pad 76: /CM5_GPIO/VBAT -> +3V_CHRG

Commit message: all
Parts:
- added C58: 10uF 6.3V, Resistor_SMD:R_0603_1608Metric_Pad0.98x0.95mm_HandSolder, F.Cu at (165.1, 82.2)
- added J13: Conn_01x22_MountingPin, CM5IO:Hirose_FH12-22S-0.5SH_1x22-1MP_P0.50mm_Horizontal, F.Cu at (145.5, 64.0)
- added J14: Micro_SD_Card_Det, CM5IO:SDCARD_MOLEX_503398-1892, F.Cu at (155.4, 84.1)
- added R36: 10K 1%, Resistor_SMD:R_0603_1608Metric_Pad0.98x0.95mm_HandSolder, F.Cu at (165.1, 84.7)
- added R37: 2.2K 1%, Resistor_SMD:R_0603_1608Metric_Pad0.98x0.95mm_HandSolder, F.Cu at (140.0, 56.5)
- added R38: 2.2K 1%, Resistor_SMD:R_0603_1608Metric_Pad0.98x0.95mm_HandSolder, F.Cu at (140.0, 59.0)
- added U18: RT9742GGJ5 / NCP380HSN10AAT1G, Package_TO_SOT_SMD:SOT-23-5, F.Cu at (169.1, 75.9)
- C23: footprint Capacitor_SMD:C_0603_1608Metric_Pad1.08x0.95mm_HandSolder -> Resistor_SMD:R_1206_3216Metric
- J4: footprint Connector_JST:JST_PH_B2B-PH-SM4-TB_1x02-1MP_P2.00mm_Vertical -> Connector_JST:JST_PH_S2B-PH-SM4-TB_1x02-1MP_P2.00mm_Horizontal
- R24: value 2.2k 1% -> 2.2K 1%
- U3: footprint TLV70430DBVR:DBV0005A_N -> TLV70430DBVR:DBV0005A_M
- moved J4 31.6 mm to (80.0, 133.5)
- moved J1 8.00 mm to (94.0, 55.5)

Commit message: all
Parts:
- removed C28: 56pF 50V, Capacitor_SMD:C_0402_1005Metric_Pad0.74x0.62mm_HandSolder
- removed J2: Conn_01x03, Connector_PinHeader_2.54mm:PinHeader_1x03_P2.54mm_Vertical
- removed J6: Conn_Coaxial, Connector_Coaxial:U.FL_Hirose_U.FL-R-SMT-1_Vertical
- removed TP1, TP2: TestPoint, TestPoint:TestPoint_Pad_2.0x2.0mm
- added J15: Conn_Coaxial, Connector_Coaxial:SMA_Molex_73251-2120_EdgeMount_Horizontal, F.Cu at (138.3, 38.8)
- D5: footprint Diode_SMD:D_SMA -> Diode_SMD:D_0201_0603Metric_Pad0.64x0.40mm_HandSolder
- J1: moved to B.Cu
- R11, R8: moved to F.Cu
- R17: footprint Resistor_SMD:R_0402_1005Metric_Pad0.72x0.64mm_HandSolder -> Resistor_SMD:R_0603_1608Metric_Pad0.98x0.95mm_HandSolder
- SW4, SW5: footprint PCM_Switch_Keyboard_Kailh:SW_Kailh_Choc_V2 -> PCM_Switch_Keyboard_Kailh:SW_Kailh_Choc_V1V2_1.00u
- moved C47 92.6 mm to (135.9, 136.8)
- moved R25 92.6 mm to (140.2, 136.8)
- moved J13 76.1 mm to (72.7, 42.0), turned to 180 degrees
- moved R37 66.6 mm to (73.9, 48.3)
- moved R38 66.6 mm to (73.9, 50.8)
- moved TP4 48.4 mm to (66.3, 139.1), turned to 0 degrees
- moved Q2 47.8 mm to (71.0, 109.3), turned to 180 degrees
- moved Q1 47.3 mm to (139.7, 66.8)
- moved R8 47.3 mm to (106.8, 91.1), turned to 180 degrees
- moved C44 45.9 mm to (99.0, 78.4)
- moved C45 45.9 mm to (99.0, 80.9)
- moved D6 45.3 mm to (142.8, 64.5), turned to 90 degrees
- moved C26 44.6 mm to (139.2, 64.0)
- moved R11 44.2 mm to (106.7, 93.4), turned to 180 degrees
- moved C24 43.8 mm to (139.3, 57.6)
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Connections:
- U6 pad 11: Net-(U6-RF_IN) -> Net-(D5-A1)
Routing:
- net Net-(D5-A1): track 0.00 -> 6.75 mm
Other:
- board outline added: 80 x 120 mm
