File: KB-01_kicad/KB-01/KB-01.kicad_pcb (KiCad board)
At the start: 6 copper layers, 80 x 120 mm, 134 parts, among them IC1 MAX17048G+T10, J1 Conn_01x22_MountingPin, J11 Conn_02x07_Odd_Even, J12 Conn_01x01_Socket, J13 Conn_01x22_MountingPin, J14 Micro_SD_Card_Det, J15 Conn_Coaxial, J3 USB_C_Receptacle_USB2.0_14P, J4 Conn_01x02_MountingPin, J5 Conn_01x01_Socket, J8 Bus_M.2_Socket_M, J9 AudioJack3_SwitchTR, Q1 MMBT3904, Q2 2N7002, SW1 Right angle Tact button, SW2 Power button, SW3 RotaryEncoder_Switch_MP, SW4 SW_Push, SW5 SW_Push, U1 BQ25895, U10 AP3441SHE-7B, U11 BMP581, U12 BMI270, U13 SHT40, U14 LIS2MDL, U18 RT9742GGJ5 / NCP380HSN10AAT1G, U2 TS3USB30ERSWR, U3 TLV70430DBVR, U4 TPS61022, U5 TLV773_SOT353, U6 TESEO-LIV4F, U9 ASEK-32.768KHZ-L-R-T

Commit message: all
Parts:
- added H1: MountingHole, MountingHole:MountingHole_2.7mm_M2.5_DIN965, F.Cu at (70.5, 100.0)
- added H2: MountingHole, MountingHole:MountingHole_2.7mm_M2.5_DIN965, F.Cu at (128.5, 100.0)
- added H3: MountingHole, MountingHole:MountingHole_2.7mm_M2.5_DIN965, F.Cu at (128.5, 51.0)
- added H4: MountingHole, MountingHole:MountingHole_2.7mm_M2.5_DIN965, F.Cu at (70.5, 51.0)

Commit message: all
Parts:
- moved U10 28.5 mm to (110.5, 94.9), turned to -90 degrees
- moved C34 27.9 mm to (93.9, 73.6), turned to -90 degrees
- moved C39 24.0 mm to (93.9, 77.9), turned to -90 degrees
- moved C35 23.9 mm to (96.4, 73.6), turned to -90 degrees
- moved R22 22.9 mm to (93.9, 82.3), turned to -90 degrees
- moved L5 22.8 mm to (96.3, 88.5), turned to -90 degrees
- moved D8 22.5 mm to (101.0, 91.9), turned to -90 degrees
- moved C36 20.5 mm to (98.9, 73.6), turned to -90 degrees
- moved U12 20.4 mm to (103.9, 58.9)
- moved U11 19.9 mm to (103.9, 42.6)
- moved C45 19.7 mm to (104.2, 61.9)
- moved C44 19.7 mm to (107.2, 60.5), turned to -90 degrees
- moved C40 19.3 mm to (96.4, 77.9), turned to -90 degrees
- moved R23 17.9 mm to (96.4, 82.3), turned to -90 degrees
- moved C37 17.8 mm to (101.5, 73.6), turned to -90 degrees
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
Commit message: all
Parts:
- C10, C11, C12, C13, C14, C15, C3, C4, C5, C6, C7, C8, C9, D1, D2, D3, D4, D8, IC1, J12, J3, J4, J5, L1, R10, R12, R13, R14, R21, R3, R4, R5, R6, R7, R9, SW1, TP3, TP4, U1, U2, U3: moved to F.Cu
- C24, C25, C26, C27, D5, J15, Module1, R11, R8, U5, U6: moved to B.Cu
- SW2: footprint Button_Switch_SMD:SW_Push_1P1T_NO_CK_KSC6xxJ -> Button_Switch_SMD:SW_SPST_EVQP7A; moved to F.Cu
- moved C47 70.0 mm to (67.2, 150.3), turned to 90 degrees
- moved J5 69.5 mm to (138.1, 154.4), turned to 180 degrees
- moved J12 63.7 mm to (135.2, 154.4), turned to 180 degrees
- moved J9 63.3 mm to (73.6, 148.1)
- moved R25 61.7 mm to (80.1, 150.8), turned to -90 degrees
- moved U10 54.8 mm to (79.3, 49.8), turned to 180 degrees
- moved C15 53.1 mm to (131.1, 143.2), turned to 90 degrees
- moved IC1 50.1 mm to (128.6, 143.1), turned to 180 degrees
- moved D8 49.3 mm to (64.4, 58.9), turned to 90 degrees
- moved R14 48.9 mm to (126.0, 143.2), turned to 90 degrees
- moved Module1 48.0 mm to (78.5, 100.3)
- moved J4 47.2 mm to (127.0, 150.1), turned to 0 degrees
- moved R2 44.9 mm to (98.6, 96.2), turned to -90 degrees
- moved C51 43.7 mm to (72.0, 79.6)
- moved U13 43.7 mm to (69.9, 79.6)
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Connections:
- U3 pad 4: unconnected-(U3-NC-Pad4) -> GND
- U3 pad 5: unconnected-(U3-NC-Pad5) -> GND
Routing:
- net Net-(C54-Pad1): track 0.00 -> 6.82 mm
- net Net-(C55-Pad1): track 0.00 -> 6.80 mm
- net Net-(C53-Pad1): track 0.00 -> 5.36 mm
- net /CM5_GPIO/GPIO12: track 0.00 -> 3.80 mm
- net /CM5_GPIO/GPIO13: track 0.00 -> 3.70 mm
