File: KB-01_kicad/KB-01/ui.kicad_sch (KiCad schematic)
At the start: 16 parts, among them Q2 2N7002, SW3 RotaryEncoder_Switch_MP, SW4 SW_Push, SW5 SW_Push

Commit message: all
Parts:
- R19, R24, R25, R26: mouser 71-CRCW060310K0FKEE -> 71-CRCW060310K0FKEE
- R28: mouser (none) -> 71-CRCW060310K0FKEE

Commit message: all
Connections:
- net +3V3 renamed +3.3v

Commit message: all
Parts:
- C48, C49: value 100n -> 100nF 6.3V; mouser 581-KGM15AR70J104KM -> 581-KGM15AR70J104KT
- SW3: footprint (none) -> Rotary_Encoder:RotaryEncoder_Bourns_Vertical_PEC12R-3x17F-Sxxxx; mouser (none) -> 652-PEC12R-4220F-S12
Changed lines of the file:
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@@
 			)
 		)
-		(property "Footprint" ""
+		(property "Footprint" "Rotary_Encoder:RotaryEncoder_Bourns_Vertical_PEC12R-3x17F-Sxxxx"
 			(at 86.36 67.056 0)
 			(hide yes)
@@
 		)
 		(property "SNAPEDA_PN" ""
+			(at 90.17 71.12 0)
+			(hide yes)
+			(show_name no)
+			(do_not_autoplace no)
+			(effects
+				(font
+					(size 1.27 1.27)
+				)
+			)
+		)
+		(property "mouser" "652-PEC12R-4220F-S12"
 			(at 90.17 71.12 0)
 			(hide yes)
@@
 			)
 		)
-		(property "Value" "100n"
+		(property "Value" "100nF 6.3V"
 			(at 67.818 83.566 0)
 			(show_name no)
@@
 			)
 		)
-		(property "mouser" "581-KGM15AR70J104KM"
+		(property "mouser" "581-KGM15AR70J104KT"
 			(at 73.66 81.28 0)
 			(hide yes)
@@
 			)
 		)
-		(property "Value" "100n"
+		(property "Value" "100nF 6.3V"
 			(at 99.568 77.216 0)
 			(show_name no)
@@
 			)
 		)
-		(property "mouser" "581-KGM15AR70J104KM"
+		(property "mouser" "581-KGM15AR70J104KT"
 			(at 105.41 74.93 0)
 			(hide yes)
@@
 			)
 		)
-		(property "Value" "100n"
+		(property "Value" "100nF 6.3V"
 			(at 57.15 82.3214 0)
 			(show_name no)
@@
 			)
 		)
-		(property "mouser" "581-KGM15AR70J104KM"
+		(property "mouser" "581-KGM15AR70J104KT"
 			(at 64.77 81.28 0)
 			(hide yes)

Commit message: all
Parts:
- added C54, C55: 100nF 6.3V, Capacitor_SMD:C_0603_1608Metric_Pad1.08x0.95mm_HandSolder, symbol Device:C
- added R32, R33, R34: 1k, Resistor_SMD:R_0603_1608Metric_Pad0.98x0.95mm_HandSolder, symbol Device:R
- D9: mouser (none) -> 637-1N4148W
- LS1: footprint CMT050203SMTTR -> CMT-0502-03SMTTR:CMT050203SMTTR; mouser (none) -> 179-CMT-0502-03SMTTR
- Q2: mouser (none) -> 621-2N7002A-7
- R27: mouser (none) -> 279-CRGH0603F180R
- SW4, SW5: footprint (none) -> PCM_Switch_Keyboard_Kailh:SW_Kailh_Choc_V2
Connections:
- net GND: now also C54.2, C55.2
- net PUSH_BT_ENC: now also R34.2; no longer C49.1, R24.2, SW3.S1
- net Push_button1: now also R32.1; no longer R25.2, SW4.1
- net Push_button2: now also R33.1; no longer R26.2, SW5.1
- new net: C55.1, R26.2, R33.2, SW5.1
- new net: C54.1, R25.2, R32.2, SW4.1
- new net: C49.1, R24.2, R34.1, SW3.S1
Other:
- moved on the sheet: R26, SW5

Commit message: all
Parts:
- R32, R33, R34: mouser 594-MCT06030C2201FP5 -> 652-CR0603FX-1001ELF
Changed lines of the file:
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@@
 			)
 		)
-		(property "mouser" "594-MCT06030C2201FP5 "
+		(property "mouser" "652-CR0603FX-1001ELF "
 			(at 227.33 71.12 0)
 			(hide yes)
@@
 			)
 		)
-		(property "mouser" "594-MCT06030C2201FP5 "
+		(property "mouser" "652-CR0603FX-1001ELF "
 			(at 160.02 71.12 0)
 			(hide yes)
@@
 			)
 		)
-		(property "mouser" "594-MCT06030C2201FP5 "
+		(property "mouser" "652-CR0603FX-1001ELF "
 			(at 111.76 68.58 0)
 			(hide yes)

Commit message: all
Parts:
- renumbered C49 to C53, C48 to C56, C48 to C57, R19 to R26, R19 to R27, R24 to R28, R25 to R29, R26 to R30, R34 to R31, R27 to R34, R28 to R35
Changed lines of the file:
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@@
 		(dnp no)
 		(fields_autoplaced yes)
-		(property "Reference" "R19"
+		(property "Reference" "R26"
 			(at 67.31 60.9599 0)
 			(show_name no)
@@
 			(project "KB-01"
 				(path "/e6144e29-1dc4-45a8-93e7-988a20131b94/223a1f40-08cb-4cda-b03a-4c087618db35"
-					(reference "R19")
+					(reference "R26")
 					(unit 1)
 				)
@@
 		(dnp no)
 		(fields_autoplaced yes)
-		(property "Reference" "#PWR079"
+		(property "Reference" "#PWR083"
 			(at 166.37 85.09 0)
 			(hide yes)
@@
 			(project "KB-01"
 				(path "/e6144e29-1dc4-45a8-93e7-988a20131b94/223a1f40-08cb-4cda-b03a-4c087618db35"
-					(reference "#PWR079")
+					(reference "#PWR083")
 					(unit 1)
 				)
@@
 		(dnp no)
 		(fields_autoplaced yes)
-		(property "Reference" "R27"
+		(property "Reference" "R34"
 			(at 144.78 118.11 90)
 			(show_name no)
@@
 			(project "KB-01"
 				(path "/e6144e29-1dc4-45a8-93e7-988a20131b94/223a1f40-08cb-4cda-b03a-4c087618db35"
-					(reference "R27")
+					(reference "R34")
 					(unit 1)
 				)
@@
 		(dnp no)
 		(fields_autoplaced yes)
-		(property "Reference" "R25"
+		(property "Reference" "R29"
 			(at 168.91 64.7699 0)
 			(show_name no)
@@
 			(project "KB-01"
 				(path "/e6144e29-1dc4-45a8-93e7-988a20131b94/223a1f40-08cb-4cda-b03a-4c087618db35"
-					(reference "R25")
+					(reference "R29")
 					(unit 1)
 				)
@@
 		(in_pos_files yes)
 		(dnp no)
-		(property "Reference" "R19"
+		(property "Reference" "R27"
 			(at 76.2 60.9599 0)
 			(show_name no)
@@
 			(project "KB-01"
 				(path "/e6144e29-1dc4-45a8-93e7-988a20131b94/223a1f40-08cb-4cda-b03a-4c087618db35"
-					(reference "R19")
+					(reference "R27")
 					(unit 1)
 				)
@@
 		(in_pos_files yes)
 		(dnp no)
-		(property "Reference" "R28"
+		(property "Reference" "R35"
 			(at 152.654 126.746 0)
 			(show_name no)
@@
 			(project "KB-01"
 				(path "/e6144e29-1dc4-45a8-93e7-988a20131b94/223a1f40-08cb-4cda-b03a-4c087618db35"
-					(reference "R28")
+					(reference "R35")
 					(unit 1)
 				)
@@
 		(dnp no)
 		(fields_autoplaced yes)
-		(property "Reference" "R24"
+		(property "Reference" "R28"
 			(at 105.41 60.9599 0)
 			(show_name no)
@@
 			(project "KB-01"
 				(path "/e6144e29-1dc4-45a8-93e7-988a20131b94/223a1f40-08cb-4cda-b03a-4c087618db35"
-					(reference "R24")
+					(reference "R28")
 					(unit 1)
 				)
@@
 		(dnp no)
 		(fields_autoplaced yes)
-		(property "Reference" "R34"
+		(property "Reference" "R31"
 			(at 111.76 62.23 90)
 			(show_name no)
@@
 			(project "KB-01"
 				(path "/e6144e29-1dc4-45a8-93e7-988a20131b94/223a1f40-08cb-4cda-b03a-4c087618db35"
-					(reference "R34")
+					(reference "R31")
 					(unit 1)
 				)
@@
 		(dnp no)
 		(fields_autoplaced yes)
-		(property "Reference" "R26"
+		(property "Reference" "R30"
 			(at 237.49 64.7699 0)
 			(show_name no)
@@
 			(project "KB-01"
 				(path "/e6144e29-1dc4-45a8-93e7-988a20131b94/223a1f40-08cb-4cda-b03a-4c087618db35"
-					(reference "R26")
+					(reference "R30")
 					(unit 1)
 				)
@@
 		(dnp no)
 		(fields_autoplaced yes)
-		(property "Reference" "#PWR072"
+		(property "Reference" "#PWR081"
 			(at 185.42 82.55 0)
 			(hide yes)
@@
 			(project "KB-01"
 				(path "/e6144e29-1dc4-45a8-93e7-988a20131b94/223a1f40-08cb-4cda-b03a-4c087618db35"
-					(reference "#PWR072")
+					(reference "#PWR081")
 					(unit 1)
 				)
@@
 		(dnp no)
 		(fields_autoplaced yes)
-		(property "Reference" "#PWR074"
+		(property "Reference" "#PWR082"
 			(at 254 82.55 0)
 			(hide yes)
@@
 			(project "KB-01"
 				(path "/e6144e29-1dc4-45a8-93e7-988a20131b94/223a1f40-08cb-4cda-b03a-4c087618db35"
-					(reference "#PWR074")
+					(reference "#PWR082")
 					(unit 1)
 				)
@@
 		(dnp no)
 		(fields_autoplaced yes)
-		(property "Reference" "#PWR080"
+		(property "Reference" "#PWR084"
 			(at 234.95 85.09 0)
 			(hide yes)
@@
 			(project "KB-01"
 				(path "/e6144e29-1dc4-45a8-93e7-988a20131b94/223a1f40-08cb-4cda-b03a-4c087618db35"
-					(reference "#PWR080")
+					(reference "#PWR084")
 					(unit 1)
 				)
@@
 		(dnp no)
 		(fields_autoplaced yes)
-		(property "Reference" "#PWR078"
+		(property "Reference" "#PWR086"
 			(at 160.02 142.24 0)
 			(hide yes)
@@
 			(project "KB-01"
 				(path "/e6144e29-1dc4-45a8-93e7-988a20131b94/223a1f40-08cb-4cda-b03a-4c087618db35"
-					(reference "#PWR078")
+					(reference "#PWR086")
 					(unit 1)
 				)
@@
 		(in_pos_files yes)
 		(dnp no)
-		(property "Reference" "C48"
+		(property "Reference" "C57"
 			(at 68.326 78.994 0)
 			(show_name no)
@@
 			(project "KB-01"
 				(path "/e6144e29-1dc4-45a8-93e7-988a20131b94/223a1f40-08cb-4cda-b03a-4c087618db35"
-					(reference "C48")
+					(reference "C57")
 					(unit 1)
 				)
@@
 		(in_pos_files yes)
 		(dnp no)
-		(property "Reference" "C49"
+		(property "Reference" "C53"
 			(at 100.076 72.644 0)
 			(show_name no)
@@
 			(project "KB-01"
 				(path "/e6144e29-1dc4-45a8-93e7-988a20131b94/223a1f40-08cb-4cda-b03a-4c087618db35"
-					(reference "C49")
+					(reference "C53")
 					(unit 1)
 				)
@@
 		(in_pos_files yes)
 		(dnp no)
-		(property "Reference" "C48"
+		(property "Reference" "C56"
 			(at 57.15 80.01 0)
 			(show_name no)
@@
 			(project "KB-01"
 				(path "/e6144e29-1dc4-45a8-93e7-988a20131b94/223a1f40-08cb-4cda-b03a-4c087618db35"
-					(reference "C48")
+					(reference "C56")
 					(unit 1)
 				)
@@
 		(dnp no)
 		(fields_autoplaced yes)
-		(property "Reference" "#PWR069"
+		(property "Reference" "#PWR085"
 			(at 78.74 97.79 0)
 			(hide yes)
@@
 			(project "KB-01"
 				(path "/e6144e29-1dc4-45a8-93e7-988a20131b94/223a1f40-08cb-4cda-b03a-4c087618db35"
-					(reference "#PWR069")
+					(reference "#PWR085")
 					(unit 1)
 				)

Commit message: all
Parts:
- SW4, SW5: footprint PCM_Switch_Keyboard_Kailh:SW_Kailh_Choc_V2 -> PCM_Switch_Keyboard_Kailh:SW_Kailh_Choc_V1V2_1.00u
Changed lines of the file:
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@@
 			)
 		)
-		(property "Footprint" "PCM_Switch_Keyboard_Kailh:SW_Kailh_Choc_V2"
+		(property "Footprint" "PCM_Switch_Keyboard_Kailh:SW_Kailh_Choc_V1V2_1.00u"
 			(at 246.38 66.04 0)
 			(hide yes)
@@
 			)
 		)
-		(property "Footprint" "PCM_Switch_Keyboard_Kailh:SW_Kailh_Choc_V2"
+		(property "Footprint" "PCM_Switch_Keyboard_Kailh:SW_Kailh_Choc_V1V2_1.00u"
 			(at 177.8 66.04 0)
 			(hide yes)
